File: board/BLDCdriver_test/untitled.sch (EAGLE design)
At the start: 0 parts

Commit message: making encorder board
Parts:
- added X1: JST-XH-03-PIN-LONG-PAD, Rembrandt Electronics - JST XH Connectors v1-0:JST-XH-03-PIN-LONG-PAD
