File: board/BLDCdriver_test/encorder.sch (EAGLE design)
At the start: 0 parts

Commit message: made encorder board
Parts:
- added 5V, CLK, CS, GND, MISO, MOSI: (no value), wirepad:SMD2
- added C1: 100nF, generic:CAPACITOR1608
- added C2: 1µF, generic:CAPACITOR1608
- added IC1: AS5047P-ATSM, rcssl_lib:AS5047P-ATSM
- added LED1: LED1608, generic:LED1608
- added R1: (no value), generic:RESISTOR1608
Connections:
- new net GND: C1.2, C2.2, GND.P, IC1.GND, IC1.TEST, LED1.K
- new net N$1: C2.1, IC1.VDD3V
- new net N$2: CS.P, IC1.CSN
- new net N$3: CLK.P, IC1.CLK
- new net N$4: IC1.MISO, MISO.P
- new net N$5: IC1.MOSI, MOSI.P
- new net N$6: LED1.A, R1.2
- new net VCC: 5V.P, C1.1, IC1.I/PWM, IC1.VDD, R1.1
