File: board/BLDCdriver_test/encorder.sch (EAGLE design)
At the start: 11 parts, among them IC1 AS5047P-ATSM

Commit message: update encorder board
Parts:
- R1: value (none) -> 1kΩ
Changed lines of the file:
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@@
 <part name="GND3" library="supply" deviceset="GND" device=""/>
 <part name="LED1" library="generic" deviceset="LED" device="1608"/>
-<part name="R1" library="generic" deviceset="RESISTOR" device="1608"/>
+<part name="R1" library="generic" deviceset="RESISTOR" device="1608" value="1kΩ"/>
 <part name="GND4" library="supply" deviceset="GND" device=""/>
 <part name="U$3" library="supply" deviceset="VCC" device=""/>
