File: board/BLDCdriver_test/encorder.brd (EAGLE design)
At the start: 18 x 12.7 mm, 11 parts, among them IC1 AS5047P-ATSM

Commit message: encorder & linesensor
Routing:
- net VCC: track 15.1 -> 17.4 mm, vias 1 -> 2
Changed lines of the file:
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@@
 <?xml version="1.0" encoding="utf-8"?>
 <!DOCTYPE eagle SYSTEM "eagle.dtd">
-<eagle version="9.6.1">
+<eagle version="9.6.2">
 <drawing>
 <settings>
-<setting alwaysvectorfont="yes"/>
+<setting alwaysvectorfont="no"/>
 <setting verticaltext="up"/>
 </settings>
@@
 </layers>
 <board>
-<fusionsync huburn="a.cGVyc29uYWw6dWUyYjhiNWJj" projecturn="a.cGVyc29uYWw6dWUyYjhiNWJjIzIwMjIwNDE2NTE3MzEzNjU2" f3durn="urn:adsk.wipprod:dm.lineage:B6GV1yHgS0yyPmqctDIGeQ" pcbguid="0ba3597e-a119-49d4-b5ec-b11a965633ef" lastpulledtime="" lastsyncedchangeguid="" latestrevisionid="170bb0a8-9025-4ee9-be30-9e13ce0d5fac" lastsyncedrevisionid="170bb0a8-9025-4ee9-be30-9e13ce0d5fac" lastboardhashguid="f80ba58b-ac47-2349-3679-81f1b1a1cb82" lastpushedtime="2022-04-23T14:40:00Z" linktopcb3d="%12"/>
+<fusionsync huburn="a.cGVyc29uYWw6dWUyYjhiNWJj" projecturn="a.cGVyc29uYWw6dWUyYjhiNWJjIzIwMjIwNDE2NTE3MzEzNjU2" f3durn="urn:adsk.wipprod:dm.lineage:B6GV1yHgS0yyPmqctDIGeQ" pcbguid="0ba3597e-a119-49d4-b5ec-b11a965633ef" lastpulledtime="" lastsyncedchangeguid="" latestrevisionid="170bb0a8-9025-4ee9-be30-9e13ce0d5fac" lastsyncedrevisionid="170bb0a8-9025-4ee9-be30-9e13ce0d5fac" lastboardhashguid="f80ba58b-ac47-2349-3679-81f1b1a1cb82" lastpushedtime="2022-04-23T14:40:00Z" linktopcb3d="false"/>
 <plain>
 <circle x="14.62" y="6.3" radius="1" width="0.001" layer="20"/>
@@
 <wire x1="11.43" y1="5.447" x2="11.43" y2="2.54" width="0.4064" layer="16"/>
 <contactref element="IC1" pad="14"/>
-<wire x1="11.035" y1="8.89" x2="10.558" y2="9.57" width="0" layer="19" extent="1-16"/>
+<wire x1="10.558" y1="9.57" x2="11.7159125" y2="9.57" width="0.3048" layer="1"/>
+<wire x1="11.7159125" y1="9.57" x2="11.78595625" y2="9.49995625" width="0.3048" layer="1"/>
+<via x="11.78595625" y="9.49995625" extent="1-16" drill="0.35"/>
+<wire x1="11.78595625" y1="9.49995625" x2="11.176" y2="8.89" width="0.3048" layer="16"/>
+<wire x1="11.176" y1="8.89" x2="11.035" y2="8.89" width="0.3048" layer="16"/>
 </signal>
 <signal name="GND">
@@
 <wire x1="4.6126" y1="8.8506" x2="3.79720625" y2="8.8506" width="0.4064" layer="1"/>
 <wire x1="3.79720625" y1="8.8506" x2="3.5889" y2="8.64229375" width="0.4064" layer="1"/>
-<wire x1="3.5889" y1="5.29770625" x2="3.79720625" y2="5.0894" width="0.4064" layer="1"/>
 <wire x1="3.5889" y1="8.64229375" x2="3.5889" y2="5.29770625" width="0.4064" layer="1"/>
-<wire x1="3.79720625" y1="5.0894" x2="3.8006" y2="5.0894" width="0.4064" layer="1"/>
 <wire x1="3.79720625" y1="5.0894" x2="3.81" y2="5.07660625" width="0.4064" layer="1"/>
 <wire x1="3.81" y1="5.07660625" x2="3.81" y2="2.54" width="0.4064" layer="1"/>
+<wire x1="3.5889" y1="5.29770625" x2="3.79720625" y2="5.0894" width="0.4064" layer="1"/>
 </signal>
 <signal name="N$4">

Commit message: update encorder board
Parts:
- R1: value (none) -> 1kΩ
