File: board/BLDCdriver_test/untitled.brd (EAGLE design)
At the start: 46 x 65 mm, 28 parts, among them M1 JST-XH-03-PIN-LONG-PAD, X1 JST-XH-02-PIN-LONG-PAD, X2 JST-XH-06-PIN-ROUND-PAD, X4 JST-XH-04-PIN-ROUND-PAD

Commit message: update boards 2022-07-14
Parts:
- C1, C2, C3: value (none) -> 1uF
- R7, R8, R9: value (none) -> 300Ω
Changed lines of the file:
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@@
 <drawing>
 <settings>
-<setting alwaysvectorfont="yes"/>
+<setting alwaysvectorfont="no"/>
 <setting verticaltext="up"/>
 </settings>
@@
 </layers>
 <board>
-<fusionsync huburn="a.cGVyc29uYWw6dWUyYjhiNWJj" projecturn="a.cGVyc29uYWw6dWUyYjhiNWJjIzIwMjIwNDE2NTE3MzEzNjU2" f3durn="urn:adsk.wipprod:dm.lineage:IwQo1QymROyITibKEIHzOA" pcbguid="16ff5ab9-c038-43ab-a8fb-72bf997d25e8" lastpulledtime="" lastsyncedchangeguid="" latestrevisionid="bef91a73-895b-44ec-aec5-9c8b8b043572" lastsyncedrevisionid="bef91a73-895b-44ec-aec5-9c8b8b043572" lastboardhashguid="baa7ce44-da11-1522-0302-304cf9931c19" lastpushedtime="2022-06-30T00:32:27Z" linktopcb3d="true"/>
+<fusionsync huburn="a.cGVyc29uYWw6dWUyYjhiNWJj" projecturn="a.cGVyc29uYWw6dWUyYjhiNWJjIzIwMjIwNDE2NTE3MzEzNjU2" f3durn="urn:adsk.wipprod:dm.lineage:IwQo1QymROyITibKEIHzOA" pcbguid="" lastpulledtime="" lastsyncedchangeguid="" latestrevisionid="bef91a73-895b-44ec-aec5-9c8b8b043572" lastsyncedrevisionid="bef91a73-895b-44ec-aec5-9c8b8b043572" lastboardhashguid="baa7ce44-da11-1522-0302-304cf9931c19" lastpushedtime="2022-06-30T00:32:27Z" linktopcb3d="false"/>
 <plain>
 <wire x1="0" y1="-3" x2="0" y2="56" width="0.001" layer="20"/>
@@
 <attribute name="VALUE" x="37.211" y="29.9085" size="1.27" layer="27" rot="R180"/>
 </element>
-<element name="C1" library="adafruit" package="C2012" value="" x="32.0675" y="16.51" smashed="yes">
+<element name="C1" library="adafruit" package="C2012" value="1uF" x="32.0675" y="16.51" smashed="yes">
 <attribute name="NAME" x="31.1785" y="17.526" size="1.27" layer="25"/>
 <attribute name="VALUE" x="31.1785" y="14.224" size="1.27" layer="27"/>
 </element>
-<element name="C2" library="adafruit" package="C2012" value="" x="36.5125" y="16.51" smashed="yes">
+<element name="C2" library="adafruit" package="C2012" value="1uF" x="36.5125" y="16.51" smashed="yes">
 <attribute name="NAME" x="35.6235" y="17.526" size="1.27" layer="25"/>
 <attribute name="VALUE" x="35.6235" y="14.224" size="1.27" layer="27"/>
@@
 <attribute name="VALUE" x="41.9735" y="25.654" size="1.27" layer="27" rot="R90"/>
 </element>
-<element name="C3" library="adafruit" package="C2012" value="" x="32.0675" y="27.6225" smashed="yes" rot="R180">
+<element name="C3" library="adafruit" package="C2012" value="1uF" x="32.0675" y="27.6225" smashed="yes" rot="R180">
 <attribute name="NAME" x="32.9565" y="26.6065" size="1.27" layer="25" rot="R180"/>
 <attribute name="VALUE" x="32.9565" y="29.9085" size="1.27" layer="27" rot="R180"/>
@@
 <attribute name="VALUE" x="-0.0825" y="39.7175" size="1.016" layer="27" ratio="10" rot="R90"/>
 </element>
-<element name="R7" library="adafruit" package="M2012" value="" x="14.9225" y="47.9425" smashed="yes" rot="R180">
+<element name="R7" library="adafruit" package="M2012" value="300Ω" x="14.9225" y="47.9425" smashed="yes" rot="R180">
 <attribute name="NAME" x="15.9385" y="46.9265" size="1.27" layer="25" rot="R180"/>
 <attribute name="VALUE" x="15.9385" y="50.2285" size="1.27" layer="27" rot="R180"/>
 </element>
-<element name="R8" library="adafruit" package="M2012" value="" x="19.05" y="46.99" smashed="yes" rot="R180">
+<element name="R8" library="adafruit" package="M2012" value="300Ω" x="19.05" y="46.99" smashed="yes" rot="R180">
 <attribute name="NAME" x="20.066" y="45.974" size="1.27" layer="25" rot="R180"/>
 <attribute name="VALUE" x="20.066" y="49.276" size="1.27" layer="27" rot="R180"/>
 </element>
-<element name="R9" library="adafruit" package="M2012" value="" x="10.795" y="48.895" smashed="yes" rot="R180">
+<element name="R9" library="adafruit" package="M2012" value="300Ω" x="10.795" y="48.895" smashed="yes" rot="R180">
 <attribute name="NAME" x="11.811" y="47.879" size="1.27" layer="25" rot="R180"/>
 <attribute name="VALUE" x="11.811" y="51.181" size="1.27" layer="27" rot="R180"/>
