File: board/line_sensor_test/untitled.brd (EAGLE design)
At the start: 100 x 100 mm, 92 parts, among them U1 74HC4067SSOP-24, U2 74HC4067SSOP-24

Commit message: making linesonsor_2
Parts:
- moved U2 47.6 mm to (38.1, 0.00), turned to 180 degrees
- moved U1 46.7 mm to (-38.1, 0.00), turned to 0 degrees
- moved R2 11.4 mm to (3.30, 35.7)
- moved R1 5.24 mm to (-0.25, 38.2)
Connections:
- net A1: now also U2.9
- net A10: now also U2.22
- net A11: now also U2.21
- net A12: now also U2.20
- net A13: now also U2.19
- net A14: now also U2.18
- net A15: now also U2.17
- net A16: now also U2.16
- net A2: now also U2.8
- net A3: now also U2.7
- net A4: now also U2.6
- net A5: now also U2.5
- net A6: now also U2.4
- net A7: now also U2.3
- net A8: now also U2.2
- net A9: now also U2.23
- net GND: now also U1.12, U2.12
- net VCC: now also U1.24, U2.24
Routing:
- net A1: track 0.00 -> 72.6 mm
- net A2: track 0.00 -> 61.2 mm
- net A3: track 0.00 -> 50.8 mm
- net A13: track 0.00 -> 41.5 mm
- net A4: track 0.00 -> 40.6 mm
- net A12: track 0.00 -> 32.2 mm
- net A5: track 0.00 -> 31.6 mm
- net A14: track 0.00 -> 31.2 mm
- net A6: track 0.00 -> 22.0 mm
- net A11: track 0.00 -> 21.7 mm
- net A15: track 0.00 -> 19.4 mm
- net A7: track 0.00 -> 12.3 mm
- net A10: track 0.00 -> 12.1 mm
- net A16: track 0.00 -> 9.55 mm
- net A9: track 0.00 -> 5.49 mm
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