File: board/line_sensor_test/untitled.brd (EAGLE design)
At the start: 100 x 100 mm, 92 parts, among them U1 74HC4067SSOP-24, U2 74HC4067SSOP-24

Commit message: making linesensor_3
Parts:
- moved R3 29.6 mm to (0.00, 45.7)
- moved R2 13.6 mm to (14.4, 43.7), flipped to the bottom, turned to 18 degrees
- moved R1 8.95 mm to (4.83, 45.6), flipped to the bottom, turned to 6 degrees
Connections:
- removed net GND1: R1.1, R10.1, R11.1, R12.1, R13.1, R14.1, R15.1, R16.1, R17.1, R18.1, R19.1, R2.1, R20.1, R21.1, R22.1, R23.1, R24.1, R25.1, R26.1, R27.1, R28.1, R29.1, R3.1, R30.1, R4.1, R5.1, R6.1, R7.1, R8.1, R9.1
- net GND: now also R1.1, R10.1, R11.1, R12.1, R13.1, R14.1, R15.1, R16.1, R17.1, R18.1, R19.1, R2.1, R20.1, R21.1, R22.1, R23.1, R24.1, R25.1, R26.1, R27.1, R28.1, R29.1, R3.1, R30.1, R4.1, R5.1, R6.1, R7.1, R8.1, R9.1
Routing:
- net A16: track 9.55 -> 69.6 mm
- net A15: track 19.4 -> 60.3 mm
- net A14: track 31.2 -> 50.6 mm
- net GND: track 0.00 -> 14.7 mm, vias 0 -> 1
- net A2: track 61.2 -> 65.2 mm
- net A1: track 72.6 -> 76.5 mm

Commit message: put resister
Parts:
- moved R30 315.0 mm to (-4.78, 45.4), flipped to the bottom, turned to 354 degrees
- moved R29 306.3 mm to (-14.1, 43.5), flipped to the bottom, turned to 342 degrees
- moved R28 302.2 mm to (-22.9, 39.6), flipped to the bottom, turned to 330 degrees
- moved R27 277.0 mm to (-30.6, 34.0), flipped to the bottom, turned to 318 degrees
- moved R26 264.4 mm to (-37.0, 26.9), flipped to the bottom, turned to 306 degrees
- moved R25 256.1 mm to (-41.7, 18.6), flipped to the bottom, turned to 294 degrees
- moved R24 228.0 mm to (-44.7, 9.50), flipped to the bottom, turned to 282 degrees
- moved R23 209.6 mm to (-45.7, 0.00), flipped to the bottom, turned to 270 degrees
- moved R22 191.2 mm to (-44.6, -9.50), flipped to the bottom, turned to 258 degrees
- moved R21 173.3 mm to (-41.7, -18.6), flipped to the bottom, turned to 246 degrees
- moved R20 156.3 mm to (-37.0, -26.9), flipped to the bottom, turned to 234 degrees
- moved R19 141.0 mm to (-30.6, -34.0), flipped to the bottom, turned to 222 degrees
- moved R18 127.8 mm to (-22.9, -39.6), flipped to the bottom, turned to 210 degrees
- moved R8 120.0 mm to (45.7, 0.00), flipped to the bottom, turned to 90 degrees
- moved R7 119.6 mm to (44.7, 9.50), flipped to the bottom, turned to 78 degrees
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Connections:
- net A24: now also U1.23
Routing:
- net GND: track 14.7 -> 391.9 mm, vias 1 -> 31
- net VCC: track 330.5 -> 341.3 mm
- net A15: track 60.3 -> 64.3 mm
- net A6: track 22.0 -> 25.8 mm
- net A19: track 0.00 -> 3.84 mm
- net A10: track 12.1 -> 15.9 mm
- net A17: track 0.00 -> 3.84 mm
- net A11: track 21.7 -> 25.5 mm
- net A7: track 12.3 -> 16.2 mm
- net A25: track 0.00 -> 3.84 mm
- net A24: track 0.00 -> 3.84 mm
- net A4: track 40.6 -> 44.5 mm
- net A23: track 0.00 -> 3.84 mm
- net A28: track 0.00 -> 3.84 mm
- net A30: track 0.00 -> 3.84 mm
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
Commit message: Making linesensor
Parts:
- added SV1: (no value), con-lstb:MA06-2
Connections:
- new net AIN0: U1.1
- new net AIN1: SV1.11, U2.1
- new net N$10: SV1.7, U2.13
- new net N$11: SV1.9, U2.14
- new net N$13: SV1.10, U2.11
- new net N$14: SV1.12, U2.10
- new net N$15: U1.4
- new net N$5: U1.10
- new net N$7: U1.11
- new net N$8: U1.14
- new net N$9: U1.13
- net A22: now also U1.3
- net A23: now also U1.2
- net GND: now also SV1.8, U1.15, U2.15
Routing:
- net GND: track 391.9 -> 449.4 mm, vias 31 -> 33
- net AIN1: track 0.00 -> 37.9 mm
- net N$10: track 0.00 -> 37.0 mm
- net N$11: track 0.00 -> 35.5 mm
- net N$13: track 0.00 -> 35.2 mm
- net N$14: track 0.00 -> 32.3 mm
- net VCC: track 341.3 -> 357.4 mm, vias 29 -> 31
- net A22: track 3.81 -> 16.9 mm
- net A23: track 3.84 -> 9.31 mm
- net A24: track 3.84 -> 9.28 mm
- net A8: track 5.42 -> 9.25 mm
- net A1: track 73.3 -> 76.1 mm
Other:
- outline, holes or cut-outs redrawn

Commit message: update linesensor
Connections:
- removed net N$15: U1.4
- net A16: now also U1.9
- net A17: now also U1.8
- net A18: now also U1.7
- net A19: now also U1.6
- net A20: now also U1.5
- net A21: now also U1.4
Routing:
- net A17: track 3.84 -> 63.5 mm
- net A18: track 3.84 -> 54.8 mm
- net A19: track 3.84 -> 45.4 mm
- net A20: track 3.84 -> 36.8 mm
- net A21: track 3.75 -> 26.8 mm

Commit message: Making linesensor
Connections:
- net A16: no longer U1.9
- net A17: now also U1.9; no longer U1.8
- net A18: now also U1.8; no longer U1.7
- net A19: now also U1.7; no longer U1.6
- net A20: now also U1.6; no longer U1.5
- net A21: now also U1.5; no longer U1.4
- net A22: now also U1.4; no longer U1.3
- net A23: now also U1.3; no longer U1.2
- net A24: now also U1.2; no longer U1.23
- net A25: now also U1.23
- net A26: now also U1.22
- net A27: now also U1.21
- net A28: now also U1.20
- net A29: now also U1.19
- net A30: now also U1.18
- net AIN0: now also SV1.1
- net N$8: now also SV1.2
Routing:
- net A30: track 3.84 -> 62.4 mm
- net A29: track 3.84 -> 53.4 mm
- net A28: track 3.84 -> 44.1 mm
- net AIN0: track 0.00 -> 38.6 mm
- net A27: track 3.84 -> 34.8 mm
- net A26: track 3.84 -> 25.6 mm
- net A25: track 3.84 -> 15.7 mm
- net A24: track 9.28 -> 16.0 mm, vias 0 -> 2
- net N$8: track 0.00 -> 2.87 mm
- net A17: track 63.5 -> 64.1 mm
- net A23: track 9.31 -> 9.88 mm

Commit message: Making linesensor
Connections:
- removed net N$5: U1.10
- removed net N$7: U1.11
- new net N$15: SV1.5, U1.11
- new net N$16: SV1.3, U1.10
- net N$9: now also SV1.4
- net VCC: now also SV1.6
Routing:
- net VCC: track 357.4 -> 400.2 mm, vias 31 -> 32
- net N$15: track 0.00 -> 37.4 mm
- net N$16: track 0.00 -> 35.7 mm
- net N$9: track 0.00 -> 34.5 mm
- net N$8: track 2.87 -> 31.9 mm
- net GND: track 449.4 -> 456.1 mm, vias 33 -> 34
- net A24: track 16.0 -> 15.0 mm
Changed lines of the file:
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@@
 <drawing>
 <settings>
-<setting alwaysvectorfont="yes"/>
+<setting alwaysvectorfont="no"/>
 <setting verticaltext="up"/>
 </settings>
@@
 <wire x1="-44.575" y1="2.54" x2="-48.00556875" y2="2.54" width="0.508" layer="16"/>
 <wire x1="-44.2702" y1="2.5674" x2="-43.2054" y2="3.6322" width="0.508" layer="1"/>
+<wire x1="-43.2054" y1="3.6322" x2="-41.9172" y2="3.6322" width="0.508" layer="1"/>
+<contactref element="SV1" pad="6"/>
 <wire x1="-41.9172" y1="3.6322" x2="-41.91" y2="3.625" width="0.508" layer="1"/>
-<wire x1="-43.2054" y1="3.6322" x2="-41.9172" y2="3.6322" width="0.508" layer="1"/>
+<wire x1="-41.91" y1="3.625" x2="-41.91" y2="2.54" width="0.508" layer="1"/>
+<wire x1="-41.91" y1="2.54" x2="-41.275" y2="1.905" width="0.508" layer="1"/>
+<wire x1="-41.275" y1="1.905" x2="-41.021" y2="1.905" width="0.508" layer="1"/>
+<via x="-41.021" y="1.905" extent="1-16" drill="0.35"/>
+<wire x1="-41.021" y1="1.905" x2="-10.795" y2="1.905" width="0.508" layer="16"/>
+<wire x1="-10.795" y1="1.905" x2="-10.16" y2="2.54" width="0.508" layer="16"/>
+<wire x1="-10.16" y1="2.54" x2="-2.54" y2="2.54" width="0.508" layer="16"/>
+<wire x1="-2.54" y1="2.54" x2="-1.27" y2="1.27" width="0.508" layer="16"/>
 </signal>
 <signal name="A6">
@@
 <wire x1="-42.668215625" y1="1.591459375" x2="-42.56963125" y2="1.492875" width="0.1524" layer="16"/>
 <wire x1="-42.56963125" y1="1.492875" x2="-42.56963125" y2="-0.99136875" width="0.1524" layer="16"/>
-<wire x1="-42.037" y1="-1.524" x2="-41.021" y2="-1.524" width="0.1524" layer="16"/>
 <via x="-41.021" y="-1.524" extent="1-16" drill="0.35"/>
 <wire x1="-41.021" y1="-1.524" x2="-41.021" y2="-3.621" width="0.1524" layer="1"/>
 <wire x1="-41.021" y1="-3.621" x2="-41.025" y2="-3.625" width="0.1524" layer="1"/>
 <wire x1="-42.56963125" y1="-0.99136875" x2="-42.037" y2="-1.524" width="0.1524" layer="16"/>
+<wire x1="-42.037" y1="-1.524" x2="-41.021" y2="-1.524" width="0" layer="19" extent="16-16"/>
 </signal>
 <signal name="A25">
@@
 <via x="-2.286" y="44.323" extent="1-16" drill="0.35"/>
 <wire x1="-2.286" y1="44.323" x2="-3.683" y2="44.069" width="0.508" layer="16"/>
-<wire x1="-34.525" y1="-3.625" x2="-34.525" y2="-2.813" width="0.508" layer="1"/>
-<wire x1="-34.525" y1="-2.813" x2="-34.970653125" y2="-2.367346875" width="0.508" layer="1"/>
 <wire x1="40.47345625" y1="-20.592315625" x2="40.132" y2="-21.336" width="0.508" layer="1"/>
 <via x="40.132" y="-21.336" extent="1-16" drill="0.35"/>
@@
 <wire x1="-45.38" y1="1.27" x2="-43.09056875" y2="1.27" width="0.508" layer="16"/>
 <wire x1="-43.06516875" y1="-2.341946875" x2="-43.06516875" y2="-2.367346875" width="0.508" layer="16"/>
-<wire x1="-43.06516875" y1="-2.367346875" x2="-34.970653125" y2="-2.367346875" width="0.508" layer="16"/>
-<via x="-34.970653125" y="-2.367346875" extent="1-16" drill="0.35"/>
-<wire x1="-34.970653125" y1="-2.367346875" x2="-35.825" y2="3.625" width="0" layer="19" extent="1-1"/>
+<wire x1="-34.462653125" y1="-2.367346875" x2="-34.29" y2="-2.54" width="0.508" layer="16"/>
+<via x="-34.29" y="-2.54" extent="1-16" drill="0.35"/>
+<wire x1="-34.29" y1="-2.54" x2="-34.29" y2="-3.39" width="0.508" layer="1"/>
+<wire x1="-43.06516875" y1="-2.367346875" x2="-36.195" y2="-2.367346875" width="0.508" layer="16"/>
+<wire x1="-36.195" y1="-2.367346875" x2="-34.462653125" y2="-2.367346875" width="0.508" layer="16"/>
+<wire x1="-34.29" y1="-3.39" x2="-34.525" y2="-3.625" width="0.4064" layer="1"/>
+<wire x1="-35.825" y1="3.625" x2="-35.825" y2="1.259" width="0.3048" layer="1"/>
+<wire x1="-35.825" y1="1.259" x2="-36.195" y2="0.889" width="0.3048" layer="1"/>
+<via x="-36.195" y="0.889" extent="1-16" drill="0.35"/>
+<wire x1="-36.195" y1="0.889" x2="-36.195" y2="-2.367346875" width="0.3048" layer="16"/>
 </signal>
 <signal name="N$6">
@@
 <contactref element="LED1" pad="4-DIN"/>
 </signal>
-<signal name="N$5">
-<contactref element="U1" pad="10"/>
-</signal>
-<signal name="N$7">
-<contactref element="U1" pad="11"/>
-</signal>
 <signal name="N$8">
 <contactref element="U1" pad="14"/>
 <contactref element="SV1" pad="2"/>
-<wire x1="-6.35" y1="1.27" x2="-7.4422" y2="0.1778" width="0.1524" layer="1"/>
-<wire x1="-7.4422" y1="0.1778" x2="-8.763" y2="0.1778" width="0.1524" layer="1"/>
-<wire x1="-8.763" y1="0.1778" x2="-35.175" y2="3.625" width="0" layer="19" extent="1-1"/>
+<wire x1="-6.35" y1="1.27" x2="-7.366" y2="0.254" width="0.3048" layer="1"/>
+<wire x1="-7.366" y1="0.254" x2="-8.89" y2="0.254" width="0.3048" layer="1"/>
+<wire x1="-8.89" y1="0.254" x2="-9.144" y2="0.254" width="0.3048" layer="1"/>
+<wire x1="-9.144" y1="0.254" x2="-34.036" y2="0.254" width="0.3048" layer="1"/>
+<wire x1="-35.175" y1="1.393" x2="-35.175" y2="3.625" width="0.3048" layer="1"/>
+<wire x1="-34.036" y1="0.254" x2="-35.175" y2="1.393" width="0.3048" layer="1"/>
 </signal>
 <signal name="N$9">
 <contactref element="U1" pad="13"/>
+<contactref element="SV1" pad="4"/>
+<wire x1="-34.525" y1="3.625" x2="-34.525" y2="1.38958125" width="0.3048" layer="1"/>
+<wire x1="-34.525" y1="1.38958125" x2="-33.84661875" y2="0.7112" width="0.3048" layer="1"/>
+<wire x1="-8.8138" y1="0.7112" x2="-6.985" y2="2.54" width="0.3048" layer="1"/>
+<wire x1="-6.985" y1="2.54" x2="-5.08" y2="2.54" width="0.3048" layer="1"/>
+<wire x1="-5.08" y1="2.54" x2="-3.81" y2="1.27" width="0.3048" layer="1"/>
+<wire x1="-33.84661875" y1="0.7112" x2="-8.8138" y2="0.7112" width="0.3048" layer="1"/>
 </signal>
 <signal name="AIN1">
@@
 <contactref element="U1" pad="1"/>
 <contactref element="SV1" pad="1"/>
-<wire x1="-41.577" y1="-1.29369375" x2="-40.53730625" y2="-0.254" width="0.1524" layer="1"/>
 <wire x1="-41.675" y1="-3.625" x2="-41.577" y2="-3.527" width="0.1524" layer="1"/>
-<wire x1="-41.577" y1="-3.527" x2="-41.577" y2="-1.29369375" width="0.1524" layer="1"/>
-<wire x1="-6.35" y1="-1.27" x2="-7.493" y2="-0.127" width="0.1524" layer="1"/>
-<wire x1="-40.41030625" y1="-0.127" x2="-40.53730625" y2="-0.254" width="0.1524" layer="1"/>
-<wire x1="-7.493" y1="-0.127" x2="-40.41030625" y2="-0.127" width="0.1524" layer="1"/>
+<wire x1="-7.4168" y1="-0.2032" x2="-6.35" y2="-1.27" width="0.3048" layer="1"/>
+<wire x1="-41.675" y1="-3.625" x2="-41.675" y2="-1.28393125" width="0.3048" layer="1"/>
+<wire x1="-41.675" y1="-1.28393125" x2="-40.59426875" y2="-0.2032" width="0.3048" layer="1"/>
+<wire x1="-40.59426875" y1="-0.2032" x2="-7.4168" y2="-0.2032" width="0.3048" layer="1"/>
 </signal>
 <signal name="N$10">
@@
 <wire x1="6.35" y1="1.27" x2="7.3914" y2="0.2286" width="0.3048" layer="1"/>
 </signal>
+<signal name="N$15">
+<contactref element="SV1" pad="5"/>
+<contactref element="U1" pad="11"/>
+<wire x1="-1.27" y1="-1.27" x2="-2.794" y2="-2.794" width="0.3048" layer="1"/>
+<wire x1="-7.25058125" y1="-2.794" x2="-8.92698125" y2="-1.1176" width="0.3048" layer="1"/>
+<wire x1="-2.794" y1="-2.794" x2="-7.25058125" y2="-2.794" width="0.3048" layer="1"/>
+<wire x1="-35.175" y1="-3.625" x2="-35.175" y2="-1.6216" width="0.3048" layer="1"/>
+<wire x1="-34.671" y1="-1.1176" x2="-35.175" y2="-1.6216" width="0.3048" layer="1"/>
+<wire x1="-8.92698125" y1="-1.1176" x2="-34.671" y2="-1.1176" width="0.3048" layer="1"/>
+</signal>
+<signal name="N$16">
+<contactref element="SV1" pad="3"/>
+<contactref element="U1" pad="10"/>
+<wire x1="-3.81" y1="-1.27" x2="-4.8768" y2="-2.3368" width="0.3048" layer="1"/>
+<wire x1="-8.7376" y1="-0.6604" x2="-7.0612" y2="-2.3368" width="0.3048" layer="1"/>
+<wire x1="-4.8768" y1="-2.3368" x2="-7.0612" y2="-2.3368" width="0.3048" layer="1"/>
+<wire x1="-35.825" y1="-3.625" x2="-35.825" y2="-1.4334" width="0.3048" layer="1"/>
+<wire x1="-35.825" y1="-1.4334" x2="-35.052" y2="-0.6604" width="0.3048" layer="1"/>
+<wire x1="-35.052" y1="-0.6604" x2="-8.7376" y2="-0.6604" width="0.3048" layer="1"/>
+</signal>
 </signals>

Commit message: encorder & linesensor
Parts:
- removed SV1: (no value), con-lstb:MA06-2
- added SV2: (no value), con-lstb:MA07-2
Connections:
- removed net N$60: LED1.4-DIN
- new net LED_IN: LED1.4-DIN, SV2.7
- new net LED_OUT: LED30.2-DOUT, SV2.8
- net AIN0: now also SV2.14; no longer SV1.1
- net AIN1: now also SV2.2; no longer SV1.11
- net GND: now also SV2.5; no longer SV1.8
- net N$10: now also SV2.6; no longer SV1.7
- net N$11: now also SV2.4; no longer SV1.9
- net N$13: now also SV2.3; no longer SV1.10
- net N$14: now also SV2.1; no longer SV1.12
- net N$15: now also SV2.10; no longer SV1.5
- net N$16: now also SV2.12; no longer SV1.3
- net N$8: now also SV2.13; no longer SV1.2
- net N$9: now also SV2.11; no longer SV1.4
- net VCC: now also SV2.9; no longer SV1.6
Routing:
- net LED_IN: track 0.00 -> 117.7 mm, vias 0 -> 3
- net LED_OUT: track 0.00 -> 104.0 mm, vias 0 -> 3
- net A1: track 76.1 -> 73.2 mm
- net AIN0: track 38.7 -> 37.3 mm
- net N$8: track 31.9 -> 30.7 mm
- net N$16: track 35.7 -> 34.4 mm
- net N$13: track 35.2 -> 34.0 mm
- net N$14: track 32.3 -> 31.0 mm
- net N$9: track 34.5 -> 33.2 mm
- net N$15: track 37.4 -> 36.2 mm
- net N$11: track 35.5 -> 34.3 mm
- net N$10: track 37.0 -> 35.7 mm
- net AIN1: track 37.9 -> 36.7 mm
- net VCC: track 400.2 -> 398.9 mm
- net GND: track 456.1 -> 454.9 mm
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Other:
- outline, holes or cut-outs redrawn
