File: board/line_sensor_test/untitled.sch (EAGLE design)
At the start: 93 parts, among them U1 74HC4067SSOP-24, U2 74HC4067SSOP-24

Commit message: Making linesensor
Connections:
- net A16: no longer U1.CHAN0
- net A17: now also U1.CHAN0; no longer U1.CHAN1
- net A18: now also U1.CHAN1; no longer U1.CHAN2
- net A19: now also U1.CHAN2; no longer U1.CHAN3
- net A20: now also U1.CHAN3; no longer U1.CHAN4
- net A21: now also U1.CHAN4; no longer U1.CHAN5
- net A22: now also U1.CHAN5; no longer U1.CHAN6
- net A23: now also U1.CHAN6; no longer U1.CHAN7
- net A24: now also U1.CHAN7; no longer U1.CHAN8
- net A25: now also U1.CHAN8
- net A26: now also U1.CHAN9
- net A27: now also U1.CHAN10
- net A28: now also U1.CHAN11
- net A29: now also U1.CHAN12
- net A30: now also U1.CHAN13
- net AIN0: now also SV1.1
- net N$8: now also SV1.2
Changed lines of the file:
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@@
 <label x="358.14" y="-93.98" size="1.778" layer="95" rot="R180" xref="yes"/>
-</segment>
-<segment>
-<pinref part="U1" gate="G$1" pin="CHAN0"/>
-<wire x1="363.22" y1="-5.08" x2="358.14" y2="-5.08" width="0.1524" layer="91"/>
-<label x="358.14" y="-5.08" size="1.778" layer="95" rot="R180" xref="yes"/>
 </segment>
 </net>
@@
 </segment>
 <segment>
-<pinref part="U1" gate="G$1" pin="CHAN1"/>
-<wire x1="363.22" y1="-7.62" x2="350.52" y2="-7.62" width="0.1524" layer="91"/>
-<label x="350.52" y="-7.62" size="1.778" layer="95" rot="R180" xref="yes"/>
+<pinref part="U1" gate="G$1" pin="CHAN0"/>
+<wire x1="363.22" y1="-5.08" x2="358.14" y2="-5.08" width="0.1524" layer="91"/>
+<label x="358.14" y="-5.08" size="1.778" layer="95" rot="R180" xref="yes"/>
 </segment>
 </net>
@@
 </segment>
 <segment>
-<pinref part="U1" gate="G$1" pin="CHAN2"/>
-<wire x1="363.22" y1="-10.16" x2="358.14" y2="-10.16" width="0.1524" layer="91"/>
-<label x="358.14" y="-10.16" size="1.778" layer="95" rot="R180" xref="yes"/>
+<pinref part="U1" gate="G$1" pin="CHAN1"/>
+<wire x1="363.22" y1="-7.62" x2="350.52" y2="-7.62" width="0.1524" layer="91"/>
+<label x="350.52" y="-7.62" size="1.778" layer="95" rot="R180" xref="yes"/>
 </segment>
 </net>
@@
 </segment>
 <segment>
-<pinref part="U1" gate="G$1" pin="CHAN3"/>
-<wire x1="363.22" y1="-12.7" x2="350.52" y2="-12.7" width="0.1524" layer="91"/>
-<label x="350.52" y="-12.7" size="1.778" layer="95" rot="R180" xref="yes"/>
+<pinref part="U1" gate="G$1" pin="CHAN2"/>
+<wire x1="363.22" y1="-10.16" x2="358.14" y2="-10.16" width="0.1524" layer="91"/>
+<label x="358.14" y="-10.16" size="1.778" layer="95" rot="R180" xref="yes"/>
 </segment>
 </net>
@@
 </segment>
 <segment>
-<pinref part="U1" gate="G$1" pin="CHAN4"/>
-<wire x1="363.22" y1="-15.24" x2="358.14" y2="-15.24" width="0.1524" layer="91"/>
-<label x="358.14" y="-15.24" size="1.778" layer="95" rot="R180" xref="yes"/>
+<pinref part="U1" gate="G$1" pin="CHAN3"/>
+<wire x1="363.22" y1="-12.7" x2="350.52" y2="-12.7" width="0.1524" layer="91"/>
+<label x="350.52" y="-12.7" size="1.778" layer="95" rot="R180" xref="yes"/>
 </segment>
 </net>
@@
 </segment>
 <segment>
-<pinref part="U1" gate="G$1" pin="CHAN5"/>
-<wire x1="363.22" y1="-17.78" x2="350.52" y2="-17.78" width="0.1524" layer="91"/>
-<label x="350.52" y="-17.78" size="1.778" layer="95" rot="R180" xref="yes"/>
+<pinref part="U1" gate="G$1" pin="CHAN4"/>
+<wire x1="363.22" y1="-15.24" x2="358.14" y2="-15.24" width="0.1524" layer="91"/>
+<label x="358.14" y="-15.24" size="1.778" layer="95" rot="R180" xref="yes"/>
 </segment>
 </net>
@@
 </segment>
 <segment>
-<pinref part="U1" gate="G$1" pin="CHAN6"/>
-<wire x1="363.22" y1="-20.32" x2="358.14" y2="-20.32" width="0.1524" layer="91"/>
-<label x="358.14" y="-20.32" size="1.778" layer="95" rot="R180" xref="yes"/>
+<pinref part="U1" gate="G$1" pin="CHAN5"/>
+<wire x1="363.22" y1="-17.78" x2="350.52" y2="-17.78" width="0.1524" layer="91"/>
+<label x="350.52" y="-17.78" size="1.778" layer="95" rot="R180" xref="yes"/>
 </segment>
 </net>
@@
 </segment>
 <segment>
-<pinref part="U1" gate="G$1" pin="CHAN7"/>
-<wire x1="363.22" y1="-22.86" x2="350.52" y2="-22.86" width="0.1524" layer="91"/>
-<label x="350.52" y="-22.86" size="1.778" layer="95" rot="R180" xref="yes"/>
+<pinref part="U1" gate="G$1" pin="CHAN6"/>
+<wire x1="363.22" y1="-20.32" x2="358.14" y2="-20.32" width="0.1524" layer="91"/>
+<label x="358.14" y="-20.32" size="1.778" layer="95" rot="R180" xref="yes"/>
 </segment>
 </net>
@@
 </segment>
 <segment>
-<pinref part="U1" gate="G$1" pin="CHAN8"/>
-<wire x1="363.22" y1="-25.4" x2="358.14" y2="-25.4" width="0.1524" layer="91"/>
-<label x="358.14" y="-25.4" size="1.778" layer="95" rot="R180" xref="yes"/>
+<pinref part="U1" gate="G$1" pin="CHAN7"/>
+<wire x1="363.22" y1="-22.86" x2="350.52" y2="-22.86" width="0.1524" layer="91"/>
+<label x="350.52" y="-22.86" size="1.778" layer="95" rot="R180" xref="yes"/>
 </segment>
 </net>
@@
 <junction x="274.32" y="-2.54"/>
 </segment>
+<segment>
+<pinref part="U1" gate="G$1" pin="CHAN8"/>
+<wire x1="363.22" y1="-25.4" x2="358.14" y2="-25.4" width="0.1524" layer="91"/>
+<label x="358.14" y="-25.4" size="1.778" layer="95" rot="R180" xref="yes"/>
+</segment>
 </net>
 <net name="A26" class="0">
@@
 <junction x="284.48" y="-2.54"/>
 </segment>
+<segment>
+<pinref part="U1" gate="G$1" pin="CHAN9"/>
+<wire x1="363.22" y1="-27.94" x2="350.52" y2="-27.94" width="0.1524" layer="91"/>
+<label x="350.52" y="-27.94" size="1.778" layer="95" rot="R180" xref="yes"/>
+</segment>
 </net>
 <net name="A27" class="0">
@@
 <junction x="294.64" y="-2.54"/>
 </segment>
+<segment>
+<pinref part="U1" gate="G$1" pin="CHAN10"/>
+<wire x1="363.22" y1="-30.48" x2="358.14" y2="-30.48" width="0.1524" layer="91"/>
+<label x="358.14" y="-30.48" size="1.778" layer="95" rot="R180" xref="yes"/>
+</segment>
 </net>
 <net name="A28" class="0">
@@
 <junction x="304.8" y="-2.54"/>
 </segment>
+<segment>
+<pinref part="U1" gate="G$1" pin="CHAN11"/>
+<wire x1="363.22" y1="-33.02" x2="350.52" y2="-33.02" width="0.1524" layer="91"/>
+<label x="350.52" y="-33.02" size="1.778" layer="95" rot="R180" xref="yes"/>
+</segment>
 </net>
 <net name="A29" class="0">
@@
 <junction x="314.96" y="-2.54"/>
 </segment>
+<segment>
+<pinref part="U1" gate="G$1" pin="CHAN12"/>
+<wire x1="363.22" y1="-35.56" x2="358.14" y2="-35.56" width="0.1524" layer="91"/>
+<label x="358.14" y="-35.56" size="1.778" layer="95" rot="R180" xref="yes"/>
+</segment>
 </net>
 <net name="A30" class="0">
@@
 <wire x1="330.2" y1="-2.54" x2="325.12" y2="-2.54" width="0.1524" layer="91"/>
 <junction x="325.12" y="-2.54"/>
+</segment>
+<segment>
+<pinref part="U1" gate="G$1" pin="CHAN13"/>
+<wire x1="363.22" y1="-38.1" x2="350.52" y2="-38.1" width="0.1524" layer="91"/>
+<label x="350.52" y="-38.1" size="1.778" layer="95" rot="R180" xref="yes"/>
 </segment>
 </net>
@@
 <segment>
 <pinref part="U1" gate="G$1" pin="S0"/>
-<wire x1="388.62" y1="-20.32" x2="441.96" y2="-20.32" width="0.1524" layer="91"/>
+<wire x1="388.62" y1="-20.32" x2="457.2" y2="-20.32" width="0.1524" layer="91"/>
 </segment>
 </net>
@@
 <segment>
 <pinref part="U1" gate="G$1" pin="S1"/>
-<wire x1="388.62" y1="-22.86" x2="439.42" y2="-22.86" width="0.1524" layer="91"/>
+<wire x1="388.62" y1="-22.86" x2="457.2" y2="-22.86" width="0.1524" layer="91"/>
 </segment>
 </net>
@@
 <segment>
 <pinref part="U1" gate="G$1" pin="S2"/>
-<wire x1="388.62" y1="-25.4" x2="436.88" y2="-25.4" width="0.1524" layer="91"/>
+<wire x1="388.62" y1="-25.4" x2="457.2" y2="-25.4" width="0.1524" layer="91"/>
+<wire x1="457.2" y1="-25.4" x2="457.2" y2="-40.64" width="0.1524" layer="91"/>
+<pinref part="SV1" gate="1" pin="2"/>
+<wire x1="457.2" y1="-40.64" x2="454.66" y2="-40.64" width="0.1524" layer="91"/>
 </segment>
 </net>
@@
 <pinref part="U1" gate="G$1" pin="COM"/>
 <wire x1="388.62" y1="-33.02" x2="431.8" y2="-33.02" width="0.1524" layer="91"/>
-</segment>
-</net>
+<pinref part="SV1" gate="1" pin="1"/>
+<wire x1="431.8" y1="-33.02" x2="431.8" y2="-40.64" width="0.1524" layer="91"/>
+<wire x1="431.8" y1="-40.64" x2="439.42" y2="-40.64" width="0.1524" layer="91"/>
+</segment>
+</net>

Commit message: Making linesensor
Connections:
- removed net N$5: U1.S0
- removed net N$7: U1.S1
- new net N$15: SV1.5, U1.S1
- new net N$16: SV1.3, U1.S0
- net N$9: now also SV1.4
- net VCC: now also SV1.6
Changed lines of the file:
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@@
 <part name="SV1" library="con-lstb" library_urn="urn:adsk.eagle:library:162" deviceset="MA06-2" device="" package3d_urn="urn:adsk.eagle:package:8342/1"/>
 <part name="GND4" library="supply" deviceset="GND" device=""/>
+<part name="U$4" library="supply" deviceset="VCC" device=""/>
 </parts>
 <sheets>
@@
 <instance part="GND4" gate="1" x="464.82" y="-58.42" smashed="yes">
 <attribute name="VALUE" x="462.534" y="-60.96" size="1.778" layer="96" font="vector"/>
+</instance>
+<instance part="U$4" gate="G$1" x="464.82" y="-35.56" smashed="yes">
+<attribute name="VALUE" x="462.534" y="-34.798" size="1.778" layer="96" font="vector"/>
 </instance>
 </instances>
@@
 <pinref part="U$3" gate="G$1" pin="VCC"/>
 </segment>
+<segment>
+<pinref part="SV1" gate="1" pin="6"/>
+<wire x1="454.66" y1="-45.72" x2="464.82" y2="-45.72" width="0.1524" layer="91"/>
+<wire x1="464.82" y1="-45.72" x2="464.82" y2="-38.1" width="0.1524" layer="91"/>
+<pinref part="U$4" gate="G$1" pin="VCC"/>
+</segment>
 </net>
 <net name="A6" class="0">
@@
 </segment>
 </net>
-<net name="N$5" class="0">
-<segment>
-<pinref part="U1" gate="G$1" pin="S0"/>
-<wire x1="388.62" y1="-20.32" x2="457.2" y2="-20.32" width="0.1524" layer="91"/>
-</segment>
-</net>
-<net name="N$7" class="0">
-<segment>
-<pinref part="U1" gate="G$1" pin="S1"/>
-<wire x1="388.62" y1="-22.86" x2="457.2" y2="-22.86" width="0.1524" layer="91"/>
-</segment>
-</net>
 <net name="N$8" class="0">
 <segment>
@@
 <segment>
 <pinref part="U1" gate="G$1" pin="S3"/>
-<wire x1="388.62" y1="-27.94" x2="434.34" y2="-27.94" width="0.1524" layer="91"/>
+<wire x1="388.62" y1="-27.94" x2="459.74" y2="-27.94" width="0.1524" layer="91"/>
+<pinref part="SV1" gate="1" pin="4"/>
+<wire x1="459.74" y1="-27.94" x2="459.74" y2="-43.18" width="0.1524" layer="91"/>
+<wire x1="459.74" y1="-43.18" x2="454.66" y2="-43.18" width="0.1524" layer="91"/>
 </segment>
 </net>
@@
 </segment>
 </net>
+<net name="N$15" class="0">
+<segment>
+<pinref part="SV1" gate="1" pin="5"/>
+<wire x1="439.42" y1="-45.72" x2="434.34" y2="-45.72" width="0.1524" layer="91"/>
+<pinref part="U1" gate="G$1" pin="S1"/>
+<wire x1="388.62" y1="-22.86" x2="434.34" y2="-22.86" width="0.1524" layer="91"/>
+<wire x1="434.34" y1="-45.72" x2="434.34" y2="-22.86" width="0.1524" layer="91"/>
+</segment>
+</net>
+<net name="N$16" class="0">
+<segment>
+<pinref part="SV1" gate="1" pin="3"/>
+<wire x1="439.42" y1="-43.18" x2="436.88" y2="-43.18" width="0.1524" layer="91"/>
+<pinref part="U1" gate="G$1" pin="S0"/>
+<wire x1="388.62" y1="-20.32" x2="436.88" y2="-20.32" width="0.1524" layer="91"/>
+<wire x1="436.88" y1="-43.18" x2="436.88" y2="-20.32" width="0.1524" layer="91"/>
+</segment>
+</net>

Commit message: encorder & linesensor
Parts:
- removed SV1: (no value), con-lstb:MA06-2
- added SV2: (no value), con-lstb:MA07-2
Connections:
- removed net N$60: LED1.DI
- new net LED_IN: LED1.DI, SV2.7
- new net LED_OUT: LED30.DO, SV2.8
- net AIN0: now also SV2.14; no longer SV1.1
- net AIN1: now also SV2.2; no longer SV1.11
- net GND: now also SV2.5; no longer SV1.8
- net N$10: now also SV2.6; no longer SV1.7
- net N$11: now also SV2.4; no longer SV1.9
- net N$13: now also SV2.3; no longer SV1.10
- net N$14: now also SV2.1; no longer SV1.12
- net N$15: now also SV2.10; no longer SV1.5
- net N$16: now also SV2.12; no longer SV1.3
- net N$8: now also SV2.13; no longer SV1.2
- net N$9: now also SV2.11; no longer SV1.4
- net VCC: now also SV2.9; no longer SV1.6
Changed lines of the file:
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@@
 <part name="GND3" library="supply" deviceset="GND" device=""/>
 <part name="GND1" library="supply" deviceset="GND" device=""/>
-<part name="SV1" library="con-lstb" library_urn="urn:adsk.eagle:library:162" deviceset="MA06-2" device="" package3d_urn="urn:adsk.eagle:package:8342/1"/>
 <part name="GND4" library="supply" deviceset="GND" device=""/>
 <part name="U$4" library="supply" deviceset="VCC" device=""/>
+<part name="SV2" library="con-lstb" library_urn="urn:adsk.eagle:library:162" deviceset="MA07-2" device="" package3d_urn="urn:adsk.eagle:package:8330/1"/>
 </parts>
 <sheets>
@@
 <attribute name="VALUE" x="23.114" y="-25.4" size="1.778" layer="96" font="vector"/>
 </instance>
-<instance part="SV1" gate="1" x="447.04" y="-48.26" smashed="yes" rot="R180">
-<attribute name="VALUE" x="450.85" y="-35.56" size="1.778" layer="96" rot="R180"/>
-<attribute name="NAME" x="450.85" y="-56.642" size="1.778" layer="95" rot="R180"/>
-</instance>
 <instance part="GND4" gate="1" x="464.82" y="-58.42" smashed="yes">
 <attribute name="VALUE" x="462.534" y="-60.96" size="1.778" layer="96" font="vector"/>
@@
 <instance part="U$4" gate="G$1" x="464.82" y="-35.56" smashed="yes">
 <attribute name="VALUE" x="462.534" y="-34.798" size="1.778" layer="96" font="vector"/>
+</instance>
+<instance part="SV2" gate="G$1" x="447.04" y="-45.72" smashed="yes">
+<attribute name="VALUE" x="443.23" y="-58.42" size="1.778" layer="96"/>
+<attribute name="NAME" x="443.23" y="-34.798" size="1.778" layer="95"/>
 </instance>
 </instances>
@@
 </segment>
 <segment>
-<pinref part="SV1" gate="1" pin="6"/>
-<wire x1="454.66" y1="-45.72" x2="464.82" y2="-45.72" width="0.1524" layer="91"/>
-<wire x1="464.82" y1="-45.72" x2="464.82" y2="-38.1" width="0.1524" layer="91"/>
 <pinref part="U$4" gate="G$1" pin="VCC"/>
+<pinref part="SV2" gate="G$1" pin="9"/>
+<wire x1="464.82" y1="-43.18" x2="464.82" y2="-38.1" width="0.1524" layer="91"/>
+<wire x1="454.66" y1="-43.18" x2="464.82" y2="-43.18" width="0.1524" layer="91"/>
 </segment>
 </net>
@@
 </segment>
 <segment>
-<pinref part="SV1" gate="1" pin="8"/>
 <wire x1="454.66" y1="-48.26" x2="464.82" y2="-48.26" width="0.1524" layer="91"/>
 <wire x1="464.82" y1="-48.26" x2="464.82" y2="-55.88" width="0.1524" layer="91"/>
 <pinref part="GND4" gate="1" pin="GND"/>
+<pinref part="SV2" gate="G$1" pin="5"/>
 </segment>
 </net>
@@
 </segment>
 </net>
-<net name="N$60" class="0">
-<segment>
-<pinref part="LED1" gate="G$1" pin="DI"/>
-<wire x1="7.62" y1="63.5" x2="-2.54" y2="63.5" width="0.1524" layer="91"/>
-</segment>
-</net>
 <net name="N$8" class="0">
 <segment>
 <pinref part="U1" gate="G$1" pin="S2"/>
 <wire x1="388.62" y1="-25.4" x2="457.2" y2="-25.4" width="0.1524" layer="91"/>
-<wire x1="457.2" y1="-25.4" x2="457.2" y2="-40.64" width="0.1524" layer="91"/>
-<pinref part="SV1" gate="1" pin="2"/>
-<wire x1="457.2" y1="-40.64" x2="454.66" y2="-40.64" width="0.1524" layer="91"/>
+<wire x1="457.2" y1="-25.4" x2="457.2" y2="-38.1" width="0.1524" layer="91"/>
+<pinref part="SV2" gate="G$1" pin="13"/>
+<wire x1="454.66" y1="-38.1" x2="457.2" y2="-38.1" width="0.1524" layer="91"/>
 </segment>
 </net>
@@
 <pinref part="U1" gate="G$1" pin="S3"/>
 <wire x1="388.62" y1="-27.94" x2="459.74" y2="-27.94" width="0.1524" layer="91"/>
-<pinref part="SV1" gate="1" pin="4"/>
-<wire x1="459.74" y1="-27.94" x2="459.74" y2="-43.18" width="0.1524" layer="91"/>
-<wire x1="459.74" y1="-43.18" x2="454.66" y2="-43.18" width="0.1524" layer="91"/>
+<wire x1="459.74" y1="-27.94" x2="459.74" y2="-40.64" width="0.1524" layer="91"/>
+<pinref part="SV2" gate="G$1" pin="11"/>
+<wire x1="454.66" y1="-40.64" x2="459.74" y2="-40.64" width="0.1524" layer="91"/>
 </segment>
 </net>
@@
 <pinref part="U2" gate="G$1" pin="COM"/>
 <wire x1="388.62" y1="-83.82" x2="431.8" y2="-83.82" width="0.1524" layer="91"/>
-<pinref part="SV1" gate="1" pin="11"/>
 <wire x1="431.8" y1="-83.82" x2="431.8" y2="-53.34" width="0.1524" layer="91"/>
 <wire x1="431.8" y1="-53.34" x2="439.42" y2="-53.34" width="0.1524" layer="91"/>
+<pinref part="SV2" gate="G$1" pin="2"/>
 </segment>
 </net>
@@
 <pinref part="U1" gate="G$1" pin="COM"/>
 <wire x1="388.62" y1="-33.02" x2="431.8" y2="-33.02" width="0.1524" layer="91"/>
-<pinref part="SV1" gate="1" pin="1"/>
-<wire x1="431.8" y1="-33.02" x2="431.8" y2="-40.64" width="0.1524" layer="91"/>
-<wire x1="431.8" y1="-40.64" x2="439.42" y2="-40.64" width="0.1524" layer="91"/>
+<wire x1="431.8" y1="-33.02" x2="431.8" y2="-38.1" width="0.1524" layer="91"/>
+<pinref part="SV2" gate="G$1" pin="14"/>
+<wire x1="439.42" y1="-38.1" x2="431.8" y2="-38.1" width="0.1524" layer="91"/>
 </segment>
 </net>
@@
 <pinref part="U2" gate="G$1" pin="S3"/>
 <wire x1="388.62" y1="-78.74" x2="434.34" y2="-78.74" width="0.1524" layer="91"/>
-<pinref part="SV1" gate="1" pin="7"/>
 <wire x1="439.42" y1="-48.26" x2="434.34" y2="-48.26" width="0.1524" layer="91"/>
 <wire x1="434.34" y1="-48.26" x2="434.34" y2="-78.74" width="0.1524" layer="91"/>
+<pinref part="SV2" gate="G$1" pin="6"/>
 </segment>
 </net>
@@
 <pinref part="U2" gate="G$1" pin="S2"/>
 <wire x1="388.62" y1="-76.2" x2="436.88" y2="-76.2" width="0.1524" layer="91"/>
-<pinref part="SV1" gate="1" pin="9"/>
 <wire x1="439.42" y1="-50.8" x2="436.88" y2="-50.8" width="0.1524" layer="91"/>
 <wire x1="436.88" y1="-50.8" x2="436.88" y2="-76.2" width="0.1524" layer="91"/>
+<pinref part="SV2" gate="G$1" pin="4"/>
 </segment>
 </net>
@@
 <pinref part="U2" gate="G$1" pin="S1"/>
 <wire x1="388.62" y1="-73.66" x2="459.74" y2="-73.66" width="0.1524" layer="91"/>
-<pinref part="SV1" gate="1" pin="10"/>
 <wire x1="454.66" y1="-50.8" x2="459.74" y2="-50.8" width="0.1524" layer="91"/>
 <wire x1="459.74" y1="-50.8" x2="459.74" y2="-73.66" width="0.1524" layer="91"/>
+<pinref part="SV2" gate="G$1" pin="3"/>
 </segment>
 </net>
@@
 <wire x1="388.62" y1="-71.12" x2="457.2" y2="-71.12" width="0.1524" layer="91"/>
 <wire x1="457.2" y1="-71.12" x2="457.2" y2="-53.34" width="0.1524" layer="91"/>
-<pinref part="SV1" gate="1" pin="12"/>
 <wire x1="457.2" y1="-53.34" x2="454.66" y2="-53.34" width="0.1524" layer="91"/>
+<pinref part="SV2" gate="G$1" pin="1"/>
 </segment>
 </net>
 <net name="N$15" class="0">
 <segment>
-<pinref part="SV1" gate="1" pin="5"/>
-<wire x1="439.42" y1="-45.72" x2="434.34" y2="-45.72" width="0.1524" layer="91"/>
 <pinref part="U1" gate="G$1" pin="S1"/>
 <wire x1="388.62" y1="-22.86" x2="434.34" y2="-22.86" width="0.1524" layer="91"/>
-<wire x1="434.34" y1="-45.72" x2="434.34" y2="-22.86" width="0.1524" layer="91"/>
+<pinref part="SV2" gate="G$1" pin="10"/>
+<wire x1="434.34" y1="-43.18" x2="434.34" y2="-22.86" width="0.1524" layer="91"/>
+<wire x1="439.42" y1="-43.18" x2="434.34" y2="-43.18" width="0.1524" layer="91"/>
 </segment>
 </net>
 <net name="N$16" class="0">
 <segment>
-<pinref part="SV1" gate="1" pin="3"/>
-<wire x1="439.42" y1="-43.18" x2="436.88" y2="-43.18" width="0.1524" layer="91"/>
 <pinref part="U1" gate="G$1" pin="S0"/>
 <wire x1="388.62" y1="-20.32" x2="436.88" y2="-20.32" width="0.1524" layer="91"/>
-<wire x1="436.88" y1="-43.18" x2="436.88" y2="-20.32" width="0.1524" layer="91"/>
-</segment>
-</net>
+<pinref part="SV2" gate="G$1" pin="12"/>
+<wire x1="436.88" y1="-40.64" x2="436.88" y2="-20.32" width="0.1524" layer="91"/>
+<wire x1="439.42" y1="-40.64" x2="436.88" y2="-40.64" width="0.1524" layer="91"/>
+</segment>
+</net>
+<net name="LED_IN" class="0">
+<segment>
+<pinref part="SV2" gate="G$1" pin="7"/>
+<wire x1="454.66" y1="-45.72" x2="457.2" y2="-45.72" width="0.1524" layer="91"/>
+<label x="457.2" y="-45.72" size="1.778" layer="95" xref="yes"/>
+</segment>
+<segment>
+<pinref part="LED1" gate="G$1" pin="DI"/>
+<wire x1="7.62" y1="63.5" x2="-2.54" y2="63.5" width="0.1524" layer="91"/>
+<label x="-2.54" y="63.5" size="1.778" layer="95" rot="R180" xref="yes"/>
+</segment>
+</net>
+<net name="LED_OUT" class="0">
+<segment>
+<pinref part="LED30" gate="G$1" pin="DO"/>
+<wire x1="769.62" y1="63.5" x2="777.24" y2="63.5" width="0.1524" layer="91"/>
+<label x="777.24" y="63.5" size="1.778" layer="95" xref="yes"/>
+</segment>
+<segment>
+<pinref part="SV2" gate="G$1" pin="8"/>
+<wire x1="439.42" y1="-45.72" x2="434.34" y2="-45.72" width="0.1524" layer="91"/>
+<label x="434.34" y="-45.72" size="1.778" layer="95" rot="R180" xref="yes"/>
+</segment>
+</net>
