File: board/power_supply/untitled.brd (EAGLE design)
At the start: 160 x 100 mm, 24 parts, among them IC1 317EMP, Q1 FDD4141TO252

Commit message: update 7/2
Parts:
- moved MD5 185.1 mm to (34.3, 41.9)
- moved MD4 183.0 mm to (34.3, 48.3)
- moved R2 178.7 mm to (31.8, 13.2)
- moved C3 167.7 mm to (21.6, 11.7)
- moved R6 165.6 mm to (35.6, 34.3)
- moved C4 159.7 mm to (25.1, 2.41)
- moved R4 157.6 mm to (54.6, 22.9), turned to 90 degrees
- moved IC1 155.4 mm to (21.6, 6.35), turned to 180 degrees
- moved U$4 151.8 mm to (47.0, 22.9)
- moved C2 146.5 mm to (43.2, 3.81)
- moved C1 138.3 mm to (50.7, 1.27), turned to 180 degrees
- moved R3 136.9 mm to (50.7, 3.68)
- moved MD3 130.9 mm to (49.4, 12.6), turned to 180 degrees
- moved KICK 127.9 mm to (82.5, 5.08)
- moved MD1 127.9 mm to (82.5, 22.9)
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Routing:
- net N$11: track 0.00 -> 11.2 mm, vias 0 -> 1
- net GND: track 0.00 -> 10.0 mm
- net VCC: track 0.00 -> 9.75 mm
- net N$3: track 0.00 -> 9.42 mm

Commit message: update powerboard
Parts:
- removed MD4, MD5: JST-XH-02-PIN-LONG-PAD, Rembrandt Electronics - JST XH Connectors v1-0:JST-XH-02-PACKAGE-LONG-PAD
- added MAIN, RASPI: JST-XH-02-PIN-LONG-PAD, Rembrandt Electronics - JST XH Connectors v1-0:JST-XH-02-PACKAGE-LONG-PAD
- added R5, R7: 10k, adafruit:M2012
- moved R4 46.9 mm to (8.26, 30.2), turned to 0 degrees
- moved U$4 41.3 mm to (8.13, 36.7), turned to 270 degrees
- moved C1 40.0 mm to (21.0, 28.1)
- moved R3 39.8 mm to (21.0, 30.2)
- moved C2 38.2 mm to (13.6, 27.9)
- moved MD3 37.9 mm to (21.2, 37.8)
- moved KICK 36.5 mm to (46.1, 6.35), turned to 270 degrees
- moved MD1 36.5 mm to (46.1, 22.1), turned to 270 degrees
- moved MD2 36.4 mm to (46.1, 14.2), turned to 270 degrees
- moved R6 22.9 mm to (12.7, 35.6), turned to 270 degrees
- moved U$1 9.76 mm to (35.9, 13.5), turned to 0 degrees
- moved U$3 3.81 mm to (35.6, 6.35)
- moved R2 0.25 mm to (31.8, 13.5), turned to 180 degrees
Connections:
- new net N$10: R7.2, U$3.7
- net GND: now also MAIN.1, RASPI.1; no longer MD4.1, MD5.1
- net N$11: now also R5.1
- net N$2: now also R5.2, R7.1; no longer U$3.7
- net N$8: now also MAIN.2, RASPI.2; no longer MD4.2, MD5.2
Routing:
- net GND: track 10.0 -> 294.6 mm, vias 0 -> 5
- net N$8: track 0.00 -> 60.2 mm, vias 0 -> 1
- net VCC: track 9.75 -> 66.4 mm, vias 0 -> 2
- net N$5: track 0.00 -> 50.8 mm, vias 0 -> 1
- net N$2: track 0.00 -> 20.3 mm
- net N$11: track 11.2 -> 31.4 mm, vias 1 -> 2
- net N$9: track 0.00 -> 10.9 mm
- net N$3: track 9.42 -> 19.0 mm
- net N$4: track 0.00 -> 9.28 mm
- net N$1: track 0.00 -> 8.03 mm
- net N$7: track 0.00 -> 6.92 mm
- net N$10: track 0.00 -> 2.35 mm
Other:
- board size 160 x 100 mm -> 52 x 46.7 mm
