File: board/power_supply/untitled.sch (EAGLE design)
At the start: 3 parts

Commit message: update7/2
Parts:
- added C1, C2: (no value), adafruit:C-USC2012
- added C3, C4: (no value), generic:CAPACITOR1608
- added IC1: 317EMP, linear:317EMP
- added KICK, MD1, MD2, MD4, MD5: JST-XH-02-PIN-LONG-PAD, Rembrandt Electronics - JST XH Connectors v1-0:JST-XH-02-PIN-LONG-PAD
- added MD3: OKL-T/6-W12P-CMURATA_OKL-T-6-W12P-C_0_0, OKL-T_6-W12P-C:OKL-T/6-W12P-CMURATA_OKL-T-6-W12P-C_0_0
- added PAD1: (no value), wirepad:3,81/1,4
- added Q1: FDD4141TO252, transistor-fet:FDD4141TO252
- added R1, R2, R3, R4: (no value), adafruit:R-US_M2012
- added R6: (no value), adafruit:FLIPFLOP-RES
- added U$2: SMD-R-TRIM, by_hirame:SMD-R-TRIM
- added U$3: ATTINY85, attiny85:ATTINY85
- added U$4: R-TRIM, by_hirame:R-TRIM
Connections:
- new net N$1: R1.2, U$1.VDD, U$2.3
- new net N$11: C4.2, IC1.VO, R2.2, U$3.VCC
- new net N$2: Q1.G, U$3.2
- new net N$4: R2.1, U$1.OUT, U$3.1
- new net N$5: KICK-2.S, MD1-2.S, MD2-2.S, Q1.D
- new net N$6: U$3.4
- new net N$7: R4.2, U$4.2, U$4.3
- new net N$8: C2.1, MD3.SENSE, MD3.VOUT, MD4-2.S, MD5-2.S, R6.2
- new net N$9: MD3.TRIM, U$4.1
- net GND: now also C1.2, C2.2, C3.2, C4.1, IC1.ADJ, KICK-1.S, MD1-1.S, MD2-1.S, MD3.1_GROUND, MD3.2_GROUND, MD3.ON/OFF_CONTROL, MD4-1.S, MD5-1.S, PAD1.P, R1.1, R3.1, R4.1, R6.1, U$3.GND
- net N$3: now also PAD3.P; no longer U$1.VDD
- net VCC: now also C1.1, C3.1, IC1.VI, MD3.VIN, Q1.S, R3.2, U$2.2
Other:
- note added: "buzzer"
- moved on the sheet: F1, PAD3

Commit message: update 7/2
Connections:
- net N$7: now also U$4.P$1; no longer U$4.3
Changed lines of the file:
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@@
 <?xml version="1.0" encoding="utf-8"?>
 <!DOCTYPE eagle SYSTEM "eagle.dtd">
-<eagle version="9.6.1">
+<eagle version="9.6.2">
 <drawing>
 <settings>
@@
 <part name="C1" library="adafruit" deviceset="C-US" device="C2012"/>
 <part name="R4" library="adafruit" deviceset="R-US_" device="M2012"/>
-<part name="U$4" library="by_hirame" deviceset="R-TRIM" device=""/>
 <part name="C2" library="adafruit" deviceset="C-US" device="C2012"/>
 <part name="R6" library="adafruit" deviceset="FLIPFLOP-RES" device=""/>
@@
 <part name="GND5" library="supply1" library_urn="urn:adsk.eagle:library:371" deviceset="GND" device=""/>
 <part name="R2" library="adafruit" deviceset="R-US_" device="M2012"/>
+<part name="U$4" library="by_hirame" deviceset="R-TRIM" device=""/>
 </parts>
 <sheets>
@@
 <attribute name="VALUE" x="51.562" y="-87.63" size="1.778" layer="96" rot="R90"/>
 </instance>
+<instance part="C2" gate="G$1" x="58.42" y="-68.58" smashed="yes">
+<attribute name="NAME" x="59.436" y="-67.945" size="1.778" layer="95"/>
+<attribute name="VALUE" x="59.436" y="-72.771" size="1.778" layer="96"/>
+</instance>
+<instance part="R6" gate="G$1" x="68.58" y="-71.12" smashed="yes" rot="R90">
+<attribute name="NAME" x="67.0814" y="-74.93" size="1.778" layer="95" rot="R90"/>
+<attribute name="VALUE" x="71.882" y="-74.93" size="1.778" layer="96" rot="R90"/>
+</instance>
+<instance part="MD4" gate="-2" x="78.74" y="-55.88" smashed="yes">
+<attribute name="NAME" x="81.28" y="-56.642" size="1.524" layer="95"/>
+</instance>
+<instance part="MD4" gate="-1" x="78.74" y="-53.34" smashed="yes">
+<attribute name="NAME" x="81.28" y="-54.102" size="1.524" layer="95"/>
+<attribute name="VALUE" x="77.978" y="-51.943" size="1.778" layer="96"/>
+</instance>
+<instance part="GND3" gate="1" x="-27.94" y="-93.98" smashed="yes">
+<attribute name="VALUE" x="-30.48" y="-96.52" size="1.778" layer="96"/>
+</instance>
+<instance part="MD5" gate="-2" x="78.74" y="-63.5" smashed="yes">
+<attribute name="NAME" x="81.28" y="-64.262" size="1.524" layer="95"/>
+</instance>
+<instance part="MD5" gate="-1" x="78.74" y="-60.96" smashed="yes">
+<attribute name="NAME" x="81.28" y="-61.722" size="1.524" layer="95"/>
+<attribute name="VALUE" x="77.978" y="-59.563" size="1.778" layer="96"/>
+</instance>
+<instance part="IC1" gate="A1" x="7.62" y="43.18" smashed="yes" rot="MR0">
+<attribute name="NAME" x="15.24" y="51.435" size="1.778" layer="95" rot="MR0"/>
+<attribute name="VALUE" x="15.24" y="48.895" size="1.778" layer="96" rot="MR0"/>
+</instance>
+<instance part="C3" gate="G$1" x="17.78" y="43.18" smashed="yes">
+<attribute name="NAME" x="18.288" y="43.434" size="1.778" layer="95" font="vector"/>
+<attribute name="VALUE" x="18.288" y="41.656" size="1.778" layer="96" font="vector" rot="MR180"/>
+</instance>
+<instance part="C4" gate="G$1" x="0" y="38.1" smashed="yes" rot="R270">
+<attribute name="NAME" x="0.254" y="37.592" size="1.778" layer="95" font="vector" rot="R270"/>
+<attribute name="VALUE" x="-1.524" y="37.592" size="1.778" layer="96" font="vector" rot="MR270"/>
+</instance>
+<instance part="GND4" gate="1" x="-7.62" y="30.48" smashed="yes">
+<attribute name="VALUE" x="-10.16" y="27.94" size="1.778" layer="96"/>
+</instance>
+<instance part="GND5" gate="1" x="-30.48" y="-10.16" smashed="yes">
+<attribute name="VALUE" x="-33.02" y="-12.7" size="1.778" layer="96"/>
+</instance>
+<instance part="R2" gate="G$1" x="5.08" y="7.62" smashed="yes" rot="R90">
+<attribute name="NAME" x="3.5814" y="3.81" size="1.778" layer="95" rot="R90"/>
+<attribute name="VALUE" x="8.382" y="3.81" size="1.778" layer="96" rot="R90"/>
+</instance>
 <instance part="U$4" gate="G$1" x="48.26" y="-73.66" smashed="yes" rot="R270">
 <attribute name="NAME" x="49.7586" y="-69.85" size="1.778" layer="95" rot="R270"/>
 <attribute name="VALUE" x="44.958" y="-69.85" size="1.778" layer="96" rot="R270"/>
-</instance>
-<instance part="C2" gate="G$1" x="58.42" y="-68.58" smashed="yes">
-<attribute name="NAME" x="59.436" y="-67.945" size="1.778" layer="95"/>
-<attribute name="VALUE" x="59.436" y="-72.771" size="1.778" layer="96"/>
-</instance>
-<instance part="R6" gate="G$1" x="68.58" y="-71.12" smashed="yes" rot="R90">
-<attribute name="NAME" x="67.0814" y="-74.93" size="1.778" layer="95" rot="R90"/>
-<attribute name="VALUE" x="71.882" y="-74.93" size="1.778" layer="96" rot="R90"/>
-</instance>
-<instance part="MD4" gate="-2" x="78.74" y="-55.88" smashed="yes">
-<attribute name="NAME" x="81.28" y="-56.642" size="1.524" layer="95"/>
-</instance>
-<instance part="MD4" gate="-1" x="78.74" y="-53.34" smashed="yes">
-<attribute name="NAME" x="81.28" y="-54.102" size="1.524" layer="95"/>
-<attribute name="VALUE" x="77.978" y="-51.943" size="1.778" layer="96"/>
-</instance>
-<instance part="GND3" gate="1" x="-27.94" y="-93.98" smashed="yes">
-<attribute name="VALUE" x="-30.48" y="-96.52" size="1.778" layer="96"/>
-</instance>
-<instance part="MD5" gate="-2" x="78.74" y="-63.5" smashed="yes">
-<attribute name="NAME" x="81.28" y="-64.262" size="1.524" layer="95"/>
-</instance>
-<instance part="MD5" gate="-1" x="78.74" y="-60.96" smashed="yes">
-<attribute name="NAME" x="81.28" y="-61.722" size="1.524" layer="95"/>
-<attribute name="VALUE" x="77.978" y="-59.563" size="1.778" layer="96"/>
-</instance>
-<instance part="IC1" gate="A1" x="7.62" y="43.18" smashed="yes" rot="MR0">
-<attribute name="NAME" x="15.24" y="51.435" size="1.778" layer="95" rot="MR0"/>
-<attribute name="VALUE" x="15.24" y="48.895" size="1.778" layer="96" rot="MR0"/>
-</instance>
-<instance part="C3" gate="G$1" x="17.78" y="43.18" smashed="yes">
-<attribute name="NAME" x="18.288" y="43.434" size="1.778" layer="95" font="vector"/>
-<attribute name="VALUE" x="18.288" y="41.656" size="1.778" layer="96" font="vector" rot="MR180"/>
-</instance>
-<instance part="C4" gate="G$1" x="0" y="38.1" smashed="yes" rot="R270">
-<attribute name="NAME" x="0.254" y="37.592" size="1.778" layer="95" font="vector" rot="R270"/>
-<attribute name="VALUE" x="-1.524" y="37.592" size="1.778" layer="96" font="vector" rot="MR270"/>
-</instance>
-<instance part="GND4" gate="1" x="-7.62" y="30.48" smashed="yes">
-<attribute name="VALUE" x="-10.16" y="27.94" size="1.778" layer="96"/>
-</instance>
-<instance part="GND5" gate="1" x="-30.48" y="-10.16" smashed="yes">
-<attribute name="VALUE" x="-33.02" y="-12.7" size="1.778" layer="96"/>
-</instance>
-<instance part="R2" gate="G$1" x="5.08" y="7.62" smashed="yes" rot="R90">
-<attribute name="NAME" x="3.5814" y="3.81" size="1.778" layer="95" rot="R90"/>
-<attribute name="VALUE" x="8.382" y="3.81" size="1.778" layer="96" rot="R90"/>
 </instance>
 </instances>
@@
 <segment>
 <pinref part="R4" gate="G$1" pin="2"/>
-<pinref part="U$4" gate="G$1" pin="3"/>
+<wire x1="48.26" y1="-78.74" x2="52.832" y2="-78.74" width="0.1524" layer="91"/>
+<pinref part="U$4" gate="G$1" pin="P$1"/>
+<junction x="48.26" y="-78.74"/>
 <pinref part="U$4" gate="G$1" pin="2"/>
-<wire x1="48.26" y1="-78.74" x2="54.61" y2="-78.74" width="0.1524" layer="91"/>
-<wire x1="54.61" y1="-78.74" x2="54.61" y2="-73.66" width="0.1524" layer="91"/>
-<junction x="48.26" y="-78.74"/>
-</segment>
-</net>
+<wire x1="52.832" y1="-73.66" x2="52.832" y2="-78.74" width="0.1524" layer="91"/>
+</segment>
+</net>

Commit message: update powerboard
Parts:
- added R5, R7: 10k, adafruit:R-US_M2012
- renumbered MD4 to MAIN, MD5 to RASPI
Connections:
- new net N$10: R7.2, U$3.2
- net N$11: now also R5.1
- net N$2: now also R5.2, R7.1; no longer U$3.2
Other:
- moved on the sheet: C3, C4, IC1, U$3

Commit message: update power board
Parts:
- added SG1: F/TMB, buzzer:F/TMB
Connections:
- net GND: now also SG1.-
- net N$6: now also SG1.+
Other:
- note removed: "buzzer"
Changed lines of the file:
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@@
 <part name="C4" library="generic" deviceset="CAPACITOR" device="1608"/>
 <part name="GND4" library="supply1" library_urn="urn:adsk.eagle:library:371" deviceset="GND" device=""/>
-<part name="GND5" library="supply1" library_urn="urn:adsk.eagle:library:371" deviceset="GND" device=""/>
 <part name="R2" library="adafruit" deviceset="R-US_" device="M2012"/>
 <part name="U$4" library="by_hirame" deviceset="R-TRIM" device=""/>
 <part name="R5" library="adafruit" deviceset="R-US_" device="M2012" value="10k"/>
 <part name="R7" library="adafruit" deviceset="R-US_" device="M2012" value="10k"/>
+<part name="SG1" library="buzzer" library_urn="urn:adsk.eagle:library:113" deviceset="F/TMB" device="" package3d_urn="urn:adsk.eagle:package:5260/1"/>
+<part name="GND5" library="supply1" library_urn="urn:adsk.eagle:library:371" deviceset="GND" device=""/>
 </parts>
 <sheets>
 <sheet>
 <plain>
-<text x="-68.58" y="0" size="1.778" layer="91">buzzer</text>
 </plain>
 <instances>
@@
 <attribute name="VALUE" x="-25.4" y="27.94" size="1.778" layer="96"/>
 </instance>
-<instance part="GND5" gate="1" x="-45.72" y="-10.16" smashed="yes">
-<attribute name="VALUE" x="-48.26" y="-12.7" size="1.778" layer="96"/>
-</instance>
 <instance part="R2" gate="G$1" x="5.08" y="7.62" smashed="yes" rot="R90">
 <attribute name="NAME" x="3.5814" y="3.81" size="1.778" layer="95" rot="R90"/>
@@
 <attribute name="NAME" x="-6.35" y="3.5814" size="1.778" layer="95" rot="R180"/>
 <attribute name="VALUE" x="-6.35" y="8.382" size="1.778" layer="96" rot="R180"/>
+</instance>
+<instance part="SG1" gate="1" x="-53.34" y="2.54" smashed="yes" rot="MR0">
+<attribute name="NAME" x="-50.8" y="8.89" size="1.778" layer="95" rot="MR0"/>
+<attribute name="VALUE" x="-58.42" y="2.54" size="1.778" layer="96" rot="MR0"/>
+</instance>
+<instance part="GND5" gate="1" x="-63.5" y="-10.16" smashed="yes">
+<attribute name="VALUE" x="-66.04" y="-12.7" size="1.778" layer="96"/>
 </instance>
 </instances>
@@
 </segment>
 <segment>
+<pinref part="SG1" gate="1" pin="-"/>
+<wire x1="-58.42" y1="0" x2="-63.5" y2="0" width="0.1524" layer="91"/>
+<wire x1="-63.5" y1="0" x2="-63.5" y2="-5.08" width="0.1524" layer="91"/>
 <pinref part="U$3" gate="G$1" pin="GND"/>
-<wire x1="-43.18" y1="-5.08" x2="-45.72" y2="-5.08" width="0.1524" layer="91"/>
-<wire x1="-45.72" y1="-5.08" x2="-45.72" y2="-7.62" width="0.1524" layer="91"/>
+<wire x1="-43.18" y1="-5.08" x2="-63.5" y2="-5.08" width="0.1524" layer="91"/>
+<wire x1="-63.5" y1="-5.08" x2="-63.5" y2="-7.62" width="0.1524" layer="91"/>
+<junction x="-63.5" y="-5.08"/>
 <pinref part="GND5" gate="1" pin="GND"/>
 </segment>
@@
 </segment>
 </net>
-<net name="N$6" class="0">
-<segment>
-<pinref part="U$3" gate="G$1" pin="4"/>
-<wire x1="-43.18" y1="0" x2="-53.34" y2="0" width="0.1524" layer="91"/>
-<wire x1="-53.34" y1="0" x2="-53.34" y2="10.16" width="0.1524" layer="91"/>
-<wire x1="-53.34" y1="10.16" x2="-73.66" y2="10.16" width="0.1524" layer="91"/>
-<wire x1="-73.66" y1="10.16" x2="-73.66" y2="-10.16" width="0.1524" layer="91"/>
-<wire x1="-73.66" y1="-10.16" x2="-53.34" y2="-10.16" width="0.1524" layer="91"/>
-<wire x1="-53.34" y1="-10.16" x2="-53.34" y2="0" width="0.1524" layer="91"/>
-<junction x="-53.34" y="0"/>
-<label x="-53.34" y="0" size="1.778" layer="95" rot="R180" xref="yes"/>
-</segment>
-</net>
 <net name="N$10" class="0">
 <segment>
@@
 </segment>
 </net>
+<net name="N$6" class="0">
+<segment>
+<pinref part="U$3" gate="G$1" pin="4"/>
+<pinref part="SG1" gate="1" pin="+"/>
+<wire x1="-43.18" y1="0" x2="-50.8" y2="0" width="0.1524" layer="91"/>
+</segment>
+</net>

Commit message: update boards 2022-07-14
Parts:
- C1: value (none) -> 22uF 25V
- C2: value (none) -> 10uF 10V
- C3, C4: value (none) -> 0.1uF
- R1: value (none) -> 300Ω
- R2: value (none) -> 470kΩ
- R3: value (none) -> 20kΩ
- R4: value (none) -> 1.2kΩ
- R6: value (none) -> 1.2KΩ 1/6W
- R7: value 10k -> 300Ω
- U$2: value SMD-R-TRIM -> 2.2kΩ
- U$4: value R-TRIM -> 20kΩ
Changed lines of the file:
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@@
 <?xml version="1.0" encoding="utf-8"?>
 <!DOCTYPE eagle SYSTEM "eagle.dtd">
-<eagle version="9.6.1">
+<eagle version="9.6.2">
 <drawing>
 <settings>
@@
 <part name="PAD3" library="wirepad" library_urn="urn:adsk.eagle:library:412" deviceset="3,81/1,4" device="" package3d_urn="urn:adsk.eagle:package:30835/1"/>
 <part name="PAD1" library="wirepad" library_urn="urn:adsk.eagle:library:412" deviceset="3,81/1,4" device="" package3d_urn="urn:adsk.eagle:package:30835/1"/>
-<part name="R1" library="adafruit" deviceset="R-US_" device="M2012"/>
-<part name="U$2" library="by_hirame" deviceset="SMD-R-TRIM" device=""/>
+<part name="R1" library="adafruit" deviceset="R-US_" device="M2012" value="300Ω"/>
+<part name="U$2" library="by_hirame" deviceset="SMD-R-TRIM" device="" value="2.2kΩ"/>
 <part name="MD1" library="Rembrandt Electronics - JST XH Connectors v1-0" deviceset="JST-XH-02-PIN" device="-LONG-PAD"/>
 <part name="MD2" library="Rembrandt Electronics - JST XH Connectors v1-0" deviceset="JST-XH-02-PIN" device="-LONG-PAD"/>
@@
 <part name="MD3" library="OKL-T_6-W12P-C" deviceset="OKL-T/6-W12P-C" device="MURATA_OKL-T-6-W12P-C_0_0"/>
 <part name="P+3" library="supply1" library_urn="urn:adsk.eagle:library:371" deviceset="VCC" device=""/>
-<part name="R3" library="adafruit" deviceset="R-US_" device="M2012"/>
-<part name="C1" library="adafruit" deviceset="C-US" device="C2012"/>
-<part name="R4" library="adafruit" deviceset="R-US_" device="M2012"/>
-<part name="C2" library="adafruit" deviceset="C-US" device="C2012"/>
-<part name="R6" library="adafruit" deviceset="FLIPFLOP-RES" device=""/>
+<part name="R3" library="adafruit" deviceset="R-US_" device="M2012" value="20kΩ"/>
+<part name="C1" library="adafruit" deviceset="C-US" device="C2012" value="22uF 25V"/>
+<part name="R4" library="adafruit" deviceset="R-US_" device="M2012" value="1.2kΩ"/>
+<part name="C2" library="adafruit" deviceset="C-US" device="C2012" value="10uF 10V"/>
+<part name="R6" library="adafruit" deviceset="FLIPFLOP-RES" device="" value="1.2KΩ  1/6W"/>
 <part name="MAIN" library="Rembrandt Electronics - JST XH Connectors v1-0" deviceset="JST-XH-02-PIN" device="-LONG-PAD"/>
 <part name="GND3" library="supply1" library_urn="urn:adsk.eagle:library:371" deviceset="GND" device=""/>
 <part name="RASPI" library="Rembrandt Electronics - JST XH Connectors v1-0" deviceset="JST-XH-02-PIN" device="-LONG-PAD"/>
 <part name="IC1" library="linear" library_urn="urn:adsk.eagle:library:262" deviceset="*317" device="EMP" package3d_urn="urn:adsk.eagle:package:28541/2"/>
-<part name="C3" library="generic" deviceset="CAPACITOR" device="1608"/>
-<part name="C4" library="generic" deviceset="CAPACITOR" device="1608"/>
+<part name="C3" library="generic" deviceset="CAPACITOR" device="1608" value="0.1uF"/>
+<part name="C4" library="generic" deviceset="CAPACITOR" device="1608" value="0.1uF"/>
 <part name="GND4" library="supply1" library_urn="urn:adsk.eagle:library:371" deviceset="GND" device=""/>
-<part name="R2" library="adafruit" deviceset="R-US_" device="M2012"/>
-<part name="U$4" library="by_hirame" deviceset="R-TRIM" device=""/>
+<part name="R2" library="adafruit" deviceset="R-US_" device="M2012" value="470kΩ"/>
+<part name="U$4" library="by_hirame" deviceset="R-TRIM" device="" value="20kΩ"/>
 <part name="R5" library="adafruit" deviceset="R-US_" device="M2012" value="10k"/>
-<part name="R7" library="adafruit" deviceset="R-US_" device="M2012" value="10k"/>
+<part name="R7" library="adafruit" deviceset="R-US_" device="M2012" value="300Ω"/>
 <part name="SG1" library="buzzer" library_urn="urn:adsk.eagle:library:113" deviceset="F/TMB" device="" package3d_urn="urn:adsk.eagle:package:5260/1"/>
 <part name="GND5" library="supply1" library_urn="urn:adsk.eagle:library:371" deviceset="GND" device=""/>

Commit message: marge前のファイル
Parts:
- removed C1: 22uF 25V, adafruit:C-USC2012
- removed C2: 10uF 10V, adafruit:C-USC2012
- removed KICK, MAIN, MD2, RASPI: JST-XH-02-PIN-LONG-PAD, Rembrandt Electronics - JST XH Connectors v1-0:JST-XH-02-PIN-LONG-PAD
- removed MD3: OKL-T/6-W12P-CMURATA_OKL-T-6-W12P-C_0_0, OKL-T_6-W12P-C:OKL-T/6-W12P-CMURATA_OKL-T-6-W12P-C_0_0
- removed R3: 20kΩ, adafruit:R-US_M2012
- removed R4: 1.2kΩ, adafruit:R-US_M2012
- removed R6: 1.2KΩ 1/6W, adafruit:FLIPFLOP-RES
- removed SG1: F/TMB, buzzer:F/TMB
- removed U$4: 20kΩ, by_hirame:R-TRIM
- added JP1, JP2, JP3, JP4: (no value), pinhead:PINHD-1X2
- added LED1: LED1608, generic:LED1608
- F1: device fuse:SHK20L -> fuse:SH32
Connections:
- removed net N$8: C2.1, MAIN-2.S, MD3.SENSE, MD3.VOUT, R6.2, RASPI-2.S
- removed net N$9: MD3.TRIM, U$4.1
- net GND: now also JP2.1, JP2.2, LED1.K; no longer C1.2, C2.2, KICK-1.S, MAIN-1.S, MD2-1.S, MD3.1_GROUND, MD3.2_GROUND, MD3.ON/OFF_CONTROL, R3.1, R4.1, R6.1, RASPI-1.S, SG1.-
- net N$11: no longer R5.1
- net N$3: now also F1.1A; no longer F1.2A
- net N$5: now also JP3.1, JP3.2; no longer KICK-2.S, MD1-2.S, MD2-2.S
- net N$6: now also LED1.A, U$3.0; no longer SG1.+, U$3.4
- net N$7: now also JP1.1, JP1.2, MD1-2.S; no longer R4.2, U$4.2, U$4.P$1
- net VCC: now also F1.2A, JP4.1, JP4.2, R5.1; no longer C1.1, F1.1A, MD3.VIN, R3.2
Other:
- moved on the sheet: C3, C4, F1, IC1, MD1-1, MD1-2, PAD1, PAD3, R1, U$2
