File: board/IRsensor/untitled.sch (EAGLE design)
At the start: 31 parts

Commit message: update boards 2022-07-14
Parts:
- C1, C2: value (none) -> 22pF
- C3: value (none) -> 0.1uF
- C4, C5: value (none) -> 1uF
- R1, R2: value (none) -> 22
- R3: value (none) -> 10k
Changed lines of the file:
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@@
 <part name="GND3" library="supply1" library_urn="urn:adsk.eagle:library:371" deviceset="GNDA" device=""/>
 <part name="JP1" library="adafruit" deviceset="PINHD-1X8" device="BIG"/>
-<part name="C3" library="generic" deviceset="CAPACITOR" device="1608"/>
-<part name="C4" library="generic" deviceset="CAPACITOR" device="1608"/>
-<part name="R1" library="generic" deviceset="RESISTOR-US" device="1608"/>
-<part name="R2" library="generic" deviceset="RESISTOR-US" device="1608"/>
-<part name="C5" library="generic" deviceset="CAPACITOR" device="1608"/>
+<part name="C3" library="generic" deviceset="CAPACITOR" device="1608" value="0.1uF"/>
+<part name="C4" library="generic" deviceset="CAPACITOR" device="1608" value="1uF"/>
+<part name="R1" library="generic" deviceset="RESISTOR-US" device="1608" value="22"/>
+<part name="R2" library="generic" deviceset="RESISTOR-US" device="1608" value="22"/>
+<part name="C5" library="generic" deviceset="CAPACITOR" device="1608" value="1uF"/>
 <part name="P+3" library="supply1" library_urn="urn:adsk.eagle:library:371" deviceset="+5V" device=""/>
-<part name="R3" library="generic" deviceset="RESISTOR-US" device="1608"/>
-<part name="C1" library="generic" deviceset="CAPACITOR" device="1608"/>
-<part name="C2" library="generic" deviceset="CAPACITOR" device="1608"/>
+<part name="R3" library="generic" deviceset="RESISTOR-US" device="1608" value="10k"/>
+<part name="C1" library="generic" deviceset="CAPACITOR" device="1608" value="22pF"/>
+<part name="C2" library="generic" deviceset="CAPACITOR" device="1608" value="22pF"/>
 <part name="TXLED" library="led" library_urn="urn:adsk.eagle:library:259" deviceset="LED" device="SML0603" package3d_urn="urn:adsk.eagle:package:15832/1"/>
 <part name="RXLED" library="led" library_urn="urn:adsk.eagle:library:259" deviceset="LED" device="SML0603" package3d_urn="urn:adsk.eagle:package:15832/1"/>
