File: board/IRsensor/untitled.brd (EAGLE design)
At the start: 100 x 100 mm, 31 parts

Commit message: update boards 2022-07-14
Parts:
- C1, C2: value (none) -> 22pF
- C3: value (none) -> 0.1uF
- C4, C5: value (none) -> 1uF
- R1, R2: value (none) -> 22
- R3: value (none) -> 10k
Changed lines of the file:
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@@
 <drawing>
 <settings>
-<setting alwaysvectorfont="yes"/>
+<setting alwaysvectorfont="no"/>
 <setting verticaltext="up"/>
 </settings>
@@
 </autorouter>
 <elements>
-<element name="C1" library="generic" package="SMD1608" value="" x="-0.508" y="-16.637" smashed="yes" rot="R180">
+<element name="C1" library="generic" package="SMD1608" value="22pF" x="-0.508" y="-16.637" smashed="yes" rot="R180">
 <attribute name="NAME" x="-2.248" y="-16.398" size="1.016" layer="25" rot="R180"/>
 <attribute name="VALUE" x="0.292" y="-14.987" size="1.016" layer="27" rot="R180"/>
 </element>
-<element name="C2" library="generic" package="SMD1608" value="" x="2.667" y="-16.637" smashed="yes">
+<element name="C2" library="generic" package="SMD1608" value="22pF" x="2.667" y="-16.637" smashed="yes">
 <attribute name="NAME" x="4.407" y="-17.257" size="1.016" layer="25"/>
 <attribute name="VALUE" x="1.867" y="-18.287" size="1.016" layer="27"/>
 </element>
-<element name="C3" library="generic" package="SMD1608" value="" x="10.287" y="-32.131" smashed="yes" rot="R270">
+<element name="C3" library="generic" package="SMD1608" value="0.1uF" x="10.287" y="-32.131" smashed="yes" rot="R270">
 <attribute name="NAME" x="11.191" y="-31.331" size="1.016" layer="25" rot="R270"/>
 <attribute name="VALUE" x="8.637" y="-31.331" size="1.016" layer="27" rot="R270"/>
 </element>
-<element name="C4" library="generic" package="SMD1608" value="" x="13.081" y="-32.131" smashed="yes" rot="R90">
+<element name="C4" library="generic" package="SMD1608" value="1uF" x="13.081" y="-32.131" smashed="yes" rot="R90">
 <attribute name="NAME" x="14.971" y="-32.931" size="1.016" layer="25" rot="R90"/>
 <attribute name="VALUE" x="14.731" y="-32.931" size="1.016" layer="27" rot="R90"/>
 </element>
-<element name="C5" library="generic" package="SMD1608" value="" x="15.875" y="-32.131" smashed="yes" rot="R90">
+<element name="C5" library="generic" package="SMD1608" value="1uF" x="15.875" y="-32.131" smashed="yes" rot="R90">
 <attribute name="NAME" x="17.765" y="-32.931" size="1.016" layer="25" rot="R90"/>
 <attribute name="VALUE" x="17.525" y="-32.931" size="1.016" layer="27" rot="R90"/>
@@
 <attribute name="VALUE" x="6.35" y="-16.383" size="1.27" layer="27" ratio="10" rot="R180"/>
 </element>
-<element name="R1" library="generic" package="SMD1608" value="" x="-8.89" y="-19.05" smashed="yes" rot="R270">
+<element name="R1" library="generic" package="SMD1608" value="22" x="-8.89" y="-19.05" smashed="yes" rot="R270">
 <attribute name="NAME" x="-8.24" y="-18.25" size="1.016" layer="25" rot="R270"/>
 <attribute name="VALUE" x="-10.54" y="-18.25" size="1.016" layer="27" rot="R270"/>
 </element>
-<element name="R2" library="generic" package="SMD1608" value="" x="-6.35" y="-19.05" smashed="yes" rot="R270">
+<element name="R2" library="generic" package="SMD1608" value="22" x="-6.35" y="-19.05" smashed="yes" rot="R270">
 <attribute name="NAME" x="-5.7" y="-18.25" size="1.016" layer="25" rot="R270"/>
 <attribute name="VALUE" x="-8" y="-18.25" size="1.016" layer="27" rot="R270"/>
 </element>
-<element name="R3" library="generic" package="SMD1608" value="" x="7.62" y="-16.891" smashed="yes" rot="R90">
+<element name="R3" library="generic" package="SMD1608" value="10k" x="7.62" y="-16.891" smashed="yes" rot="R90">
 <attribute name="NAME" x="6.97" y="-17.691" size="1.016" layer="25" rot="R90"/>
 <attribute name="VALUE" x="9.27" y="-17.691" size="1.016" layer="27" rot="R90"/>

Commit message: update 2022-07-15
Parts:
- moved IR13 1.00 mm to (-40.0, 0.00)
Routing:
- net +5V: track 359.5 -> 360.5 mm
- net IR13: track 64.9 -> 64.0 mm
Changed lines of the file:
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@@
 <element name="IR11" library="ir" package="IRM_V" value="IRM2121-A538" x="-28.284271875" y="-28.284271875" smashed="yes" rot="R315"/>
 <element name="IR12" library="ir" package="IRM_V" value="IRM2121-A538" x="-36.95518125" y="-15.3073375" smashed="yes" rot="R292.5"/>
-<element name="IR13" library="ir" package="IRM_V" value="IRM2121-A538" x="-40" y="1" smashed="yes" rot="R270"/>
+<element name="IR13" library="ir" package="IRM_V" value="IRM2121-A538" x="-40" y="0" smashed="yes" rot="R270"/>
 <element name="IR14" library="ir" package="IRM_V" value="IRM2121-A538" x="-36.95518125" y="15.3073375" smashed="yes" rot="R247.5"/>
 <element name="IR15" library="ir" package="IRM_V" value="IRM2121-A538" x="-28.284271875" y="28.284271875" smashed="yes" rot="R225"/>
@@
 <wire x1="-36.95518125" y1="-15.3073375" x2="-39.624" y2="-16.256" width="0.8128" layer="16"/>
 <wire x1="-39.624" y1="-16.256" x2="-30.48" y2="-30.48" width="0.8128" layer="16"/>
-<wire x1="-40" y1="1" x2="-42.926" y2="1.016" width="0.8128" layer="16"/>
-<wire x1="-42.926" y1="1.016" x2="-42.234321875" y2="-2.602003125" width="0.8128" layer="16"/>
-<wire x1="-42.234321875" y1="-2.602003125" x2="-39.624" y2="-16.256" width="0.8128" layer="16"/>
-<wire x1="-36.95518125" y1="15.3073375" x2="-39.751" y2="16.51" width="0.8128" layer="16"/>
-<wire x1="-39.751" y1="16.51" x2="-42.926" y2="1.016" width="0.8128" layer="16"/>
+<wire x1="-36.95518125" y1="15.3073375" x2="-39.74813125" y2="16.508765625" width="0.8128" layer="16"/>
+<wire x1="-39.74813125" y1="16.508765625" x2="-39.751" y2="16.51" width="0.8128" layer="16"/>
 <wire x1="-28.284271875" y1="28.284271875" x2="-30.48" y2="30.48" width="0.8128" layer="16"/>
 <wire x1="-30.48" y1="30.48" x2="-39.751" y2="16.51" width="0.8128" layer="16"/>
@@
 <wire x1="0" y1="-36.322" x2="1.27" y2="-35.052" width="0.8128" layer="16"/>
 <wire x1="7.366" y1="-35.052" x2="7.874" y2="-34.544" width="0.8128" layer="1"/>
-<wire x1="7.874" y1="-34.544" x2="7.874" y2="-30.226" width="0.8128" layer="1"/>
-<wire x1="7.874" y1="-30.226" x2="7.874" y2="-25.4" width="0.8128" layer="1"/>
+<wire x1="7.874" y1="-34.544" x2="7.874" y2="-25.4" width="0.8128" layer="1"/>
 <wire x1="7.874" y1="-25.4" x2="7.874" y2="-20.574" width="0.8128" layer="1"/>
 <wire x1="6.35" y1="-35.052" x2="5.461" y2="-34.163" width="0.254" layer="1"/>
@@
 <wire x1="1.6" y1="-25.273" x2="1.6" y2="-18.72" width="0.254" layer="16"/>
 <wire x1="1.6" y1="-18.72" x2="2.667" y2="-17.653" width="0.254" layer="16"/>
+<wire x1="-40" y1="0" x2="-43.18" y2="0" width="0.8128" layer="16"/>
+<wire x1="-43.18" y1="0" x2="-39.624" y2="-16.256" width="0.8128" layer="16"/>
+<wire x1="-39.751" y1="16.51" x2="-43.18" y2="0" width="0.8128" layer="16"/>
 </signal>
 <signal name="+5V">
@@
 <wire x1="-28.575" y1="-32.258" x2="-13.97" y2="-40.64" width="0.8128" layer="1"/>
 <wire x1="-35.9831625" y1="-17.653990625" x2="-38.608" y2="-18.796" width="0.8128" layer="1"/>
+<wire x1="-38.82485625" y1="-18.89035" x2="-38.608" y2="-18.796" width="0.8128" layer="1"/>
 <wire x1="-38.608" y1="-18.796" x2="-28.575" y2="-32.258" width="0.8128" layer="1"/>
-<wire x1="-40" y1="-1.54" x2="-42.672" y2="-1.524" width="0.8128" layer="1"/>
-<wire x1="-42.672" y1="-1.524" x2="-38.608" y2="-18.796" width="0.8128" layer="1"/>
 <wire x1="-37.927196875" y1="12.96068125" x2="-40.513" y2="13.97" width="0.8128" layer="1"/>
-<wire x1="-40.513" y1="13.97" x2="-42.672" y2="-1.524" width="0.8128" layer="1"/>
 <wire x1="-30.080321875" y1="26.48821875" x2="-32.004" y2="28.448" width="0.8128" layer="1"/>
 <wire x1="-32.004" y1="28.448" x2="-40.513" y2="13.97" width="0.8128" layer="1"/>
@@
 <wire x1="7.62" y1="-16.016" x2="8.876" y2="-16.016" width="0.254" layer="1"/>
 <wire x1="8.876" y1="-16.016" x2="8.89" y2="-16.002" width="0.254" layer="1"/>
+<wire x1="-40" y1="-2.54" x2="-43.18" y2="-2.54" width="0.8128" layer="1"/>
+<wire x1="-40.513" y1="13.97" x2="-43.18" y2="-2.54" width="0.8128" layer="1"/>
+<wire x1="-43.18" y1="-2.54" x2="-38.82485625" y2="-18.89035" width="0.8128" layer="1"/>
 </signal>
 <signal name="N$6">
@@
 <contactref element="IR13" pad="1"/>
 <contactref element="U$1" pad="36"/>
-<wire x1="-40" y1="3.54" x2="-38.846" y2="3.54" width="0.254" layer="1"/>
-<wire x1="-38.354" y1="3.048" x2="-38.846" y2="3.54" width="0.254" layer="1"/>
 <wire x1="-2.4" y1="-35.391" x2="-2.4" y2="-36.2074" width="0.254" layer="1"/>
 <wire x1="-2.4" y1="-36.2074" x2="-2.667" y2="-36.4744" width="0.254" layer="1"/>
@@
 <wire x1="-31.484425" y1="-22.998575" x2="-30.6324" y2="-23.8506" width="0.254" layer="1"/>
 <wire x1="-37.846" y1="-7.62" x2="-32.791125" y2="-20.22575625" width="0.254" layer="1"/>
-<wire x1="-38.354" y1="3.048" x2="-38.354" y2="-6.35" width="0.254" layer="1"/>
-<wire x1="-38.354" y1="-6.35" x2="-37.846" y2="-7.62" width="0.254" layer="1"/>
+<wire x1="-38.354" y1="-6.35" x2="-38.318965625" y2="-6.4375875" width="0.254" layer="1"/>
+<wire x1="-38.318965625" y1="-6.4375875" x2="-37.846" y2="-7.62" width="0.254" layer="1"/>
 <wire x1="-32.159884375" y1="-21.758775" x2="-31.484425" y2="-22.998575" width="0.254" layer="1"/>
+<wire x1="-38.318965625" y1="-6.4375875" x2="-38.318965625" y2="1.996965625" width="0.254" layer="1"/>
+<wire x1="-38.318965625" y1="1.996965625" x2="-38.862" y2="2.54" width="0.254" layer="1"/>
+<wire x1="-38.862" y1="2.54" x2="-40" y2="2.54" width="0.254" layer="1"/>
 </signal>
 <signal name="IR14">
