File: board/power_supply/v2/5v_unit.sch (EAGLE design)
At the start: 13 parts

Commit message: provisional completion
Parts:
- removed SP1: AL11P, buzzer:AL11P
Changed lines of the file:
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@@
 <?xml version="1.0" encoding="utf-8"?>
 <!DOCTYPE eagle SYSTEM "eagle.dtd">
-<eagle version="9.6.1">
+<eagle version="9.6.2">
 <drawing>
 <settings>
@@
 <part name="JP1" library="pinhead" deviceset="PINHD-1X2" device=""/>
 <part name="JP3" library="pinhead" deviceset="PINHD-1X2" device=""/>
-<part name="SP1" library="buzzer" library_urn="urn:adsk.eagle:library:113" deviceset="AL11P" device="" package3d_urn="urn:adsk.eagle:package:5308/1"/>
 </parts>
 <sheets>
@@
 <attribute name="NAME" x="59.69" y="97.155" size="1.778" layer="95"/>
 <attribute name="VALUE" x="59.69" y="86.36" size="1.778" layer="96"/>
-</instance>
-<instance part="SP1" gate="G$1" x="104.14" y="55.88" smashed="yes">
-<attribute name="NAME" x="100.33" y="62.23" size="1.778" layer="95"/>
-<attribute name="VALUE" x="100.33" y="52.705" size="1.778" layer="96"/>
 </instance>
 </instances>
@@
 will not be understood (or retained) with this version.
 </note>
-<note version="8.3" severity="warning">
-Since Version 8.3, EAGLE supports the association of 3D packages
-with devices in libraries, schematics, and board files. Those 3D
-packages will not be understood (or retained) with this version.
-</note>
 </compatibility>
