File: board/power_supply/v2/untitled.brd (EAGLE design)
At the start: 25.5 x 51.9 mm, 20 parts, among them IC1 317EMP, Q1 FDD4141TO252

Commit message: provisional completion
Parts:
- removed SG1: F/TMB, buzzer:F/TMB
- added LED1: LED1608, generic:LED1608
Connections:
- net GND: now also LED1.K; no longer SG1.-
- net N$6: now also LED1.A, U$3.5; no longer SG1.+, U$3.3
Routing:
- net N$6: track 0.00 -> 3.83 mm
- net GND: track 60.6 -> 63.1 mm
Changed lines of the file:
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@@
 </layers>
 <board>
+<fusionsync huburn="a.cGVyc29uYWw6dWUyYjhiNWJj" projecturn="a.cGVyc29uYWw6dWUyYjhiNWJjIzIwMjIwNDE2NTE3MzEzNjU2" f3durn="urn:adsk.wipprod:dm.lineage:YKynwMgpTfuc3o3DEV7zsg" pcbguid="1d484079-7f64-4e53-9d91-916d00d18d7d" lastpulledtime="" lastsyncedchangeguid="" latestrevisionid="62647a80-3215-48a6-98c3-7560700ce938" lastsyncedrevisionid="62647a80-3215-48a6-98c3-7560700ce938" lastboardhashguid="fa2de31a-8e13-641e-9703-410382d00077" lastpushedtime="2022-10-03T23:37:55Z" linktopcb3d="true"/>
 <plain>
 <wire x1="0.37778125" y1="26.860090625" x2="5.32753125" y2="21.91035" width="0.001" layer="20"/>
@@
 <attribute name="VALUE" x="12.52906875" y="31.614065625" size="1.27" layer="28" rot="MR225"/>
 </element>
-<element name="SG1" library="buzzer" library_urn="urn:adsk.eagle:library:113" package="F/TMB" package3d_urn="urn:adsk.eagle:package:5260/1" value="F/TMB" x="-4.878959375" y="41.9792" smashed="yes">
-<attribute name="MF" value="" x="52.271040625" y="35.6292" size="1.778" layer="27" display="off"/>
-<attribute name="MPN" value="" x="52.271040625" y="35.6292" size="1.778" layer="27" display="off"/>
-<attribute name="NAME" x="-1.576959375" y="47.6942" size="1.27" layer="25" ratio="10"/>
-<attribute name="OC_FARNELL" value="unknown" x="52.271040625" y="35.6292" size="1.778" layer="27" display="off"/>
-<attribute name="OC_NEWARK" value="unknown" x="52.271040625" y="35.6292" size="1.778" layer="27" display="off"/>
-<attribute name="POPULARITY" value="1" x="-4.878959375" y="41.9792" size="1.778" layer="27" display="off"/>
-<attribute name="VALUE" x="-8.688959375" y="38.1692" size="1.27" layer="27" ratio="10"/>
-</element>
 <element name="U$1" library="R3111N211A" package="R3111N211A" value="R3111N211A" x="16.406240625" y="33.8004" smashed="yes" rot="MR45"/>
 <element name="U$2" library="by_hirame" package="SMD-R-TRIM" value="2.2kΩ" x="13.536040625" y="36.2642" smashed="yes" rot="R315"/>
@@
 <attribute name="VALUE" x="17.399" y="4.318" size="1.27" layer="27" rot="R90"/>
 </element>
+<element name="LED1" library="generic" package="LED1608" value="LED1608" x="15.0622" y="23.2664" smashed="yes">
+<attribute name="NAME" x="14.2622" y="23.9164" size="1.016" layer="25"/>
+<attribute name="VALUE" x="14.2622" y="21.5664" size="1.016" layer="27"/>
+</element>
 </elements>
 <signals>
@@
 <contactref element="PAD3" pad="1"/>
 <contactref element="F1" pad="1A"/>
-<polygon width="0.1524" layer="1" isolate="0.6096" rank="3">
+<polygon width="0.1524" layer="1" isolate="0.6096" thermals="no" rank="3">
 <vertex x="20.5994" y="44.5516"/>
 <vertex x="20.5994" y="40.386"/>
@@
 <contactref element="C4" pad="1"/>
 <contactref element="C3" pad="2"/>
-<contactref element="SG1" pad="-"/>
 <contactref element="U$3" pad="4"/>
 <contactref element="JP2" pad="1"/>
@@
 <wire x1="22.1234" y1="20.8534" x2="19.0246" y2="20.8534" width="0.508" layer="16"/>
 <via x="19.0246" y="20.8534" extent="1-16" drill="0.35"/>
-<wire x1="19.0246" y1="20.8534" x2="17.8689" y2="22.0091" width="0.508" layer="1"/>
+<wire x1="19.0246" y1="20.8534" x2="18.034" y2="21.844" width="0.508" layer="1"/>
+<wire x1="18.034" y1="21.844" x2="17.8689" y2="22.0091" width="0.508" layer="1"/>
 <wire x1="22.832440625" y1="20.144359375" x2="22.1234" y2="20.8534" width="0.508" layer="16"/>
 <wire x1="17.8689" y1="22.0091" x2="17.8689" y2="28.6131" width="0.508" layer="1"/>
@@
 <wire x1="15.3924" y1="32.8676" x2="16.5608" y2="31.6992" width="0.508" layer="1"/>
 <wire x1="16.5608" y1="31.6992" x2="16.5608" y2="29.9212" width="0.508" layer="1"/>
-<wire x1="4.972884375" y1="28.6442" x2="-8.688959375" y2="41.9792" width="0" layer="19" extent="1-1"/>
+<contactref element="LED1" pad="K"/>
+<wire x1="15.9372" y1="23.2664" x2="16.6116" y2="23.2664" width="0.508" layer="1"/>
+<wire x1="16.6116" y1="23.2664" x2="17.8689" y2="22.0091" width="0.508" layer="1"/>
 </signal>
 <signal name="VCC">
@@
 <wire x1="13.953140625" y1="26.9571" x2="13.953140625" y2="26.848146875" width="0.508" layer="16"/>
 </signal>
-<signal name="N$6">
-<contactref element="U$3" pad="3"/>
-<contactref element="SG1" pad="+"/>
-<wire x1="6.7689375" y1="30.44025" x2="-1.068959375" y2="41.9792" width="0" layer="19" extent="1-1"/>
-</signal>
 <signal name="N$7">
 <contactref element="JP1" pad="2"/>
@@
 </polygon>
 </signal>
+<signal name="N$6">
+<contactref element="U$3" pad="5"/>
+<contactref element="LED1" pad="A"/>
+<wire x1="10.361040625" y1="23.25604375" x2="14.17684375" y2="23.25604375" width="0.508" layer="1"/>
+<wire x1="14.17684375" y1="23.25604375" x2="14.1872" y2="23.2664" width="0.508" layer="1"/>
+</signal>
 </signals>
 <mfgpreviewcolors>
@@
 </note>
 <note version="8.3" severity="warning">
+Since Version 8.3, EAGLE supports Fusion synchronisation.
+This feature will not be available in this version and saving
+the document will break the link to the Fusion PCB feature.
+</note>
+<note version="8.3" severity="warning">

Commit message: change dimention & check DRC
Other:
- board size 25.5 x 51.9 mm -> 25.1 x 51.4 mm
Changed lines of the file:
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@@
 <drawing>
 <settings>
-<setting alwaysvectorfont="yes"/>
+<setting alwaysvectorfont="no"/>
 <setting verticaltext="up"/>
 </settings>
@@
 </layers>
 <board>
-<fusionsync huburn="a.cGVyc29uYWw6dWUyYjhiNWJj" projecturn="a.cGVyc29uYWw6dWUyYjhiNWJjIzIwMjIwNDE2NTE3MzEzNjU2" f3durn="urn:adsk.wipprod:dm.lineage:YKynwMgpTfuc3o3DEV7zsg" pcbguid="1d484079-7f64-4e53-9d91-916d00d18d7d" lastpulledtime="" lastsyncedchangeguid="" latestrevisionid="62647a80-3215-48a6-98c3-7560700ce938" lastsyncedrevisionid="62647a80-3215-48a6-98c3-7560700ce938" lastboardhashguid="fa2de31a-8e13-641e-9703-410382d00077" lastpushedtime="2022-10-03T23:37:55Z" linktopcb3d="true"/>
+<fusionsync huburn="a.cGVyc29uYWw6dWUyYjhiNWJj" projecturn="a.cGVyc29uYWw6dWUyYjhiNWJjIzIwMjIwNDE2NTE3MzEzNjU2" f3durn="urn:adsk.wipprod:dm.lineage:YKynwMgpTfuc3o3DEV7zsg" pcbguid="" lastpulledtime="" lastsyncedchangeguid="" latestrevisionid="62647a80-3215-48a6-98c3-7560700ce938" lastsyncedrevisionid="62647a80-3215-48a6-98c3-7560700ce938" lastboardhashguid="fa2de31a-8e13-641e-9703-410382d00077" lastpushedtime="2022-10-03T23:37:55Z" linktopcb3d="true"/>
 <plain>
-<wire x1="0.37778125" y1="26.860090625" x2="5.32753125" y2="21.91035" width="0.001" layer="20"/>
-<wire x1="5.32753125" y1="21.91035" x2="5.32753125" y2="14.83928125" width="0.001" layer="20" curve="-90"/>
-<wire x1="5.32753125" y1="14.83928125" x2="0" y2="9.51175" width="0.001" layer="20"/>
-<wire x1="0" y1="9.51175" x2="25.461040625" y2="0" width="0.001" layer="20" curve="15.16"/>
-<wire x1="25.461040625" y1="0" x2="25.461040625" y2="51.943359375" width="0.001" layer="20"/>
-<wire x1="25.461040625" y1="51.943359375" x2="13.461040625" y2="51.943359375" width="0.001" layer="20"/>
-<wire x1="13.461040625" y1="51.943359375" x2="13.461040625" y2="39.943359375" width="0.001" layer="20"/>
-<wire x1="13.461040625" y1="39.943359375" x2="0.37778125" y2="26.860090625" width="0.001" layer="20"/>
+<wire x1="25.083259375" y1="51.943359375" x2="25.083259375" y2="2.542159375" width="0.001" layer="20"/>
+<wire x1="25.083259375" y1="51.943359375" x2="13.083259375" y2="51.943359375" width="0.001" layer="20"/>
+<wire x1="13.083259375" y1="51.943359375" x2="13.083259375" y2="39.943359375" width="0.001" layer="20"/>
+<wire x1="13.083259375" y1="39.943359375" x2="0" y2="26.8601" width="0.001" layer="20"/>
+<wire x1="0" y1="26.8601" x2="4.94975" y2="21.91035" width="0.001" layer="20"/>
+<wire x1="4.94975" y1="14.83928125" x2="4.94975" y2="21.91035" width="0.001" layer="20" curve="90"/>
+<wire x1="2.706109375" y1="7.933459375" x2="22.58841875" y2="0.60435" width="0.001" layer="20" curve="11.808321"/>
+<wire x1="22.58841875" y1="0.60435" x2="25.083259375" y2="2.542159375" width="0.001" layer="20" curve="104.324739"/>
+<wire x1="2.05935" y1="11.948890625" x2="2.706109375" y2="7.933459375" width="0.001" layer="20" curve="108.864352"/>
+<wire x1="4.94975" y1="14.83928125" x2="2.05935" y2="11.948890625" width="0.001" layer="20"/>
 </plain>
 <attributes>
@@
 </class>
 </classes>
-<designrules name="default">
+<designrules name="Elecrow_2-layer_PCB_eagle_rule">
+<description language="de">&lt;b&gt;EAGLE Design Rules&lt;/b&gt;
+&lt;p&gt;
+Die Standard-Design-Rules sind so gewählt, dass sie für
+die meisten Anwendungen passen. Sollte ihre Platine
+besondere Anforderungen haben, treffen Sie die erforderlichen
+Einstellungen hier und speichern die Design Rules unter
+einem neuen Namen ab.</description>
 <description language="en">&lt;b&gt;EAGLE Design Rules&lt;/b&gt;
 &lt;p&gt;
@@
 may have different requirements, so please make the
 necessary adjustments and save your customized
-design rules under a new name.
+design rules under a new name.</description>
+<description language="zh">&lt;b&gt;Elecrow PCB EAGLE Design Rules&lt;/b&gt;
 </description>
 <param name="layerSetup" value="(1*16)"/>
 <param name="mtCopper" value="0.035mm 0.035mm 0.035mm 0.035mm 0.035mm 0.035mm 0.035mm 0.035mm 0.035mm 0.035mm 0.035mm 0.035mm 0.035mm 0.035mm 0.035mm 0.035mm"/>
-<param name="mtIsolate" value="0.15mm 0.15mm 0.2mm 0.15mm 0.2mm 0.15mm 0.2mm 0.15mm 0.2mm 0.15mm 0.2mm 0.15mm 0.2mm 0.15mm 0.2mm"/>
+<param name="mtIsolate" value="1.6mm 1.2mm 0.2mm 0.15mm 0.2mm 0.15mm 0.2mm 0.15mm 0.2mm 0.15mm 0.2mm 0.15mm 0.2mm 0.15mm 0.2mm"/>
 <param name="mdWireWire" value="6mil"/>
 <param name="mdWirePad" value="6mil"/>
@@
 <param name="mdPadPad" value="6mil"/>
 <param name="mdPadVia" value="6mil"/>
-<param name="mdViaVia" value="6mil"/>
-<param name="mdSmdPad" value="6mil"/>
-<param name="mdSmdVia" value="6mil"/>
-<param name="mdSmdSmd" value="6mil"/>
-<param name="mdViaViaSameLayer" value="6mil"/>
+<param name="mdViaVia" value="8mil"/>
+<param name="mdSmdPad" value="0mil"/>
+<param name="mdSmdVia" value="0mil"/>
+<param name="mdSmdSmd" value="0mil"/>
+<param name="mdViaViaSameLayer" value="8mil"/>
 <param name="mnLayersViaInSmd" value="2"/>
-<param name="mdCopperDimension" value="40mil"/>
-<param name="mdDrill" value="6mil"/>
+<param name="mdCopperDimension" value="20mil"/>
+<param name="mdDrill" value="10mil"/>
 <param name="mdSmdStop" value="0mil"/>
 <param name="msWidth" value="6mil"/>
-<param name="msDrill" value="0.35mm"/>
-<param name="msMicroVia" value="9.99mm"/>
+<param name="msDrill" value="12mil"/>
+<param name="msMicroVia" value="12mil"/>
 <param name="msBlindViaRatio" value="0.5"/>
 <param name="rvPadTop" value="0.25"/>
@@
 <param name="rvMicroViaOuter" value="0.25"/>
 <param name="rvMicroViaInner" value="0.25"/>
-<param name="rlMinPadTop" value="10mil"/>
+<param name="rlMinPadTop" value="6mil"/>
 <param name="rlMaxPadTop" value="20mil"/>
-<param name="rlMinPadInner" value="10mil"/>
+<param name="rlMinPadInner" value="6mil"/>
 <param name="rlMaxPadInner" value="20mil"/>
-<param name="rlMinPadBottom" value="10mil"/>
+<param name="rlMinPadBottom" value="6mil"/>
 <param name="rlMaxPadBottom" value="20mil"/>
-<param name="rlMinViaOuter" value="8mil"/>
+<param name="rlMinViaOuter" value="6mil"/>
 <param name="rlMaxViaOuter" value="20mil"/>
-<param name="rlMinViaInner" value="8mil"/>
+<param name="rlMinViaInner" value="6mil"/>
 <param name="rlMaxViaInner" value="20mil"/>
 <param name="rlMinMicroViaOuter" value="4mil"/>
@@
 <param name="psTop" value="-1"/>
 <param name="psBottom" value="-1"/>
-<param name="psFirst" value="-1"/>
+<param name="psFirst" value="0"/>
 <param name="psElongationLong" value="100"/>
 <param name="psElongationOffset" value="100"/>
 <param name="mvStopFrame" value="1"/>
 <param name="mvCreamFrame" value="0"/>
-<param name="mlMinStopFrame" value="4mil"/>
-<param name="mlMaxStopFrame" value="4mil"/>
+<param name="mlMinStopFrame" value="0mil"/>
+<param name="mlMaxStopFrame" value="0mil"/>
 <param name="mlMinCreamFrame" value="0mil"/>
 <param name="mlMaxCreamFrame" value="0mil"/>
-<param name="mlViaStopLimit" value="0mil"/>
+<param name="mlViaStopLimit" value="100mil"/>
 <param name="srRoundness" value="0"/>
 <param name="srMinRoundness" value="0mil"/>
@@
 <param name="checkAngle" value="0"/>
 <param name="checkFont" value="1"/>
-<param name="checkRestrict" value="1"/>
+<param name="checkRestrict" value="0"/>
 <param name="checkStop" value="0"/>
 <param name="checkValues" value="0"/>
@@
 <param name="checkPolygonWidth" value="0"/>
 <param name="useDiameter" value="13"/>
-<param name="maxErrors" value="999999"/>
+<param name="maxErrors" value="50"/>
 </designrules>
 <autorouter>

Commit message: marge前のファイル
Connections:
- net N$11: no longer R5.1
- net VCC: now also R5.1
Routing:
- net VCC: track 33.3 -> 44.6 mm, vias 0 -> 1
Changed lines of the file:
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@@
 <?xml version="1.0" encoding="utf-8"?>
 <!DOCTYPE eagle SYSTEM "eagle.dtd">
-<eagle version="9.6.2">
+<eagle version="9.6.1">
 <drawing>
 <settings>
@@
 </layers>
 <board>
-<fusionsync huburn="a.cGVyc29uYWw6dWUyYjhiNWJj" projecturn="a.cGVyc29uYWw6dWUyYjhiNWJjIzIwMjIwNDE2NTE3MzEzNjU2" f3durn="urn:adsk.wipprod:dm.lineage:YKynwMgpTfuc3o3DEV7zsg" pcbguid="" lastpulledtime="" lastsyncedchangeguid="" latestrevisionid="62647a80-3215-48a6-98c3-7560700ce938" lastsyncedrevisionid="62647a80-3215-48a6-98c3-7560700ce938" lastboardhashguid="fa2de31a-8e13-641e-9703-410382d00077" lastpushedtime="2022-10-03T23:37:55Z" linktopcb3d="true"/>
+<fusionsync huburn="a.cGVyc29uYWw6dWUyYjhiNWJj" projecturn="a.cGVyc29uYWw6dWUyYjhiNWJjIzIwMjIwNDE2NTE3MzEzNjU2" f3durn="urn:adsk.wipprod:dm.lineage:YKynwMgpTfuc3o3DEV7zsg" pcbguid="" lastpulledtime="" lastsyncedchangeguid="" latestrevisionid="62647a80-3215-48a6-98c3-7560700ce938" lastsyncedrevisionid="62647a80-3215-48a6-98c3-7560700ce938" lastboardhashguid="fa2de31a-8e13-641e-9703-410382d00077" lastpushedtime="2022-10-03T23:37:55Z" linktopcb3d="%12"/>
 <plain>
 <wire x1="25.083259375" y1="51.943359375" x2="25.083259375" y2="2.542159375" width="0.001" layer="20"/>
@@
 <wire x1="22.1234" y1="20.8534" x2="19.0246" y2="20.8534" width="0.508" layer="16"/>
 <via x="19.0246" y="20.8534" extent="1-16" drill="0.35"/>
-<wire x1="19.0246" y1="20.8534" x2="18.034" y2="21.844" width="0.508" layer="1"/>
-<wire x1="18.034" y1="21.844" x2="17.8689" y2="22.0091" width="0.508" layer="1"/>
+<wire x1="19.0246" y1="20.8534" x2="17.8689" y2="22.0091" width="0.508" layer="1"/>
 <wire x1="22.832440625" y1="20.144359375" x2="22.1234" y2="20.8534" width="0.508" layer="16"/>
 <wire x1="17.8689" y1="22.0091" x2="17.8689" y2="28.6131" width="0.508" layer="1"/>
@@
 <wire x1="8.8392" y1="21.7424" x2="14.097" y2="21.7424" width="0.508" layer="16"/>
 <wire x1="14.097" y1="21.7424" x2="14.986" y2="20.8534" width="0.508" layer="16"/>
-<wire x1="14.8859625" y1="33.623621875" x2="14.129940625" y2="32.8676" width="0.508" layer="16"/>
-<wire x1="14.129940625" y1="32.8676" x2="14.097" y2="32.8676" width="0.508" layer="16"/>
-<via x="14.097" y="32.8676" extent="1-16" drill="0.35"/>
-<wire x1="14.097" y1="32.8676" x2="15.3924" y2="32.8676" width="0.508" layer="1"/>
+<wire x1="14.8859625" y1="33.623621875" x2="14.625984375" y2="33.8836" width="0.508" layer="16"/>
+<wire x1="14.625984375" y1="33.8836" x2="13.97" y2="33.8836" width="0.508" layer="16"/>
+<via x="13.97" y="33.8836" extent="1-16" drill="0.35"/>
+<wire x1="13.97" y1="33.8836" x2="14.3764" y2="33.8836" width="0.508" layer="1"/>
 <wire x1="16.5608" y1="29.9212" x2="17.8689" y2="28.6131" width="0.508" layer="1"/>
-<wire x1="15.3924" y1="32.8676" x2="16.5608" y2="31.6992" width="0.508" layer="1"/>
+<wire x1="14.3764" y1="33.8836" x2="16.5608" y2="31.6992" width="0.508" layer="1"/>
 <wire x1="16.5608" y1="31.6992" x2="16.5608" y2="29.9212" width="0.508" layer="1"/>
 <contactref element="LED1" pad="K"/>
@@
 <wire x1="17.560846875" y1="34.29" x2="22.86" y2="34.29" width="0.508" layer="1"/>
 <wire x1="24.13" y1="33.02" x2="24.13" y2="16.124159375" width="0.508" layer="1"/>
+<contactref element="R5" pad="1"/>
+<wire x1="14.20779375" y1="30.512446875" x2="14.20779375" y2="32.42660625" width="0.3048" layer="16"/>
+<wire x1="11.7602" y1="37.2364" x2="12.6492" y2="38.1254" width="0.3048" layer="16"/>
+<via x="12.6492" y="38.1254" extent="1-16" drill="0.35"/>
+<wire x1="12.6492" y1="38.1254" x2="13.725446875" y2="38.1254" width="0.3048" layer="1"/>
+<wire x1="13.725446875" y1="38.1254" x2="14.56134375" y2="37.289503125" width="0.3048" layer="1"/>
+<wire x1="14.20779375" y1="32.42660625" x2="11.7602" y2="34.8742" width="0.3048" layer="16"/>
+<wire x1="11.7602" y1="34.8742" x2="11.7602" y2="37.2364" width="0.3048" layer="16"/>
 </signal>
 <signal name="N$1">
@@
 <contactref element="C4" pad="2"/>
 <contactref element="U$3" pad="8"/>
-<contactref element="R5" pad="1"/>
 <contactref element="R2" pad="2"/>
 <wire x1="8.312759375" y1="25.10448125" x2="8.312759375" y2="27.30441875" width="0.508" layer="16"/>
 <wire x1="8.312759375" y1="27.30441875" x2="9.054290625" y2="28.04595" width="0.508" layer="16"/>
-<wire x1="15.74919375" y1="28.6442" x2="14.20779375" y2="30.1856" width="0.508" layer="16"/>
-<wire x1="14.20779375" y1="30.1856" x2="14.20779375" y2="30.512446875" width="0.508" layer="16"/>
 <wire x1="15.74919375" y1="28.6442" x2="19.63519375" y2="24.7582" width="0.508" layer="16"/>
 <wire x1="19.63519375" y1="24.7582" x2="20.521040625" y2="24.7582" width="0.508" layer="16"/>
@@
 <wire x1="10.795" y1="28.4226" x2="12.5984" y2="30.226" width="0.508" layer="1"/>
 <via x="12.5984" y="30.226" extent="1-16" drill="0.35"/>
-<wire x1="12.5984" y1="30.226" x2="13.921346875" y2="30.226" width="0.508" layer="16"/>
-<wire x1="13.921346875" y1="30.226" x2="14.20779375" y2="30.512446875" width="0.508" layer="16"/>
+<wire x1="12.5984" y1="30.226" x2="14.1802" y2="28.6442" width="0.3048" layer="16"/>
+<wire x1="14.1802" y1="28.6442" x2="15.74919375" y2="28.6442" width="0.3048" layer="16"/>
 </signal>
 <signal name="N$10">
