File: board/power_supply/v2/untitled.sch (EAGLE design)
At the start: 27 parts, among them IC1 317EMP, Q1 FDD4141TO252

Commit message: update powerboard v2
Parts:
- removed C1: 22uF 25V, adafruit:C-USC2012
- removed C2: 10uF 10V, adafruit:C-USC2012
- removed KICK, MAIN, MD2, RASPI: JST-XH-02-PIN-LONG-PAD, Rembrandt Electronics - JST XH Connectors v1-0:JST-XH-02-PIN-LONG-PAD
- removed MD3: OKL-T/6-W12P-CMURATA_OKL-T-6-W12P-C_0_0, OKL-T_6-W12P-C:OKL-T/6-W12P-CMURATA_OKL-T-6-W12P-C_0_0
- removed R3: 20kΩ, adafruit:R-US_M2012
- removed R4: 1.2kΩ, adafruit:R-US_M2012
- removed R6: 1.2KΩ 1/6W, adafruit:FLIPFLOP-RES
- removed U$4: 20kΩ, by_hirame:R-TRIM
- added JP1, JP2, JP3, JP4: (no value), pinhead:PINHD-1X2
Connections:
- removed net N$8: C2.1, MAIN-2.S, MD3.SENSE, MD3.VOUT, R6.2, RASPI-2.S
- removed net N$9: MD3.TRIM, U$4.1
- net GND: now also JP2.1, JP2.2; no longer C1.2, C2.2, KICK-1.S, MAIN-1.S, MD2-1.S, MD3.1_GROUND, MD3.2_GROUND, MD3.ON/OFF_CONTROL, R3.1, R4.1, R6.1, RASPI-1.S
- net N$3: now also F1.1A; no longer F1.2A
- net N$5: now also JP3.1, JP3.2; no longer KICK-2.S, MD1-2.S, MD2-2.S
- net N$7: now also JP1.1, JP1.2, MD1-2.S; no longer R4.2, U$4.2, U$4.P$1
- net VCC: now also F1.2A, JP4.1, JP4.2; no longer C1.1, F1.1A, MD3.VIN, R3.2
Other:
- moved on the sheet: F1, MD1-1, MD1-2

Commit message: provisional completion
Parts:
- removed SG1: F/TMB, buzzer:F/TMB
- added LED1: LED1608, generic:LED1608
Connections:
- net GND: now also LED1.K; no longer SG1.-
- net N$6: now also LED1.A, U$3.0; no longer SG1.+, U$3.4
Changed lines of the file:
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@@
 <part name="R5" library="adafruit" deviceset="R-US_" device="M2012" value="10k"/>
 <part name="R7" library="adafruit" deviceset="R-US_" device="M2012" value="300Ω"/>
-<part name="SG1" library="buzzer" library_urn="urn:adsk.eagle:library:113" deviceset="F/TMB" device="" package3d_urn="urn:adsk.eagle:package:5260/1"/>
 <part name="GND5" library="supply1" library_urn="urn:adsk.eagle:library:371" deviceset="GND" device=""/>
 <part name="F1" library="fuse" library_urn="urn:adsk.eagle:library:233" deviceset="SH32" device="" package3d_urn="urn:adsk.eagle:package:14068/1"/>
@@
 <part name="JP4" library="pinhead" deviceset="PINHD-1X2" device=""/>
 <part name="P+3" library="supply1" library_urn="urn:adsk.eagle:library:371" deviceset="VCC" device=""/>
+<part name="LED1" library="generic" deviceset="LED" device="1608"/>
+<part name="GND6" library="supply1" library_urn="urn:adsk.eagle:library:371" deviceset="GND" device=""/>
 </parts>
 <sheets>
@@
 <attribute name="VALUE" x="-6.35" y="8.382" size="1.778" layer="96" rot="R180"/>
 </instance>
-<instance part="SG1" gate="1" x="-53.34" y="2.54" smashed="yes" rot="MR0">
-<attribute name="NAME" x="-50.8" y="8.89" size="1.778" layer="95" rot="MR0"/>
-<attribute name="VALUE" x="-58.42" y="2.54" size="1.778" layer="96" rot="MR0"/>
-</instance>
-<instance part="GND5" gate="1" x="-63.5" y="-10.16" smashed="yes">
-<attribute name="VALUE" x="-66.04" y="-12.7" size="1.778" layer="96"/>
+<instance part="GND5" gate="1" x="-45.72" y="-10.16" smashed="yes">
+<attribute name="VALUE" x="-48.26" y="-12.7" size="1.778" layer="96"/>
 </instance>
 <instance part="F1" gate="G$1" x="38.1" y="50.8" smashed="yes" rot="R180">
@@
 <instance part="P+3" gate="VCC" x="20.32" y="78.74" smashed="yes">
 <attribute name="VALUE" x="17.78" y="76.2" size="1.778" layer="96" rot="R90"/>
+</instance>
+<instance part="LED1" gate="G$1" x="-12.7" y="-12.7" smashed="yes">
+<attribute name="NAME" x="-11.43" y="-9.906" size="1.778" layer="95" font="vector"/>
+</instance>
+<instance part="GND6" gate="1" x="-12.7" y="-22.86" smashed="yes">
+<attribute name="VALUE" x="-15.24" y="-25.4" size="1.778" layer="96"/>
 </instance>
 </instances>
@@
 </segment>
 <segment>
-<pinref part="SG1" gate="1" pin="-"/>
-<wire x1="-58.42" y1="0" x2="-63.5" y2="0" width="0.1524" layer="91"/>
-<wire x1="-63.5" y1="0" x2="-63.5" y2="-5.08" width="0.1524" layer="91"/>
 <pinref part="U$3" gate="G$1" pin="GND"/>
-<wire x1="-43.18" y1="-5.08" x2="-63.5" y2="-5.08" width="0.1524" layer="91"/>
-<wire x1="-63.5" y1="-5.08" x2="-63.5" y2="-7.62" width="0.1524" layer="91"/>
-<junction x="-63.5" y="-5.08"/>
+<wire x1="-43.18" y1="-5.08" x2="-45.72" y2="-5.08" width="0.1524" layer="91"/>
+<wire x1="-45.72" y1="-5.08" x2="-45.72" y2="-7.62" width="0.1524" layer="91"/>
 <pinref part="GND5" gate="1" pin="GND"/>
 </segment>
@@
 <junction x="0" y="68.58"/>
 <pinref part="GND3" gate="1" pin="GND"/>
+</segment>
+<segment>
+<pinref part="LED1" gate="G$1" pin="K"/>
+<wire x1="-12.7" y1="-15.24" x2="-12.7" y2="-20.32" width="0.1524" layer="91"/>
+<pinref part="GND6" gate="1" pin="GND"/>
 </segment>
 </net>
@@
 </segment>
 </net>
-<net name="N$6" class="0">
-<segment>
-<pinref part="U$3" gate="G$1" pin="4"/>
-<pinref part="SG1" gate="1" pin="+"/>
-<wire x1="-43.18" y1="0" x2="-50.8" y2="0" width="0.1524" layer="91"/>
-</segment>
-</net>
 <net name="N$7" class="0">
 <segment>
@@
 </segment>
 </net>
+<net name="N$6" class="0">
+<segment>
+<pinref part="U$3" gate="G$1" pin="0"/>
+<pinref part="LED1" gate="G$1" pin="A"/>
+<wire x1="-17.78" y1="-5.08" x2="-12.7" y2="-5.08" width="0.1524" layer="91"/>
+<wire x1="-12.7" y1="-5.08" x2="-12.7" y2="-7.62" width="0.1524" layer="91"/>
+</segment>
+</net>

Commit message: marge前のファイル
Connections:
- net N$11: no longer R5.1
- net VCC: now also R5.1
Other:
- moved on the sheet: C3, C4, F1, IC1, JP2, JP4, PAD1, PAD3, R1, U$2

Commit message: Revert "Merge remote-tracking branch 'origin/Develop' into feature_#37"
This reverts commit cb103155361e8766478c6830db153463370c0739, reversing
changes made to 84e093fe944e1f8653a6822ff34e6f8740617cb5.
Connections:
- net N$11: now also R5.1
- net VCC: no longer R5.1
Other:
- moved on the sheet: C3, C4, F1, IC1, JP2, JP4, PAD1, PAD3, R1, U$2
