File: board/UI_board/v1/untitled.brd (EAGLE design)
At the start: 160 x 100 mm, 19 parts

Commit message: complete wiring
Parts:
- added RASPI_RESET: (no value), SparkFun-Switches:TACTILE_SWITCH_SMD_5.2MM
- JP1: device pinhead:1X10 -> pinhead:1X14
- moved R6 37.8 mm to (27.9, 6.35), turned to 270 degrees
- moved R5 33.2 mm to (25.4, 6.35), turned to 270 degrees
- moved R2 32.5 mm to (30.5, 10.2), turned to 180 degrees
- moved R4 28.7 mm to (22.9, 6.35), turned to 270 degrees
- moved LED3 25.8 mm to (20.3, 3.17)
- moved R3 24.3 mm to (20.3, 6.35), turned to 270 degrees
- moved LED4 21.3 mm to (22.9, 3.17)
- moved LED5 21.3 mm to (25.4, 3.17)
- moved LED6 21.3 mm to (27.9, 3.17)
- moved R1 19.8 mm to (17.8, 10.2)
- moved MAIN_RESET 10.2 mm to (11.4, 6.35)
- moved LED2 9.92 mm to (26.7, 10.2)
- moved LED1 6.84 mm to (21.6, 10.2)
- moved GYRO_RESET 5.24 mm to (3.81, 6.35)
- moved JP1 4.58 mm to (24.1, 22.9)
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Connections:
- removed net N$10: R2.1
- removed net N$11: R1.1
- removed net N$7: R6.1
- removed net N$8: R4.1
- removed net N$9: R3.1
- new net D+: JP1.12, JP4.3
- new net D-: JP1.13, JP4.2
- new net GYRO_L: JP1.5, R1.1
- new net GYRO_R: JP1.6, R2.1
- new net LINE: JP1.3, R3.1
- new net RASPI_RESET: JP1.10, RASPI_RESET.3, RASPI_RESET.4
- new net UVCC: JP1.14, JP4.1
- net CAM_STATUS: now also JP1.8, R6.1; no longer JP1.3
- net GND: now also JP1.11, JP4.4, JP4.7, RASPI_RESET.1, RASPI_RESET.2; no longer JP1.10
- net GYRO_RESET: now also JP1.1
- net GYRO_STATUS: now also JP1.4, R4.1; no longer JP1.1
- net IR_RESET: now also JP1.9
- net IR_STATUS: now also JP1.7; no longer JP1.2
- net MAIN_RESET: now also JP1.2
Routing:
- net GND: track 66.0 -> 113.9 mm
- net IR_STATUS: track 0.00 -> 30.9 mm
- net RASPI_RESET: track 0.00 -> 28.1 mm
- net CAM_STATUS: track 0.00 -> 27.9 mm, vias 0 -> 2
- net GYRO_R: track 0.00 -> 24.6 mm
- net IR_RESET: track 0.00 -> 23.8 mm
- net GYRO_STATUS: track 0.00 -> 23.7 mm
- net LINE: track 0.00 -> 20.2 mm, vias 0 -> 1
- net GYRO_L: track 0.00 -> 15.9 mm
- net MAIN_RESET: track 0.00 -> 15.0 mm
- net GYRO_RESET: track 5.59 -> 20.1 mm
- net UVCC: track 0.00 -> 13.8 mm
- net D-: track 0.00 -> 13.8 mm
- net D+: track 0.00 -> 13.8 mm
- net N$6: track 0.00 -> 1.42 mm
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