File: board/UI_board/v1/untitled.brd (EAGLE design)
At the start: 56 x 25 mm, 22 parts, among them X1 JST-XH-02-PIN-ROUND-PAD

Commit message: Revert "Merge remote-tracking branch 'origin/Develop' into feature_#37"
This reverts commit cb103155361e8766478c6830db153463370c0739, reversing
changes made to 84e093fe944e1f8653a6822ff34e6f8740617cb5.
Parts:
- removed JP1: (no value), pinhead:1X18
- removed U$1: TRIM-3386K, R-trim:TRIM-3386K
- added JP5: (no value), pinhead:1X16
Connections:
- removed net +3V3: JP1.13, U$1.P$3
- removed net TRIM: JP1.1, U$1.P$1
- net CAM_STATUS: now also JP5.8; no longer JP1.9
- net D+: now also JP5.14; no longer JP1.16
- net D-: now also JP5.15; no longer JP1.17
- net GND: now also JP5.12, JP5.13; no longer JP1.14, JP1.15, U$1.P$2
- net GYRO_L: now also JP5.5; no longer JP1.6
- net GYRO_R: now also JP5.6; no longer JP1.7
- net GYRO_RESET: now also JP5.1; no longer JP1.2
- net GYRO_STATUS: now also JP5.4; no longer JP1.5
- net IR_RESET: now also JP5.9; no longer JP1.10
- net IR_STATUS: now also JP5.7; no longer JP1.8
- net LINE: now also JP5.3; no longer JP1.4
- net MAIN_RESET: now also JP5.2; no longer JP1.3
- net RASPI_RESET: now also JP5.10; no longer JP1.11
- net SWITCH: now also JP5.11; no longer JP1.12
- net UVCC: now also JP5.16; no longer JP1.18
Routing:
- net +3V3: track 31.6 -> 0.00 mm, vias 2 -> 0
- net TRIM: track 7.74 -> 0.00 mm
- net GND: track 134.9 -> 128.0 mm, vias 2 -> 1
- net UVCC: track 19.2 -> 15.6 mm
- net GYRO_RESET: track 21.7 -> 19.6 mm
- net N$2: track 2.06 -> 0.00 mm
- net N$1: track 2.06 -> 0.00 mm
- net D-: track 18.3 -> 16.5 mm
- net D+: track 18.5 -> 17.4 mm
- net SWITCH: track 13.8 -> 12.9 mm

Commit message: marge前のファイル
Parts:
- removed JP5: (no value), pinhead:1X16
- added JP1: (no value), pinhead:1X18
- added U$1: TRIM-3386K, R-trim:TRIM-3386K
Connections:
- new net +3V3: JP1.13, U$1.P$3
- new net TRIM: JP1.1, U$1.P$1
- net CAM_STATUS: now also JP1.9; no longer JP5.8
- net D+: now also JP1.16; no longer JP5.14
- net D-: now also JP1.17; no longer JP5.15
- net GND: now also JP1.14, JP1.15, U$1.P$2; no longer JP5.12, JP5.13
- net GYRO_L: now also JP1.6; no longer JP5.5
- net GYRO_R: now also JP1.7; no longer JP5.6
- net GYRO_RESET: now also JP1.2; no longer JP5.1
- net GYRO_STATUS: now also JP1.5; no longer JP5.4
- net IR_RESET: now also JP1.10; no longer JP5.9
- net IR_STATUS: now also JP1.8; no longer JP5.7
- net LINE: now also JP1.4; no longer JP5.3
- net MAIN_RESET: now also JP1.3; no longer JP5.2
- net RASPI_RESET: now also JP1.11; no longer JP5.10
- net SWITCH: now also JP1.12; no longer JP5.11
- net UVCC: now also JP1.18; no longer JP5.16
Routing:
- net +3V3: track 0.00 -> 31.6 mm, vias 0 -> 2
- net TRIM: track 0.00 -> 7.74 mm
- net GND: track 128.0 -> 134.9 mm, vias 1 -> 2
- net UVCC: track 15.6 -> 19.2 mm
- net GYRO_RESET: track 19.6 -> 21.7 mm
- net D-: track 16.5 -> 18.3 mm
- net D+: track 17.4 -> 18.5 mm
- net SWITCH: track 12.9 -> 13.8 mm
