File: board/UI_board/v1/untitled.sch (EAGLE design)
At the start: 19 parts

Commit message: complete wiring
Parts:
- added RASPI_RESET: (no value), SparkFun-Switches:MOMENTARY-SWITCH-SPST-2-SMD-5.2MM
- JP1: device pinhead:PINHD-1X10 -> pinhead:PINHD-1X14
Connections:
- removed net N$10: R2.1
- removed net N$11: R1.1
- removed net N$7: R6.1
- removed net N$8: R4.1
- removed net N$9: R3.1
- new net D+: JP1.12, JP4.3
- new net D-: JP1.13, JP4.2
- new net GYRO_L: JP1.5, R1.1
- new net GYRO_R: JP1.6, R2.1
- new net LINE: JP1.3, R3.1
- new net RASPI_RESET: JP1.10, RASPI_RESET.3, RASPI_RESET.4
- new net UVCC: JP1.14, JP4.1
- net CAM_STATUS: now also JP1.8, R6.1; no longer JP1.3
- net GND: now also JP1.11, JP4.4, JP4.7, RASPI_RESET.1, RASPI_RESET.2; no longer JP1.10
- net GYRO_RESET: now also JP1.1
- net GYRO_STATUS: now also JP1.4, R4.1; no longer JP1.1
- net IR_RESET: now also JP1.9
- net IR_STATUS: now also JP1.7; no longer JP1.2
- net MAIN_RESET: now also JP1.2

Commit message: complete UI board
Parts:
- removed JP1: (no value), pinhead:PINHD-1X14
- added JP5: (no value), pinhead:PINHD-1X16
- added X1: JST-XH-02-PIN-ROUND-PAD, Rembrandt Electronics - JST XH Connectors v1-0:JST-XH-02-PIN-ROUND-PAD
Connections:
- new net SWITCH: JP5.11, X1-2.S
- net CAM_STATUS: now also JP5.8; no longer JP1.8
- net D+: now also JP5.14; no longer JP1.12
- net D-: now also JP5.15; no longer JP1.13
- net GND: now also JP5.12, JP5.13, X1-1.S; no longer JP1.11
- net GYRO_L: now also JP5.5; no longer JP1.5
- net GYRO_R: now also JP5.6; no longer JP1.6
- net GYRO_RESET: now also JP5.1; no longer JP1.1
- net GYRO_STATUS: now also JP5.4; no longer JP1.4
- net IR_RESET: now also JP5.9; no longer JP1.9
- net IR_STATUS: now also JP5.7; no longer JP1.7
- net LINE: now also JP5.3; no longer JP1.3
- net MAIN_RESET: now also JP5.2; no longer JP1.2
- net RASPI_RESET: now also JP5.10; no longer JP1.10
- net UVCC: now also JP5.16; no longer JP1.14
Changed lines of the file:
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@@
 <part name="JP4" library="pinhead" deviceset="PINHD-1X7" device=""/>
 <part name="RASPI_RESET" library="SparkFun-Switches" deviceset="MOMENTARY-SWITCH-SPST-2" device="-SMD-5.2MM"/>
-<part name="JP1" library="pinhead" deviceset="PINHD-1X14" device=""/>
 <part name="GND4" library="supply1" library_urn="urn:adsk.eagle:library:371" deviceset="GND" device=""/>
+<part name="X1" library="Rembrandt Electronics - JST XH Connectors v1-0" deviceset="JST-XH-02-PIN" device="-ROUND-PAD"/>
+<part name="GND5" library="supply1" library_urn="urn:adsk.eagle:library:371" deviceset="GND" device=""/>
+<part name="JP5" library="pinhead" deviceset="PINHD-1X16" device=""/>
 </parts>
 <sheets>
@@
 <attribute name="NAME" x="125.73" y="65.024" size="1.778" layer="95" font="vector"/>
 </instance>
-<instance part="GND3" gate="1" x="171.45" y="52.07" smashed="yes">
-<attribute name="VALUE" x="168.91" y="49.53" size="1.778" layer="96"/>
+<instance part="GND3" gate="1" x="171.45" y="46.99" smashed="yes">
+<attribute name="VALUE" x="168.91" y="44.45" size="1.778" layer="96"/>
 </instance>
 <instance part="R1" gate="G$1" x="76.2" y="76.2" smashed="yes">
@@
 <attribute name="VALUE" x="29.21" y="13.716" size="1.778" layer="96" font="vector" align="top-center"/>
 </instance>
-<instance part="JP1" gate="A" x="180.34" y="73.66" smashed="yes">
-<attribute name="NAME" x="173.99" y="92.075" size="1.778" layer="95"/>
-<attribute name="VALUE" x="173.99" y="50.8" size="1.778" layer="96"/>
-</instance>
 <instance part="GND4" gate="1" x="27.94" y="96.52" smashed="yes">
 <attribute name="VALUE" x="25.4" y="93.98" size="1.778" layer="96"/>
+</instance>
+<instance part="X1" gate="-2" x="157.48" y="30.48" smashed="yes">
+<attribute name="NAME" x="160.02" y="29.718" size="1.524" layer="95"/>
+</instance>
+<instance part="X1" gate="-1" x="157.48" y="33.02" smashed="yes">
+<attribute name="NAME" x="160.02" y="32.258" size="1.524" layer="95"/>
+<attribute name="VALUE" x="156.718" y="34.417" size="1.778" layer="96"/>
+</instance>
+<instance part="GND5" gate="1" x="152.4" y="20.32" smashed="yes">
+<attribute name="VALUE" x="149.86" y="17.78" size="1.778" layer="96"/>
+</instance>
+<instance part="JP5" gate="A" x="180.34" y="71.12" smashed="yes">
+<attribute name="NAME" x="173.99" y="92.075" size="1.778" layer="95"/>
+<attribute name="VALUE" x="173.99" y="45.72" size="1.778" layer="96"/>
 </instance>
 </instances>
@@
 </segment>
 <segment>
-<wire x1="177.8" y1="63.5" x2="171.45" y2="63.5" width="0.1524" layer="91"/>
-<wire x1="171.45" y1="63.5" x2="171.45" y2="54.61" width="0.1524" layer="91"/>
+<wire x1="177.8" y1="58.42" x2="171.45" y2="58.42" width="0.1524" layer="91"/>
+<wire x1="171.45" y1="58.42" x2="171.45" y2="49.53" width="0.1524" layer="91"/>
 <pinref part="GND3" gate="1" pin="GND"/>
-<pinref part="JP1" gate="A" pin="11"/>
+<pinref part="JP5" gate="A" pin="13"/>
+<pinref part="JP5" gate="A" pin="12"/>
+<wire x1="177.8" y1="60.96" x2="171.45" y2="60.96" width="0.1524" layer="91"/>
+<wire x1="171.45" y1="60.96" x2="171.45" y2="58.42" width="0.1524" layer="91"/>
+<junction x="171.45" y="58.42"/>
 </segment>
 <segment>
@@
 <wire x1="27.94" y1="104.14" x2="27.94" y2="99.06" width="0.1524" layer="91"/>
 </segment>
+<segment>
+<pinref part="X1" gate="-1" pin="S"/>
+<wire x1="154.94" y1="33.02" x2="152.4" y2="33.02" width="0.1524" layer="91"/>
+<wire x1="152.4" y1="33.02" x2="152.4" y2="22.86" width="0.1524" layer="91"/>
+<pinref part="GND5" gate="1" pin="GND"/>
+</segment>
 </net>
 <net name="IR_RESET" class="0">
@@
 <wire x1="177.8" y1="68.58" x2="171.45" y2="68.58" width="0.1524" layer="91"/>
 <label x="171.45" y="68.58" size="1.778" layer="95" rot="R180" xref="yes"/>
-<pinref part="JP1" gate="A" pin="9"/>
+<pinref part="JP5" gate="A" pin="9"/>
 </segment>
 </net>
@@
 <wire x1="177.8" y1="88.9" x2="171.45" y2="88.9" width="0.1524" layer="91"/>
 <label x="171.45" y="88.9" size="1.778" layer="95" rot="R180" xref="yes"/>
-<pinref part="JP1" gate="A" pin="1"/>
+<pinref part="JP5" gate="A" pin="1"/>
 </segment>
 </net>
@@
 <wire x1="177.8" y1="86.36" x2="151.13" y2="86.36" width="0.1524" layer="91"/>
 <label x="151.13" y="86.36" size="1.778" layer="95" rot="R180" xref="yes"/>
-<pinref part="JP1" gate="A" pin="2"/>
+<pinref part="JP5" gate="A" pin="2"/>
 </segment>
 </net>
@@
 <wire x1="177.8" y1="78.74" x2="171.45" y2="78.74" width="0.1524" layer="91"/>
 <label x="171.45" y="78.74" size="1.778" layer="95" rot="R180" xref="yes"/>
-<pinref part="JP1" gate="A" pin="5"/>
+<pinref part="JP5" gate="A" pin="5"/>
 </segment>
 </net>
@@
 <wire x1="177.8" y1="76.2" x2="151.13" y2="76.2" width="0.1524" layer="91"/>
 <label x="151.13" y="76.2" size="1.778" layer="95" rot="R180" xref="yes"/>
-<pinref part="JP1" gate="A" pin="6"/>
+<pinref part="JP5" gate="A" pin="6"/>
 </segment>
 </net>
@@
 <wire x1="177.8" y1="83.82" x2="171.45" y2="83.82" width="0.1524" layer="91"/>
 <label x="171.45" y="83.82" size="1.778" layer="95" rot="R180" xref="yes"/>
-<pinref part="JP1" gate="A" pin="3"/>
+<pinref part="JP5" gate="A" pin="3"/>
 </segment>
 </net>
@@
 <wire x1="177.8" y1="71.12" x2="151.13" y2="71.12" width="0.1524" layer="91"/>
 <label x="151.13" y="71.12" size="1.778" layer="95" rot="R180" xref="yes"/>
-<pinref part="JP1" gate="A" pin="8"/>
+<pinref part="JP5" gate="A" pin="8"/>
 </segment>
 </net>
@@
 <wire x1="177.8" y1="81.28" x2="151.13" y2="81.28" width="0.1524" layer="91"/>
 <label x="151.13" y="81.28" size="1.778" layer="95" rot="R180" xref="yes"/>
-<pinref part="JP1" gate="A" pin="4"/>
+<pinref part="JP5" gate="A" pin="4"/>
 </segment>
 </net>
@@
 <wire x1="177.8" y1="73.66" x2="171.45" y2="73.66" width="0.1524" layer="91"/>
 <label x="171.45" y="73.66" size="1.778" layer="95" rot="R180" xref="yes"/>
-<pinref part="JP1" gate="A" pin="7"/>
+<pinref part="JP5" gate="A" pin="7"/>
 </segment>
 </net>
@@
 </segment>
 <segment>
-<pinref part="JP1" gate="A" pin="10"/>
 <wire x1="177.8" y1="66.04" x2="152.4" y2="66.04" width="0.1524" layer="91"/>
 <label x="152.4" y="66.04" size="1.778" layer="95" rot="R180" xref="yes"/>
+<pinref part="JP5" gate="A" pin="10"/>
 </segment>
 </net>
@@
 </segment>
 <segment>
-<pinref part="JP1" gate="A" pin="13"/>
-<wire x1="177.8" y1="58.42" x2="152.4" y2="58.42" width="0.1524" layer="91"/>
-<label x="152.4" y="58.42" size="1.778" layer="95" rot="R180" xref="yes"/>
+<wire x1="177.8" y1="53.34" x2="152.4" y2="53.34" width="0.1524" layer="91"/>
+<label x="152.4" y="53.34" size="1.778" layer="95" rot="R180" xref="yes"/>
+<pinref part="JP5" gate="A" pin="15"/>
 </segment>
 </net>
@@
 </segment>
 <segment>
-<pinref part="JP1" gate="A" pin="12"/>
-<wire x1="177.8" y1="60.96" x2="170.18" y2="60.96" width="0.1524" layer="91"/>
-<label x="170.18" y="60.96" size="1.778" layer="95" rot="R180" xref="yes"/>
-</segment>
-</net>
-<net name="UVCC" class="0">
-<segment>
-<pinref part="JP1" gate="A" pin="14"/>
 <wire x1="177.8" y1="55.88" x2="170.18" y2="55.88" width="0.1524" layer="91"/>
 <label x="170.18" y="55.88" size="1.778" layer="95" rot="R180" xref="yes"/>
+<pinref part="JP5" gate="A" pin="14"/>
+</segment>
+</net>
+<net name="UVCC" class="0">
+<segment>
+<wire x1="177.8" y1="50.8" x2="170.18" y2="50.8" width="0.1524" layer="91"/>
+<label x="170.18" y="50.8" size="1.778" layer="95" rot="R180" xref="yes"/>
+<pinref part="JP5" gate="A" pin="16"/>
 </segment>
 <segment>
@@
 </segment>
 </net>
+<net name="SWITCH" class="0">
+<segment>
+<pinref part="X1" gate="-2" pin="S"/>
+<wire x1="154.94" y1="30.48" x2="147.32" y2="30.48" width="0.1524" layer="91"/>
+<label x="147.32" y="30.48" size="1.778" layer="95" rot="R180" xref="yes"/>
+</segment>
+<segment>
+<pinref part="JP5" gate="A" pin="11"/>
+<wire x1="177.8" y1="63.5" x2="172.72" y2="63.5" width="0.1524" layer="91"/>
+<label x="172.72" y="63.5" size="1.778" layer="95" rot="R180" xref="yes"/>
+</segment>
+</net>
