File: board/mainboard/untitled.sch (EAGLE design)
At the start: 41 parts, among them X1 JST-XH-03-PIN-ROUND-PAD, X2 JST-XH-04-PIN-ROUND-PAD, X3 JST-XH-02-PIN-ROUND-PAD, X4 JST-XH-02-PIN-ROUND-PAD, X5 JST-XH-02-PIN-ROUND-PAD

Commit message: Revert "Merge remote-tracking branch 'origin/Develop' into feature_#37"
This reverts commit cb103155361e8766478c6830db153463370c0739, reversing
changes made to 84e093fe944e1f8653a6822ff34e6f8740617cb5.
Parts:
- removed JP7: (no value), pinhead:PINHD-2X7
- added JP5: (no value), pinhead:PINHD-2X6
Connections:
- removed net TRIM: JP7.14, U$1.A16/40
- net +3V3: no longer JP7.13
- net GND: now also JP5.2; no longer JP7.2
- net GYRO_RESET: now also JP5.1; no longer JP7.1
- net IR_RESET: now also JP5.9; no longer JP7.9
- net LED1: now also JP5.4; no longer JP7.4
- net LED2: now also JP5.6; no longer JP7.6
- net LED3: now also JP5.5; no longer JP7.5
- net LED4: now also JP5.7; no longer JP7.7
- net LED5: now also JP5.8; no longer JP7.8
- net LED6: now also JP5.10; no longer JP7.10
- net MAIN_RESET: now also JP5.11; no longer JP7.11
- net RASPI_RESET: now also JP5.12; no longer JP7.12
- net SWITCH: now also JP5.3; no longer JP7.3
Changed lines of the file:
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@@
 <?xml version="1.0" encoding="utf-8"?>
 <!DOCTYPE eagle SYSTEM "eagle.dtd">
-<eagle version="9.6.2">
+<eagle version="9.6.1">
 <drawing>
 <settings>
@@
 <part name="GND14" library="supply1" library_urn="urn:adsk.eagle:library:371" deviceset="GND" device=""/>
 <part name="P+14" library="supply1" library_urn="urn:adsk.eagle:library:371" deviceset="+5V" device=""/>
+<part name="JP5" library="pinhead" deviceset="PINHD-2X6" device=""/>
 <part name="GND15" library="supply1" library_urn="urn:adsk.eagle:library:371" deviceset="GND" device=""/>
-<part name="JP7" library="pinhead" deviceset="PINHD-2X7" device=""/>
-<part name="+3V9" library="supply1" library_urn="urn:adsk.eagle:library:371" deviceset="+3V3" device=""/>
 </parts>
 <sheets>
@@
 <attribute name="VALUE" x="-76.2" y="-45.72" size="1.778" layer="96" rot="R90"/>
 </instance>
+<instance part="JP5" gate="A" x="25.4" y="-7.62" smashed="yes">
+<attribute name="NAME" x="19.05" y="0.635" size="1.778" layer="95"/>
+<attribute name="VALUE" x="19.05" y="-20.32" size="1.778" layer="96"/>
+</instance>
 <instance part="GND15" gate="1" x="35.56" y="-22.86" smashed="yes">
 <attribute name="VALUE" x="33.02" y="-25.4" size="1.778" layer="96"/>
-</instance>
-<instance part="JP7" gate="A" x="25.4" y="-10.16" smashed="yes">
-<attribute name="NAME" x="19.05" y="0.635" size="1.778" layer="95"/>
-<attribute name="VALUE" x="19.05" y="-22.86" size="1.778" layer="96"/>
-</instance>
-<instance part="+3V9" gate="G$1" x="15.24" y="5.08" smashed="yes">
-<attribute name="VALUE" x="12.7" y="0" size="1.778" layer="96" rot="R90"/>
 </instance>
 </instances>
@@
 </segment>
 <segment>
+<pinref part="JP5" gate="A" pin="2"/>
 <wire x1="30.48" y1="-2.54" x2="35.56" y2="-2.54" width="0.1524" layer="91"/>
 <wire x1="35.56" y1="-2.54" x2="35.56" y2="-20.32" width="0.1524" layer="91"/>
 <pinref part="GND15" gate="1" pin="GND"/>
-<pinref part="JP7" gate="A" pin="2"/>
 </segment>
 </net>
@@
 <pinref part="+3V8" gate="G$1" pin="+3V3"/>
 </segment>
-<segment>
-<pinref part="JP7" gate="A" pin="13"/>
-<wire x1="22.86" y1="-17.78" x2="15.24" y2="-17.78" width="0.1524" layer="91"/>
-<wire x1="15.24" y1="-17.78" x2="15.24" y2="2.54" width="0.1524" layer="91"/>
-<pinref part="+3V9" gate="G$1" pin="+3V3"/>
-</segment>
 </net>
 <net name="LINE_LED" class="0">
@@
 </segment>
 <segment>
-<wire x1="22.86" y1="-12.7" x2="-12.7" y2="-12.7" width="0.1524" layer="91"/>
-<label x="-12.7" y="-12.7" size="1.778" layer="95" rot="R180" xref="yes"/>
-<pinref part="JP7" gate="A" pin="9"/>
+<pinref part="JP5" gate="A" pin="9"/>
+<wire x1="22.86" y1="-12.7" x2="-2.54" y2="-12.7" width="0.1524" layer="91"/>
+<label x="-2.54" y="-12.7" size="1.778" layer="95" rot="R180" xref="yes"/>
 </segment>
 </net>
@@
 </segment>
 <segment>
-<wire x1="22.86" y1="-2.54" x2="7.62" y2="-2.54" width="0.1524" layer="91"/>
-<label x="7.62" y="-2.54" size="1.778" layer="95" rot="R180" xref="yes"/>
-<pinref part="JP7" gate="A" pin="1"/>
+<wire x1="22.86" y1="-2.54" x2="17.78" y2="-2.54" width="0.1524" layer="91"/>
+<label x="17.78" y="-2.54" size="1.778" layer="95" rot="R180" xref="yes"/>
+<pinref part="JP5" gate="A" pin="1"/>
 </segment>
 </net>
@@
 <wire x1="30.48" y1="-5.08" x2="48.26" y2="-5.08" width="0.1524" layer="91"/>
 <label x="48.26" y="-5.08" size="1.778" layer="95" xref="yes"/>
-<pinref part="JP7" gate="A" pin="4"/>
+<pinref part="JP5" gate="A" pin="4"/>
 </segment>
 </net>
@@
 <wire x1="30.48" y1="-7.62" x2="38.1" y2="-7.62" width="0.1524" layer="91"/>
 <label x="38.1" y="-7.62" size="1.778" layer="95" xref="yes"/>
-<pinref part="JP7" gate="A" pin="6"/>
+<pinref part="JP5" gate="A" pin="6"/>
 </segment>
 </net>
@@
 </segment>
 <segment>
-<wire x1="22.86" y1="-7.62" x2="7.62" y2="-7.62" width="0.1524" layer="91"/>
-<label x="7.62" y="-7.62" size="1.778" layer="95" rot="R180" xref="yes"/>
-<pinref part="JP7" gate="A" pin="5"/>
+<pinref part="JP5" gate="A" pin="5"/>
+<wire x1="22.86" y1="-7.62" x2="17.78" y2="-7.62" width="0.1524" layer="91"/>
+<label x="17.78" y="-7.62" size="1.778" layer="95" rot="R180" xref="yes"/>
 </segment>
 </net>
@@
 </segment>
 <segment>
+<pinref part="JP5" gate="A" pin="12"/>
 <wire x1="30.48" y1="-15.24" x2="48.26" y2="-15.24" width="0.1524" layer="91"/>
 <label x="48.26" y="-15.24" size="1.778" layer="95" xref="yes"/>
-<pinref part="JP7" gate="A" pin="12"/>
 </segment>
 </net>
@@
 </segment>
 <segment>
-<wire x1="22.86" y1="-10.16" x2="-2.54" y2="-10.16" width="0.1524" layer="91"/>
-<label x="-2.54" y="-10.16" size="1.778" layer="95" rot="R180" xref="yes"/>
-<pinref part="JP7" gate="A" pin="7"/>
+<pinref part="JP5" gate="A" pin="7"/>
+<wire x1="22.86" y1="-10.16" x2="7.62" y2="-10.16" width="0.1524" layer="91"/>
+<label x="7.62" y="-10.16" size="1.778" layer="95" rot="R180" xref="yes"/>
 </segment>
 </net>
@@
 </segment>
 <segment>
+<pinref part="JP5" gate="A" pin="8"/>
 <wire x1="30.48" y1="-10.16" x2="48.26" y2="-10.16" width="0.1524" layer="91"/>
 <label x="48.26" y="-10.16" size="1.778" layer="95" xref="yes"/>
-<pinref part="JP7" gate="A" pin="8"/>
 </segment>
 </net>
@@
 </segment>
 <segment>
-<wire x1="22.86" y1="-5.08" x2="-12.7" y2="-5.08" width="0.1524" layer="91"/>
-<label x="-12.7" y="-5.08" size="1.778" layer="95" rot="R180" xref="yes"/>
-<pinref part="JP7" gate="A" pin="3"/>
+<pinref part="JP5" gate="A" pin="3"/>
+<wire x1="22.86" y1="-5.08" x2="-2.54" y2="-5.08" width="0.1524" layer="91"/>
+<label x="-2.54" y="-5.08" size="1.778" layer="95" rot="R180" xref="yes"/>
 </segment>
 </net>
 <net name="LED6" class="0">
 <segment>
+<pinref part="JP5" gate="A" pin="10"/>
 <wire x1="30.48" y1="-12.7" x2="38.1" y2="-12.7" width="0.1524" layer="91"/>
 <label x="38.1" y="-12.7" size="1.778" layer="95" xref="yes"/>
-<pinref part="JP7" gate="A" pin="10"/>
 </segment>
 <segment>
@@
 </segment>
 <segment>
-<wire x1="22.86" y1="-15.24" x2="7.62" y2="-15.24" width="0.1524" layer="91"/>
-<label x="7.62" y="-15.24" size="1.778" layer="95" rot="R180" xref="yes"/>
-<pinref part="JP7" gate="A" pin="11"/>
-</segment>
-</net>
-<net name="TRIM" class="0">
-<segment>
-<pinref part="JP7" gate="A" pin="14"/>
-<wire x1="30.48" y1="-17.78" x2="38.1" y2="-17.78" width="0.1524" layer="91"/>
-<label x="38.1" y="-17.78" size="1.778" layer="95" xref="yes"/>
-</segment>
-<segment>
-<pinref part="U$1" gate="G$1" pin="A16/40"/>
-<wire x1="58.42" y1="40.64" x2="81.28" y2="40.64" width="0.1524" layer="91"/>
-<label x="81.28" y="40.64" size="1.778" layer="95" xref="yes"/>
-</segment>
-</net>
+<pinref part="JP5" gate="A" pin="11"/>
+<wire x1="22.86" y1="-15.24" x2="17.78" y2="-15.24" width="0.1524" layer="91"/>
+<label x="17.78" y="-15.24" size="1.778" layer="95" rot="R180" xref="yes"/>
+</segment>
+</net>
