File: board/mainboard/untitled.sch (EAGLE design)
At the start: 38 parts, among them X1 JST-XH-03-PIN-ROUND-PAD, X2 JST-XH-04-PIN-ROUND-PAD, X3 JST-XH-02-PIN-ROUND-PAD

Commit message: 作業PCの変更
Parts:
- added JP6: (no value), pinhead:PINHD-2X7
- added X4: JST-XH-02-PIN-ROUND-PAD, Rembrandt Electronics - JST XH Connectors v1-0:JST-XH-02-PIN-ROUND-PAD
Connections:
- new net KICK: U$1.A8/22, X4-2.S
- net GND: now also X4-1.S
Changed lines of the file:
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@@
 <?xml version="1.0" encoding="utf-8"?>
 <!DOCTYPE eagle SYSTEM "eagle.dtd">
-<eagle version="9.6.1">
+<eagle version="9.6.2">
 <drawing>
 <settings>
@@
 <setting verticaltext="up"/>
 </settings>
-<grid distance="0.1" unitdist="inch" unit="inch" style="lines" multiple="1" display="no" altdistance="0.05" altunitdist="inch" altunit="inch"/>
+<grid distance="0.1" unitdist="inch" unit="inch" style="lines" multiple="1" display="no" altdistance="0.01" altunitdist="inch" altunit="inch"/>
 <layers>
 <layer number="1" name="Top" color="4" fill="1" visible="no" active="no"/>
@@
 <part name="JP4" library="pinhead" deviceset="PINHD-1X4" device=""/>
 <part name="GND12" library="supply1" library_urn="urn:adsk.eagle:library:371" deviceset="GND" device=""/>
+<part name="X4" library="Rembrandt Electronics - JST XH Connectors v1-0" deviceset="JST-XH-02-PIN" device="-ROUND-PAD"/>
+<part name="GND13" library="supply1" library_urn="urn:adsk.eagle:library:371" deviceset="GND" device=""/>
+<part name="JP6" library="pinhead" deviceset="PINHD-2X7" device=""/>
 </parts>
 <sheets>
@@
 <attribute name="VALUE" x="60.96" y="86.36" size="1.778" layer="96" rot="R90"/>
 </instance>
-<instance part="GND1" gate="1" x="76.2" y="73.66" smashed="yes">
-<attribute name="VALUE" x="73.66" y="71.12" size="1.778" layer="96"/>
+<instance part="GND1" gate="1" x="76.2" y="7.62" smashed="yes">
+<attribute name="VALUE" x="73.66" y="5.08" size="1.778" layer="96"/>
 </instance>
 <instance part="RASPI" gate="G$1" x="-73.66" y="53.34" smashed="yes" rot="R180">
@@
 <instance part="GND12" gate="1" x="10.16" y="-55.88" smashed="yes">
 <attribute name="VALUE" x="7.62" y="-58.42" size="1.778" layer="96"/>
+</instance>
+<instance part="X4" gate="-2" x="83.82" y="-30.48" smashed="yes">
+<attribute name="NAME" x="86.36" y="-31.242" size="1.524" layer="95"/>
+</instance>
+<instance part="X4" gate="-1" x="83.82" y="-27.94" smashed="yes">
+<attribute name="NAME" x="86.36" y="-28.702" size="1.524" layer="95"/>
+<attribute name="VALUE" x="83.058" y="-26.543" size="1.778" layer="96"/>
+</instance>
+<instance part="GND13" gate="1" x="78.74" y="-40.64" smashed="yes">
+<attribute name="VALUE" x="76.2" y="-43.18" size="1.778" layer="96"/>
+</instance>
+<instance part="JP6" gate="A" x="60.96" y="-137.16" smashed="yes">
+<attribute name="NAME" x="54.61" y="-126.365" size="1.778" layer="95"/>
+<attribute name="VALUE" x="54.61" y="-149.86" size="1.778" layer="96"/>
 </instance>
 </instances>
@@
 <pinref part="U$1" gate="G$1" pin="GND"/>
 <wire x1="58.42" y1="78.74" x2="76.2" y2="78.74" width="0.1524" layer="91"/>
-<wire x1="76.2" y1="78.74" x2="76.2" y2="76.2" width="0.1524" layer="91"/>
+<wire x1="76.2" y1="78.74" x2="76.2" y2="10.16" width="0.1524" layer="91"/>
 <pinref part="GND1" gate="1" pin="GND"/>
 </segment>
@@
 <pinref part="GND12" gate="1" pin="GND"/>
 </segment>
+<segment>
+<pinref part="X4" gate="-1" pin="S"/>
+<wire x1="81.28" y1="-27.94" x2="78.74" y2="-27.94" width="0.1524" layer="91"/>
+<wire x1="78.74" y1="-27.94" x2="78.74" y2="-38.1" width="0.1524" layer="91"/>
+<pinref part="GND13" gate="1" pin="GND"/>
+</segment>
 </net>
 <net name="+5V" class="0">
@@
 </segment>
 </net>
+<net name="KICK" class="0">
+<segment>
+<pinref part="X4" gate="-2" pin="S"/>
+<wire x1="81.28" y1="-30.48" x2="73.66" y2="-30.48" width="0.1524" layer="91"/>
+<label x="73.66" y="-30.48" size="1.778" layer="95" rot="R180" xref="yes"/>
+</segment>
+<segment>
+<pinref part="U$1" gate="G$1" pin="A8/22"/>
+<wire x1="58.42" y1="71.12" x2="68.58" y2="71.12" width="0.1524" layer="91"/>
+<label x="68.58" y="71.12" size="1.778" layer="95" xref="yes"/>
+</segment>
+</net>

Commit message: complete mainboard
Parts:
- removed JP6: (no value), pinhead:PINHD-2X7
- added JP5: (no value), pinhead:PINHD-2X6
- added X5: JST-XH-02-PIN-ROUND-PAD, Rembrandt Electronics - JST XH Connectors v1-0:JST-XH-02-PIN-ROUND-PAD
Connections:
- new net LED1: JP5.4, U$1.3
- new net LED2: JP5.6, U$1.2
- new net LED3: JP5.5, U$1.A4/18
- new net LED4: JP5.7, U$1.A5/19
- new net LED5: JP5.8, U$1.A8/22
- new net LED6: JP5.10, U$1.33
- new net MAIN_RESET: JP5.11, U$1.36
- new net RASPI_RESET: JP5.12, RASPI.5
- new net SWITCH: JP5.3, U$1.A17/41
- net +5V: now also X5-2.S
- net GND: now also JP5.2, X5-1.S
- net GYRO_RESET: now also JP5.1
- net GYRO_RX: now also U$1.29/TX7
- net GYRO_TX: now also U$1.28/RX7
- net IR_RESET: now also JP5.9
- net KICK: now also U$1.A9/23; no longer U$1.A8/22
- net MD3_RX: now also U$1.8/TX2; no longer U$1.24/A10/TX6
- net MD3_TX: now also U$1.7/RX2; no longer U$1.25/A11/RX6
- net MD4_RX: now also U$1.24/A10/TX6; no longer U$1.29/TX7
- net MD4_TX: now also U$1.25/A11/RX6; no longer U$1.28/RX7
Other:
- moved on the sheet: JP1, JP2, JP3, JP4

Commit message: marge前のファイル
Parts:
- removed JP5: (no value), pinhead:PINHD-2X6
- added JP7: (no value), pinhead:PINHD-2X7
Connections:
- new net TRIM: JP7.14, U$1.A16/40
- net +3V3: now also JP7.13
- net GND: now also JP7.2; no longer JP5.2
- net GYRO_RESET: now also JP7.1; no longer JP5.1
- net IR_RESET: now also JP7.9; no longer JP5.9
- net LED1: now also JP7.4; no longer JP5.4
- net LED2: now also JP7.6; no longer JP5.6
- net LED3: now also JP7.5; no longer JP5.5
- net LED4: now also JP7.7; no longer JP5.7
- net LED5: now also JP7.8; no longer JP5.8
- net LED6: now also JP7.10; no longer JP5.10
- net MAIN_RESET: now also JP7.11; no longer JP5.11
- net RASPI_RESET: now also JP7.12; no longer JP5.12
- net SWITCH: now also JP7.3; no longer JP5.3
Changed lines of the file:
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@@
 <?xml version="1.0" encoding="utf-8"?>
 <!DOCTYPE eagle SYSTEM "eagle.dtd">
-<eagle version="9.6.1">
+<eagle version="9.6.2">
 <drawing>
 <settings>
@@
 <part name="GND14" library="supply1" library_urn="urn:adsk.eagle:library:371" deviceset="GND" device=""/>
 <part name="P+14" library="supply1" library_urn="urn:adsk.eagle:library:371" deviceset="+5V" device=""/>
-<part name="JP5" library="pinhead" deviceset="PINHD-2X6" device=""/>
 <part name="GND15" library="supply1" library_urn="urn:adsk.eagle:library:371" deviceset="GND" device=""/>
+<part name="JP7" library="pinhead" deviceset="PINHD-2X7" device=""/>
+<part name="+3V9" library="supply1" library_urn="urn:adsk.eagle:library:371" deviceset="+3V3" device=""/>
 </parts>
 <sheets>
@@
 <attribute name="VALUE" x="-76.2" y="-45.72" size="1.778" layer="96" rot="R90"/>
 </instance>
-<instance part="JP5" gate="A" x="25.4" y="-7.62" smashed="yes">
-<attribute name="NAME" x="19.05" y="0.635" size="1.778" layer="95"/>
-<attribute name="VALUE" x="19.05" y="-20.32" size="1.778" layer="96"/>
-</instance>
 <instance part="GND15" gate="1" x="35.56" y="-22.86" smashed="yes">
 <attribute name="VALUE" x="33.02" y="-25.4" size="1.778" layer="96"/>
+</instance>
+<instance part="JP7" gate="A" x="25.4" y="-10.16" smashed="yes">
+<attribute name="NAME" x="19.05" y="0.635" size="1.778" layer="95"/>
+<attribute name="VALUE" x="19.05" y="-22.86" size="1.778" layer="96"/>
+</instance>
+<instance part="+3V9" gate="G$1" x="15.24" y="5.08" smashed="yes">
+<attribute name="VALUE" x="12.7" y="0" size="1.778" layer="96" rot="R90"/>
 </instance>
 </instances>
@@
 </segment>
 <segment>
-<pinref part="JP5" gate="A" pin="2"/>
 <wire x1="30.48" y1="-2.54" x2="35.56" y2="-2.54" width="0.1524" layer="91"/>
 <wire x1="35.56" y1="-2.54" x2="35.56" y2="-20.32" width="0.1524" layer="91"/>
 <pinref part="GND15" gate="1" pin="GND"/>
+<pinref part="JP7" gate="A" pin="2"/>
 </segment>
 </net>
@@
 <pinref part="+3V8" gate="G$1" pin="+3V3"/>
 </segment>
+<segment>
+<pinref part="JP7" gate="A" pin="13"/>
+<wire x1="22.86" y1="-17.78" x2="15.24" y2="-17.78" width="0.1524" layer="91"/>
+<wire x1="15.24" y1="-17.78" x2="15.24" y2="2.54" width="0.1524" layer="91"/>
+<pinref part="+3V9" gate="G$1" pin="+3V3"/>
+</segment>
 </net>
 <net name="LINE_LED" class="0">
@@
 </segment>
 <segment>
-<pinref part="JP5" gate="A" pin="9"/>
-<wire x1="22.86" y1="-12.7" x2="-2.54" y2="-12.7" width="0.1524" layer="91"/>
-<label x="-2.54" y="-12.7" size="1.778" layer="95" rot="R180" xref="yes"/>
+<wire x1="22.86" y1="-12.7" x2="-12.7" y2="-12.7" width="0.1524" layer="91"/>
+<label x="-12.7" y="-12.7" size="1.778" layer="95" rot="R180" xref="yes"/>
+<pinref part="JP7" gate="A" pin="9"/>
 </segment>
 </net>
@@
 </segment>
 <segment>
-<wire x1="22.86" y1="-2.54" x2="17.78" y2="-2.54" width="0.1524" layer="91"/>
-<label x="17.78" y="-2.54" size="1.778" layer="95" rot="R180" xref="yes"/>
-<pinref part="JP5" gate="A" pin="1"/>
+<wire x1="22.86" y1="-2.54" x2="7.62" y2="-2.54" width="0.1524" layer="91"/>
+<label x="7.62" y="-2.54" size="1.778" layer="95" rot="R180" xref="yes"/>
+<pinref part="JP7" gate="A" pin="1"/>
 </segment>
 </net>
@@
 <wire x1="30.48" y1="-5.08" x2="48.26" y2="-5.08" width="0.1524" layer="91"/>
 <label x="48.26" y="-5.08" size="1.778" layer="95" xref="yes"/>
-<pinref part="JP5" gate="A" pin="4"/>
+<pinref part="JP7" gate="A" pin="4"/>
 </segment>
 </net>
@@
 <wire x1="30.48" y1="-7.62" x2="38.1" y2="-7.62" width="0.1524" layer="91"/>
 <label x="38.1" y="-7.62" size="1.778" layer="95" xref="yes"/>
-<pinref part="JP5" gate="A" pin="6"/>
+<pinref part="JP7" gate="A" pin="6"/>
 </segment>
 </net>
@@
 </segment>
 <segment>
-<pinref part="JP5" gate="A" pin="5"/>
-<wire x1="22.86" y1="-7.62" x2="17.78" y2="-7.62" width="0.1524" layer="91"/>
-<label x="17.78" y="-7.62" size="1.778" layer="95" rot="R180" xref="yes"/>
+<wire x1="22.86" y1="-7.62" x2="7.62" y2="-7.62" width="0.1524" layer="91"/>
+<label x="7.62" y="-7.62" size="1.778" layer="95" rot="R180" xref="yes"/>
+<pinref part="JP7" gate="A" pin="5"/>
 </segment>
 </net>
@@
 </segment>
 <segment>
-<pinref part="JP5" gate="A" pin="12"/>
 <wire x1="30.48" y1="-15.24" x2="48.26" y2="-15.24" width="0.1524" layer="91"/>
 <label x="48.26" y="-15.24" size="1.778" layer="95" xref="yes"/>
+<pinref part="JP7" gate="A" pin="12"/>
 </segment>
 </net>
@@
 </segment>
 <segment>
-<pinref part="JP5" gate="A" pin="7"/>
-<wire x1="22.86" y1="-10.16" x2="7.62" y2="-10.16" width="0.1524" layer="91"/>
-<label x="7.62" y="-10.16" size="1.778" layer="95" rot="R180" xref="yes"/>
+<wire x1="22.86" y1="-10.16" x2="-2.54" y2="-10.16" width="0.1524" layer="91"/>
+<label x="-2.54" y="-10.16" size="1.778" layer="95" rot="R180" xref="yes"/>
+<pinref part="JP7" gate="A" pin="7"/>
 </segment>
 </net>
@@
 </segment>
 <segment>
-<pinref part="JP5" gate="A" pin="8"/>
 <wire x1="30.48" y1="-10.16" x2="48.26" y2="-10.16" width="0.1524" layer="91"/>
 <label x="48.26" y="-10.16" size="1.778" layer="95" xref="yes"/>
+<pinref part="JP7" gate="A" pin="8"/>
 </segment>
 </net>
@@
 </segment>
 <segment>
-<pinref part="JP5" gate="A" pin="3"/>
-<wire x1="22.86" y1="-5.08" x2="-2.54" y2="-5.08" width="0.1524" layer="91"/>
-<label x="-2.54" y="-5.08" size="1.778" layer="95" rot="R180" xref="yes"/>
+<wire x1="22.86" y1="-5.08" x2="-12.7" y2="-5.08" width="0.1524" layer="91"/>
+<label x="-12.7" y="-5.08" size="1.778" layer="95" rot="R180" xref="yes"/>
+<pinref part="JP7" gate="A" pin="3"/>
 </segment>
 </net>
 <net name="LED6" class="0">
 <segment>
-<pinref part="JP5" gate="A" pin="10"/>
 <wire x1="30.48" y1="-12.7" x2="38.1" y2="-12.7" width="0.1524" layer="91"/>
 <label x="38.1" y="-12.7" size="1.778" layer="95" xref="yes"/>
+<pinref part="JP7" gate="A" pin="10"/>
 </segment>
 <segment>
@@
 </segment>
 <segment>
-<pinref part="JP5" gate="A" pin="11"/>
-<wire x1="22.86" y1="-15.24" x2="17.78" y2="-15.24" width="0.1524" layer="91"/>
-<label x="17.78" y="-15.24" size="1.778" layer="95" rot="R180" xref="yes"/>
-</segment>
-</net>
+<wire x1="22.86" y1="-15.24" x2="7.62" y2="-15.24" width="0.1524" layer="91"/>
+<label x="7.62" y="-15.24" size="1.778" layer="95" rot="R180" xref="yes"/>
+<pinref part="JP7" gate="A" pin="11"/>
+</segment>
+</net>
+<net name="TRIM" class="0">
+<segment>
+<pinref part="JP7" gate="A" pin="14"/>
+<wire x1="30.48" y1="-17.78" x2="38.1" y2="-17.78" width="0.1524" layer="91"/>
+<label x="38.1" y="-17.78" size="1.778" layer="95" xref="yes"/>
+</segment>
+<segment>
+<pinref part="U$1" gate="G$1" pin="A16/40"/>
+<wire x1="58.42" y1="40.64" x2="81.28" y2="40.64" width="0.1524" layer="91"/>
+<label x="81.28" y="40.64" size="1.778" layer="95" xref="yes"/>
+</segment>
+</net>
