File: board/line_sensor_test/long/untitled.brd (EAGLE design)
At the start: 1317.6 x 228.6 mm, 15 parts

Commit message: 配線おわり
Parts:
- added JP2: 11PIN, jst_eph:B11B-PH-K-S
- moved R3 127.2 mm to (62.0, 2.56), flipped to the bottom
- moved R2 124.5 mm to (74.0, 2.54), flipped to the bottom
- moved R1 122.1 mm to (83.2, 2.16), flipped to the bottom
Connections:
- removed net N$10: R1.1, U$4.E
- removed net N$11: R3.1, U$5.E
- removed net N$4: LED1.A, LED2.A, LED3.A
- removed net N$8: LED4.1-VDD, LED5.1-VDD, LED6.1-VDD
- removed net N$9: R2.1, U$6.E
- new net LED_A: JP2.4, LED1.A, LED2.A, LED3.A
- new net LED_IN: JP2.6, LED6.4-DIN
- new net LED_O: JP2.5, LED4.2-DOUT
- new net LINE1: JP2.9, R3.1, U$6.E
- new net LINE2: JP2.8, R2.1, U$5.E
- new net LINE3: JP2.7, R1.1, U$4.E
- new net LINE4: JP2.3, U$3.P$3
- new net LINE5: JP2.2, U$2.P$3
- new net LINE6: JP2.1, U$1.P$3
- net +5V: now also JP2.10, LED4.1-VDD, LED5.1-VDD, LED6.1-VDD
- net GND: now also JP2.11
Routing:
- net +5V: track 0.00 -> 102.4 mm, vias 0 -> 1
- net LED_A: track 0.00 -> 71.3 mm
- net GND: track 65.9 -> 109.4 mm, vias 0 -> 4
- net LINE6: track 0.00 -> 43.4 mm
- net LINE4: track 0.00 -> 40.4 mm, vias 0 -> 1
- net LED_O: track 0.00 -> 32.9 mm, vias 0 -> 3
- net LINE3: track 0.00 -> 31.8 mm
- net LINE5: track 0.00 -> 29.2 mm
- net LINE2: track 0.00 -> 21.1 mm
- net LINE1: track 0.00 -> 10.9 mm
- net N$6: track 0.00 -> 9.53 mm
- net N$7: track 0.00 -> 9.49 mm
- net LED_IN: track 0.00 -> 6.65 mm, vias 0 -> 1
- net N$4: track 2.20 -> 0.00 mm
Other:
- board size 1317.6 x 228.6 mm -> 49 x 55.1 mm
