File: board/campile_wiring/untitled.brd (EAGLE design)
At the start: 38.7 x 33.3 mm, 9 parts, among them U1 74HC4067SSOP-24, U2 74HC4067SSOP-24

Commit message: 追加
Parts:
- removed U$1, U$2: SMD-R-TRIM, by_hirame:SMD-R-TRIM
- moved LINE 26.3 mm to (33.7, 9.53), flipped to the top, turned to 270 degrees
Routing:
- net GND: track 5.08 -> 0.00 mm
- net +5V: track 5.08 -> 0.00 mm
Changed lines of the file:
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@@
 <drawing>
 <settings>
-<setting alwaysvectorfont="yes"/>
+<setting alwaysvectorfont="no"/>
 <setting verticaltext="up"/>
 </settings>
@@
 <attribute name="NAME" x="20.16" y="7.31" size="1.27" layer="25" rot="R180"/>
 </element>
-<element name="LINE" library="con-lstb" library_urn="urn:adsk.eagle:library:162" package="MA07-2" package3d_urn="urn:adsk.eagle:package:8330/1" value="" x="8.255" y="16.51" smashed="yes" rot="MR90">
-<attribute name="MF" value="" x="3.175" y="39.37" size="1.778" layer="28" rot="MR90" display="off"/>
-<attribute name="MPN" value="" x="3.175" y="39.37" size="1.778" layer="28" rot="MR90" display="off"/>
-<attribute name="NAME" x="11.176" y="7.62" size="1.27" layer="26" ratio="10" rot="MR90"/>
-<attribute name="OC_FARNELL" value="unknown" x="3.175" y="39.37" size="1.778" layer="28" rot="MR90" display="off"/>
-<attribute name="OC_NEWARK" value="unknown" x="3.175" y="39.37" size="1.778" layer="28" rot="MR90" display="off"/>
-<attribute name="POPULARITY" value="1" x="3.175" y="39.37" size="1.778" layer="28" rot="MR90" display="off"/>
-<attribute name="VALUE" x="4.064" y="13.97" size="1.27" layer="28" ratio="10" rot="MR90"/>
+<element name="LINE" library="con-lstb" library_urn="urn:adsk.eagle:library:162" package="MA07-2" package3d_urn="urn:adsk.eagle:package:8330/1" value="" x="33.655" y="9.525" smashed="yes" rot="R270">
+<attribute name="MF" value="" x="28.575" y="-13.335" size="1.778" layer="27" rot="R270" display="off"/>
+<attribute name="MPN" value="" x="28.575" y="-13.335" size="1.778" layer="27" rot="R270" display="off"/>
+<attribute name="NAME" x="36.576" y="18.415" size="1.27" layer="25" ratio="10" rot="R270"/>
+<attribute name="OC_FARNELL" value="unknown" x="28.575" y="-13.335" size="1.778" layer="27" rot="R270" display="off"/>
+<attribute name="OC_NEWARK" value="unknown" x="28.575" y="-13.335" size="1.778" layer="27" rot="R270" display="off"/>
+<attribute name="POPULARITY" value="1" x="28.575" y="-13.335" size="1.778" layer="27" rot="R270" display="off"/>
+<attribute name="VALUE" x="29.464" y="12.065" size="1.27" layer="27" ratio="10" rot="R270"/>
 </element>
 <element name="U1" library="74HC4067" package="SSOP24" value="74HC4067SSOP-24" x="15.875" y="20.955" smashed="yes" rot="R90">
@@
 <attribute name="VALUE" x="16.555" y="8.1801" size="1.27" layer="27" rot="R90"/>
 </element>
-<element name="U$1" library="by_hirame" package="SMD-R-TRIM" value="SMD-R-TRIM" x="3.175" y="19.05" smashed="yes" rot="R270"/>
-<element name="U$2" library="by_hirame" package="SMD-R-TRIM" value="SMD-R-TRIM" x="3.175" y="22.86" smashed="yes" rot="R270"/>
 </elements>
 <signals>
@@
 <contactref element="JP3" pad="10"/>
 <contactref element="JP4" pad="7"/>
-<wire x1="23.495" y1="22.605" x2="28.575" y2="22.605" width="0.508" layer="1"/>
+<wire x1="23.495" y1="22.605" x2="14.16" y2="3.81" width="0" layer="19" extent="1-1"/>
 <wire x1="4.065" y1="28.575" x2="23.495" y2="22.605" width="0" layer="19" extent="1-1"/>
-<wire x1="14.16" y1="3.81" x2="23.495" y2="22.605" width="0" layer="19" extent="1-1"/>
+<wire x1="28.575" y1="22.605" x2="4.065" y2="28.575" width="0" layer="19" extent="1-1"/>
 </signal>
 <signal name="GND">
@@
 <contactref element="U1" pad="12"/>
 <contactref element="U2" pad="12"/>
-<wire x1="28.575" y1="24.605" x2="23.495" y2="24.605" width="0.508" layer="1"/>
-<wire x1="28.575" y1="24.605" x2="6.985" y2="13.97" width="0" layer="19" extent="1-1"/>
-<wire x1="19.5" y1="24.53" x2="23.495" y2="24.605" width="0" layer="19" extent="1-1"/>
+<wire x1="16.16" y1="3.81" x2="23.495" y2="24.605" width="0" layer="19" extent="1-1"/>
+<wire x1="2.065" y1="28.575" x2="23.495" y2="24.605" width="0" layer="19" extent="1-1"/>
+<wire x1="28.575" y1="24.605" x2="2.065" y2="28.575" width="0" layer="19" extent="1-1"/>
+<wire x1="19.5" y1="15.005" x2="28.575" y2="24.605" width="0" layer="19" extent="1-1"/>
 <wire x1="19.5" y1="15.005" x2="19.5" y2="24.53" width="0" layer="19" extent="1-1"/>
-<wire x1="16.16" y1="3.81" x2="19.5" y2="15.005" width="0" layer="19" extent="1-1"/>
-<wire x1="2.065" y1="28.575" x2="19.5" y2="24.53" width="0" layer="19" extent="1-1"/>
+<wire x1="32.385" y1="12.065" x2="19.5" y2="24.53" width="0" layer="19" extent="1-1"/>
 </signal>
 <signal name="LED_LA">
@@
 <contactref element="U2" pad="24"/>
 <contactref element="U1" pad="24"/>
-<wire x1="12.25" y1="7.855" x2="6.985" y2="19.05" width="0" layer="19" extent="1-1"/>
-<wire x1="12.25" y1="17.38" x2="12.25" y2="7.855" width="0" layer="19" extent="1-1"/>
+<wire x1="12.25" y1="17.38" x2="32.385" y2="6.985" width="0" layer="19" extent="1-1"/>
+<wire x1="12.25" y1="7.855" x2="12.25" y2="17.38" width="0" layer="19" extent="1-1"/>
 </signal>
 <signal name="LINE_LED">
@@
 <contactref element="U2" pad="10"/>
 <contactref element="LINE" pad="1"/>
-<wire x1="9.525" y1="21.59" x2="6.985" y2="8.89" width="0" layer="19" extent="1-1"/>
-<wire x1="19.5" y1="13.705" x2="9.525" y2="21.59" width="0" layer="19" extent="1-1"/>
-<wire x1="19.5" y1="23.23" x2="19.5" y2="13.705" width="0" layer="19" extent="1-1"/>
+<wire x1="19.5" y1="23.23" x2="32.385" y2="17.145" width="0" layer="19" extent="1-1"/>
+<wire x1="19.5" y1="23.23" x2="34.925" y2="4.445" width="0" layer="19" extent="1-1"/>
+<wire x1="19.5" y1="13.705" x2="19.5" y2="23.23" width="0" layer="19" extent="1-1"/>
 </signal>
 <signal name="LINE_S11">
@@
 <contactref element="U2" pad="11"/>
 <contactref element="LINE" pad="3"/>
-<wire x1="9.525" y1="19.05" x2="6.985" y2="11.43" width="0" layer="19" extent="1-1"/>
-<wire x1="19.5" y1="14.355" x2="9.525" y2="19.05" width="0" layer="19" extent="1-1"/>
-<wire x1="19.5" y1="23.88" x2="19.5" y2="14.355" width="0" layer="19" extent="1-1"/>
+<wire x1="34.925" y1="6.985" x2="32.385" y2="14.605" width="0" layer="19" extent="1-1"/>
+<wire x1="19.5" y1="23.88" x2="34.925" y2="6.985" width="0" layer="19" extent="1-1"/>
+<wire x1="19.5" y1="14.355" x2="19.5" y2="23.88" width="0" layer="19" extent="1-1"/>
 </signal>
 <signal name="LINE_S12">
@@
 <contactref element="U2" pad="14"/>
 <contactref element="LINE" pad="4"/>
-<wire x1="6.985" y1="24.13" x2="9.525" y2="11.43" width="0" layer="19" extent="1-1"/>
-<wire x1="12.25" y1="23.88" x2="9.525" y2="11.43" width="0" layer="19" extent="1-1"/>
+<wire x1="32.385" y1="1.905" x2="34.925" y2="14.605" width="0" layer="19" extent="1-1"/>
+<wire x1="12.25" y1="23.88" x2="34.925" y2="14.605" width="0" layer="19" extent="1-1"/>
 <wire x1="12.25" y1="14.355" x2="12.25" y2="23.88" width="0" layer="19" extent="1-1"/>
 </signal>
@@
 <contactref element="U2" pad="13"/>
 <contactref element="LINE" pad="6"/>
-<wire x1="6.985" y1="21.59" x2="9.525" y2="13.97" width="0" layer="19" extent="1-1"/>
-<wire x1="12.25" y1="15.005" x2="9.525" y2="13.97" width="0" layer="19" extent="1-1"/>
-<wire x1="12.25" y1="24.53" x2="12.25" y2="15.005" width="0" layer="19" extent="1-1"/>
+<wire x1="32.385" y1="4.445" x2="34.925" y2="12.065" width="0" layer="19" extent="1-1"/>
+<wire x1="12.25" y1="24.53" x2="34.925" y2="12.065" width="0" layer="19" extent="1-1"/>
+<wire x1="12.25" y1="15.005" x2="12.25" y2="24.53" width="0" layer="19" extent="1-1"/>
 </signal>
 <signal name="LINE_A1">
