File: board/campile_wiring/untitled.sch (EAGLE design)
At the start: 4 parts

Commit message: 追加
Parts:
- added LINE: (no value), con-lstb:MA07-2
- added U1, U2: 74HC4067SSOP-24, 74HC4067:74HC4067SSOP-24
Connections:
- removed net LINE_\F4: JP4.4
- new net +3V3: LINE.9, U1.VCC, U2.VCC
- new net LINE_A1: LINE.14
- new net LINE_A2: LINE.2
- new net LINE_F4: JP4.4, U1.CHAN3
- new net LINE_LED: LINE.7
- new net LINE_R3: U1.CHAN8
- new net LINE_S10: LINE.1, LINE.12, U1.S0, U2.S0
- new net LINE_S11: LINE.10, LINE.3, U1.S1, U2.S1
- new net LINE_S12: LINE.13, LINE.4, U1.S2, U2.S2
- new net LINE_S13: LINE.11, LINE.6, U1.S3, U2.S3
- net GND: now also LINE.5, U1.GND, U2.GND
- net LINE_B1: now also U2.CHAN0
- net LINE_B2: now also U2.CHAN1
- net LINE_B3: now also U2.CHAN2
- net LINE_B4: now also U2.CHAN3
- net LINE_B5: now also U2.CHAN4
- net LINE_B6: now also U2.CHAN5
- net LINE_F1: now also U1.CHAN0
- net LINE_F2: now also U1.CHAN1
- net LINE_F3: now also U1.CHAN2
- net LINE_F5: now also U1.CHAN4
- net LINE_F6: now also U1.CHAN5
- net LINE_L1: now also U2.CHAN6
- net LINE_L2: now also U2.CHAN7
- net LINE_L3: now also U2.CHAN8
- net LINE_L4: now also U2.CHAN9
- net LINE_L5: now also U2.CHAN10
- net LINE_L6: now also U2.CHAN11
- net LINE_R1: now also U1.CHAN6
- net LINE_R2: now also U1.CHAN7
- net LINE_R4: now also U1.CHAN9
- net LINE_R5: now also U1.CHAN10
- net LINE_R6: now also U1.CHAN11
